Commit message: fix: COMPACT MODE FINALLY WORKS

File: src/indomitus_rover_description/urdf/indomitus_rover_s1.urdf.xacro (robot description, xacro)
@@ -163,5 +163,5 @@
     <origin xyz="0.53 0 0" rpy="0 0 0"/>
     <axis xyz="0 0 1"/>
-    <limit lower="-1.5708" upper="1.5708" effort="500" velocity="2"/>
+    <limit lower="-4.71238898" upper="4.71238898" effort="500" velocity="2"/>
     <dynamics damping="0.5" friction="0.3"/>
   </joint>
@@ -220,5 +220,5 @@
     <origin xyz="0.53 0 0" rpy="0 0 0"/>
     <axis xyz="0 0 1"/>
-    <limit lower="-1.5708" upper="1.5708" effort="500" velocity="2"/>
+    <limit lower="-4.71238898" upper="4.71238898" effort="500" velocity="2"/>
     <dynamics damping="0.5" friction="0.3"/>
   </joint>
@@ -277,5 +277,5 @@
     <origin xyz="-0.53 0 0" rpy="0 0 0"/>
     <axis xyz="0 0 1"/>
-    <limit lower="-1.5708" upper="1.5708" effort="500" velocity="2"/>
+    <limit lower="-4.71238898" upper="4.71238898" effort="500" velocity="2"/>
     <dynamics damping="0.5" friction="0.3"/>
   </joint>
@@ -334,5 +334,5 @@
     <origin xyz="-0.53 0 0" rpy="0 0 0"/>
     <axis xyz="0 0 1"/>
-    <limit lower="-1.5708" upper="1.5708" effort="500" velocity="2"/>
+    <limit lower="-4.71238898" upper="4.71238898" effort="500" velocity="2"/>
     <dynamics damping="0.5" friction="0.3"/>
   </joint>
