Commit message: fix: minor fixes to urdf files; it works now, I tested, but some improvements are needed

File: src/rover_description/urdf/ros2_control_real.urdf.xacro (robot description, xacro)
@@ -5,24 +5,22 @@
       <plugin>rover_hardware_interface/RoverHardwareInterface</plugin>
       <param name="can_interface">$(arg can_interface)</param>
+      <param name="steer_ids">11 13 17 15</param>
+      <param name="drive_ids">10 12 16 14</param>
     </hardware>
     <joint name="fl_wheel_mount_joint">
       <command_interface name="position"/>
       <state_interface name="position"/>
-      <state_interface name="velocity"/>
     </joint>
     <joint name="fr_wheel_mount_joint">
       <command_interface name="position"/>
       <state_interface name="position"/>
-      <state_interface name="velocity"/>
     </joint>
     <joint name="bl_wheel_mount_joint">
       <command_interface name="position"/>
       <state_interface name="position"/>
-      <state_interface name="velocity"/>
     </joint>
     <joint name="br_wheel_mount_joint">
       <command_interface name="position"/>
       <state_interface name="position"/>
-      <state_interface name="velocity"/>
     </joint>
     <joint name="fl_wheel_joint">
@@ -46,12 +44,4 @@
       <state_interface name="velocity"/>
     </joint>
-    <joint name="l_rocker_joint">
-      <state_interface name="position"/>
-      <state_interface name="velocity"/>
-    </joint>
-    <joint name="r_rocker_joint">
-      <state_interface name="position"/>
-      <state_interface name="velocity"/>
-    </joint>
   </ros2_control>
 </robot>

File: src/rover_description/urdf/rover_s1.urdf.xacro (robot description, xacro)
@@ -41,5 +41,5 @@
       <origin xyz="0 0 0" rpy="0 0 0"/>
       <geometry>
-        <box size="0.1 0.65 0.05"/>
+        <box size="0.1 0.68 0.05"/>
       </geometry>
     </collision>
@@ -103,5 +103,5 @@
     <parent link="suspension_base_axii_link"/>
     <child link="l_rocker_link"/>
-    <origin xyz="0 0.305 0" rpy="0 0 0"/>
+    <origin xyz="0 0.34 0" rpy="0 0 0"/>
     <axis xyz="0 1 0"/>
     <limit lower="-0.5" upper="0.5" effort="100" velocity="1.0"/>
@@ -132,5 +132,5 @@
     <parent link="suspension_base_axii_link"/>
     <child link="r_rocker_link"/>
-    <origin xyz="0 -0.305 0" rpy="0 0 0"/>
+    <origin xyz="0 -0.34 0" rpy="0 0 0"/>
     <axis xyz="0 1 0"/>
     <limit lower="-0.5" upper="0.5" effort="100" velocity="1.0"/>
@@ -161,5 +161,5 @@
     <parent link="l_rocker_link"/>
     <child link="fl_wheel_mount_link"/>
-    <origin xyz="0.53 0 0" rpy="0 0 0"/>
+    <origin xyz="0.421 0 0" rpy="0 0 0"/>
     <axis xyz="0 0 1"/>
     <limit lower="-4.71238898" upper="4.71238898" effort="500" velocity="2"/>
@@ -218,5 +218,5 @@
     <parent link="r_rocker_link"/>
     <child link="fr_wheel_mount_link"/>
-    <origin xyz="0.53 0 0" rpy="0 0 0"/>
+    <origin xyz="0.421 0 0" rpy="0 0 0"/>
     <axis xyz="0 0 1"/>
     <limit lower="-4.71238898" upper="4.71238898" effort="500" velocity="2"/>
@@ -275,5 +275,5 @@
     <parent link="l_rocker_link"/>
     <child link="bl_wheel_mount_link"/>
-    <origin xyz="-0.53 0 0" rpy="0 0 0"/>
+    <origin xyz="-0.421 0 0" rpy="0 0 0"/>
     <axis xyz="0 0 1"/>
     <limit lower="-4.71238898" upper="4.71238898" effort="500" velocity="2"/>
@@ -332,5 +332,5 @@
     <parent link="r_rocker_link"/>
     <child link="br_wheel_mount_link"/>
-    <origin xyz="-0.53 0 0" rpy="0 0 0"/>
+    <origin xyz="-0.421 0 0" rpy="0 0 0"/>
     <axis xyz="0 0 1"/>
     <limit lower="-4.71238898" upper="4.71238898" effort="500" velocity="2"/>
