Commit message: Refactor/suspension/ros2 control architecture (#452)
* feature: add chassis_controller package structure

* feature: add swerve_controller.cpp

* feature: add hardware_interface

* fix: fix hardware_interface.hpp

* fix: fix launch files and edsccription files

* fix: now it compiles

* fix: fix swerveController names

* fix: at least it compiles

* fix: IT WORKS

* fix: remap ~/cmd_vel into /cmd_vel

* fix: restructure urdf files

* fix: minor fixes to urdf files; it works now, I tested, but some improvements are needed

* fix: change names of urdf files to make structure more consistent

* fix: add hardwawre_component deactivate via joystick

* fix: fix bug related with slow rotation

* fix: remove one of step_angles functions calls

* fix: fix parameters in config yaml files

* fix: fix bug with controller deactivation, make turning smoother

* fix: fix bugs that appeared on humble

* fix: fix all minor bugs caused by transition on jetson nano; change joy package, optimize deployment pipeline

* feature: add granny mode, speed*0.1

* chore: change readme for harware_interface package

* fix: move ros2 dependencies to package.xml from dockerfile

* fix: fix issues mentined in PR review

* chore: remove deprecated tests for kinematics in rover_control pkg

File: src/rover_description/urdf/ros2_control_real.xacro (robot description, xacro)
@@ -1,29 +1,28 @@
 <?xml version="1.0"?>
 <robot xmlns:xacro="http://www.ros.org/wiki/xacro">
-  <ros2_control name="GazeboSystem" type="system">
+  <ros2_control name="RoverHardware" type="system">
     <hardware>
-      <plugin>gz_ros2_control/GazeboSimSystem</plugin>
+      <plugin>rover_hardware_interface/RoverHardwareInterface</plugin>
+      <param name="can_interface">$(arg can_interface)</param>
+      <param name="steer_ids">11 13 17 15</param>
+      <param name="drive_ids">10 12 16 14</param>
+      <param name="lifecycle_initial_state">inactive</param>
     </hardware>
     <joint name="fl_wheel_mount_joint">
       <command_interface name="position"/>
       <state_interface name="position"/>
-      <state_interface name="velocity"/>
     </joint>
     <joint name="fr_wheel_mount_joint">
       <command_interface name="position"/>
       <state_interface name="position"/>
-      <state_interface name="velocity"/>
     </joint>
     <joint name="bl_wheel_mount_joint">
       <command_interface name="position"/>
       <state_interface name="position"/>
-      <state_interface name="velocity"/>
     </joint>
     <joint name="br_wheel_mount_joint">
       <command_interface name="position"/>
       <state_interface name="position"/>
-      <state_interface name="velocity"/>
     </joint>
-    <!-- Drive joints — керування швидкістю обертання -->
     <joint name="fl_wheel_joint">
       <command_interface name="velocity"/>
@@ -46,26 +45,4 @@
       <state_interface name="velocity"/>
     </joint>
-    <joint name="l_rocker_joint">
-      <!-- <command_interface name="position"/> -->
-      <state_interface name="position"/>
-      <state_interface name="velocity"/>
-    </joint>
-    <joint name="r_rocker_joint">
-      <command_interface name="position"/>
-      <state_interface name="position"/>
-      <state_interface name="velocity"/>
-    </joint>
   </ros2_control>
-  <!-- gz_ros2_control plugin -->
-  <gazebo>
-    <plugin filename="gz_ros2_control-system"
-            name="gz_ros2_control::GazeboSimROS2ControlPlugin">
-      <parameters>$(find rover_sim)/parameters/ros2_control.yaml</parameters>
-    </plugin>
-  </gazebo>
-  <gazebo>
-    <plugin filename="gz-sim-joint-state-publisher-system"
-            name="gz::sim::systems::JointStatePublisher">
-    </plugin>
-  </gazebo>
 </robot>

File: src/rover_description/urdf/rover.urdf.xacro (robot description, xacro)
@@ -41,5 +41,5 @@
       <origin xyz="0 0 0" rpy="0 0 0"/>
       <geometry>
-        <box size="0.1 0.65 0.05"/>
+        <box size="0.1 0.68 0.05"/>
       </geometry>
     </collision>
@@ -77,5 +77,5 @@
   </joint>
   <!-- ===================== CAMERA ===================== -->
-  <xacro:include filename="$(find rover_description)/urdf/camera.urdf.xacro"/>
+  <xacro:include filename="$(find rover_description)/urdf/camera.xacro"/>
   <xacro:camera/>
   <!-- ===================== LEFT ROCKER ===================== -->
@@ -103,5 +103,5 @@
     <parent link="suspension_base_axii_link"/>
     <child link="l_rocker_link"/>
-    <origin xyz="0 0.305 0" rpy="0 0 0"/>
+    <origin xyz="0 0.34 0" rpy="0 0 0"/>
     <axis xyz="0 1 0"/>
     <limit lower="-0.5" upper="0.5" effort="100" velocity="1.0"/>
@@ -132,5 +132,5 @@
     <parent link="suspension_base_axii_link"/>
     <child link="r_rocker_link"/>
-    <origin xyz="0 -0.305 0" rpy="0 0 0"/>
+    <origin xyz="0 -0.34 0" rpy="0 0 0"/>
     <axis xyz="0 1 0"/>
     <limit lower="-0.5" upper="0.5" effort="100" velocity="1.0"/>
@@ -161,5 +161,5 @@
     <parent link="l_rocker_link"/>
     <child link="fl_wheel_mount_link"/>
-    <origin xyz="0.53 0 0" rpy="0 0 0"/>
+    <origin xyz="0.421 0 0" rpy="0 0 0"/>
     <axis xyz="0 0 1"/>
     <limit lower="-4.71238898" upper="4.71238898" effort="500" velocity="2"/>
@@ -218,5 +218,5 @@
     <parent link="r_rocker_link"/>
     <child link="fr_wheel_mount_link"/>
-    <origin xyz="0.53 0 0" rpy="0 0 0"/>
+    <origin xyz="0.421 0 0" rpy="0 0 0"/>
     <axis xyz="0 0 1"/>
     <limit lower="-4.71238898" upper="4.71238898" effort="500" velocity="2"/>
@@ -275,5 +275,5 @@
     <parent link="l_rocker_link"/>
     <child link="bl_wheel_mount_link"/>
-    <origin xyz="-0.53 0 0" rpy="0 0 0"/>
+    <origin xyz="-0.421 0 0" rpy="0 0 0"/>
     <axis xyz="0 0 1"/>
     <limit lower="-4.71238898" upper="4.71238898" effort="500" velocity="2"/>
@@ -332,5 +332,5 @@
     <parent link="r_rocker_link"/>
     <child link="br_wheel_mount_link"/>
-    <origin xyz="-0.53 0 0" rpy="0 0 0"/>
+    <origin xyz="-0.421 0 0" rpy="0 0 0"/>
     <axis xyz="0 0 1"/>
     <limit lower="-4.71238898" upper="4.71238898" effort="500" velocity="2"/>
