Commit message: feat(sim): add simulation-only lidar for nav2 testing

File: src/rover_description/urdf/rover.urdf.xacro (robot description, xacro)
@@ -79,4 +79,53 @@
   <xacro:include filename="$(find rover_description)/urdf/camera.xacro"/>
   <xacro:camera/>
+  <!-- NOTE: Simulation-only lidar for nav2 testing. Replace with real sensor
+     description and bridge when deploying on hardware. -->
+  <link name="lidar_link">
+    <inertial>
+      <origin xyz="0 0 0" rpy="0 0 0"/>
+      <mass value="0.2"/>
+      <inertia ixx="0.0001" iyy="0.0001" izz="0.0002" ixy="0" ixz="0" iyz="0"/>
+    </inertial>
+    <visual>
+      <origin xyz="0 0 0" rpy="0 0 0"/>
+      <geometry>
+        <cylinder radius="0.05" length="0.04"/>
+      </geometry>
+      <material name="orange_mount"/>
+    </visual>
+    <collision>
+      <origin xyz="0 0 0" rpy="0 0 0"/>
+      <geometry>
+        <cylinder radius="0.05" length="0.04"/>
+      </geometry>
+    </collision>
+  </link>
+  <joint name="lidar_joint" type="fixed">
+    <parent link="main_body_link"/>
+    <child link="lidar_link"/>
+    <origin xyz="0.2 0 0.12" rpy="0 0 0"/>
+  </joint>
+  <gazebo reference="lidar_link">
+    <sensor type="gpu_lidar" name="generic_laser">
+      <update_rate>10.0</update_rate>
+      <topic>/scan</topic>
+      <gz_frame_id>lidar_link</gz_frame_id>
+      <lidar>
+        <scan>
+          <horizontal>
+            <samples>360</samples>
+            <resolution>1</resolution>
+            <min_angle>-3.141592</min_angle>
+            <max_angle>3.141592</max_angle>
+          </horizontal>
+        </scan>
+        <range>
+          <min>0.12</min>
+          <max>10.0</max>
+          <resolution>0.01</resolution>
+        </range>
+      </lidar>
+    </sensor>
+  </gazebo>
   <!-- ===================== LEFT ROCKER ===================== -->
   <link name="l_rocker_link">

Commit message: fix(nav2): align lidar frame id to laser_link to match RPLidar driver output

File: src/rover_description/urdf/rover.urdf.xacro (robot description, xacro)
@@ -81,5 +81,5 @@
   <!-- NOTE: Simulation-only lidar for nav2 testing. Replace with real sensor
      description and bridge when deploying on hardware. -->
-  <link name="lidar_link">
+  <link name="laser_link">
     <inertial>
       <origin xyz="0 0 0" rpy="0 0 0"/>
@@ -101,14 +101,14 @@
     </collision>
   </link>
-  <joint name="lidar_joint" type="fixed">
+  <joint name="laser_joint" type="fixed">
     <parent link="main_body_link"/>
-    <child link="lidar_link"/>
+    <child link="laser_link"/>
     <origin xyz="0.2 0 0.12" rpy="0 0 0"/>
   </joint>
-  <gazebo reference="lidar_link">
+  <gazebo reference="laser_link">
     <sensor type="gpu_lidar" name="generic_laser">
       <update_rate>10.0</update_rate>
       <topic>/scan</topic>
-      <gz_frame_id>lidar_link</gz_frame_id>
+      <gz_frame_id>laser_link</gz_frame_id>
       <lidar>
         <scan>
