Commit message: fix(sim): decouple nav2 lidar and bridge config from base simulation

File: src/rover_description/urdf/rover.urdf.xacro (robot description, xacro)
@@ -79,53 +79,4 @@
   <xacro:include filename="$(find rover_description)/urdf/camera.xacro"/>
   <xacro:camera/>
-  <!-- NOTE: Simulation-only lidar for nav2 testing. Replace with real sensor
-     description and bridge when deploying on hardware. -->
-  <link name="laser_link">
-    <inertial>
-      <origin xyz="0 0 0" rpy="0 0 0"/>
-      <mass value="0.2"/>
-      <inertia ixx="0.0001" iyy="0.0001" izz="0.0002" ixy="0" ixz="0" iyz="0"/>
-    </inertial>
-    <visual>
-      <origin xyz="0 0 0" rpy="0 0 0"/>
-      <geometry>
-        <cylinder radius="0.05" length="0.04"/>
-      </geometry>
-      <material name="orange_mount"/>
-    </visual>
-    <collision>
-      <origin xyz="0 0 0" rpy="0 0 0"/>
-      <geometry>
-        <cylinder radius="0.05" length="0.04"/>
-      </geometry>
-    </collision>
-  </link>
-  <joint name="laser_joint" type="fixed">
-    <parent link="main_body_link"/>
-    <child link="laser_link"/>
-    <origin xyz="0.2 0 0.12" rpy="0 0 0"/>
-  </joint>
-  <gazebo reference="laser_link">
-    <sensor type="gpu_lidar" name="generic_laser">
-      <update_rate>10.0</update_rate>
-      <topic>/scan</topic>
-      <gz_frame_id>laser_link</gz_frame_id>
-      <lidar>
-        <scan>
-          <horizontal>
-            <samples>360</samples>
-            <resolution>1</resolution>
-            <min_angle>-3.141592</min_angle>
-            <max_angle>3.141592</max_angle>
-          </horizontal>
-        </scan>
-        <range>
-          <min>0.12</min>
-          <max>10.0</max>
-          <resolution>0.01</resolution>
-        </range>
-      </lidar>
-    </sensor>
-  </gazebo>
   <!-- ===================== LEFT ROCKER ===================== -->
   <link name="l_rocker_link">

File: src/rover_sim/urdf/rover_sim_nav2.urdf.xacro (robot description, xacro)
@@ -4,4 +4,5 @@
   <xacro:include filename="$(find rover_description)/urdf/ros2_control_sim.xacro"/>
   <xacro:include filename="$(find rover_description)/urdf/gz_odometry.xacro"/>
+  <xacro:include filename="$(find rover_description)/urdf/lidar_sim.xacro"/>
   <gazebo>
     <plugin filename="gz_ros2_control-system"

Commit message: feat: basic setup for the real world autonomous navigation wiht zed2i made

File: src/rover_description/urdf/rover.urdf.xacro (robot description, xacro)
@@ -76,7 +76,9 @@
     <origin xyz="-0.04 0 0.05" rpy="0 0 0"/>
   </joint>
-  <!-- ===================== CAMERA ===================== -->
-  <xacro:include filename="$(find rover_description)/urdf/camera.xacro"/>
-  <xacro:camera/>
+  <!-- ===================== ZED2i STEREO CAMERA ===================== -->
+  <xacro:include filename="$(find zed_wrapper)/urdf/zed_macro.urdf.xacro" />
+  <xacro:zed_camera name="zed2i" model="zed2i" parent="main_body_link">
+    <origin xyz="0.65 0 0.50" rpy="0 ${pi/12} 0"/>
+  </xacro:zed_camera>
   <!-- ===================== LEFT ROCKER ===================== -->
   <link name="l_rocker_link">

Commit message: fix: in the include of the zed2i to the urdf

File: src/rover_description/urdf/rover.urdf.xacro (robot description, xacro)
@@ -78,7 +78,10 @@
   <!-- ===================== ZED2i STEREO CAMERA ===================== -->
   <xacro:include filename="$(find zed_wrapper)/urdf/zed_macro.urdf.xacro" />
-  <xacro:zed_camera name="zed2i" model="zed2i" parent="main_body_link">
-    <origin xyz="0.65 0 0.50" rpy="0 ${pi/12} 0"/>
-  </xacro:zed_camera>
+  <xacro:zed_camera name="zed2i" model="zed2i"/>
+  <joint name="zed2i_base_joint" type="fixed">
+    <parent link="main_body_link"/>
+    <child link="zed2i_camera_link"/>
+    <origin xyz="0.65 0 0.08" rpy="0 ${pi/12} 0"/>
+  </joint>
   <!-- ===================== LEFT ROCKER ===================== -->
   <link name="l_rocker_link">

Commit message: zed2i stereo camera added to the robot urdf

File: src/rover_description/urdf/rover.urdf.xacro (robot description, xacro)
@@ -77,10 +77,14 @@
   </joint>
   <!-- ===================== ZED2i STEREO CAMERA ===================== -->
-  <xacro:include filename="$(find zed_wrapper)/urdf/zed_macro.urdf.xacro" />
-  <xacro:zed_camera name="zed2i" model="zed2i"/>
+  <xacro:include filename="$(find zed_description)/urdf/zed_macro.urdf.xacro" />
+  <xacro:zed_camera name="zed2i" model="zed2i">
+      <gnss_origin>
+          <origin xyz="0 0 0" rpy="0 0 0" />
+      </gnss_origin>
+  </xacro:zed_camera>
   <joint name="zed2i_base_joint" type="fixed">
     <parent link="main_body_link"/>
     <child link="zed2i_camera_link"/>
-    <origin xyz="0.65 0 0.08" rpy="0 ${pi/12} 0"/>
+    <origin xyz="0.35 0 0.18" rpy="0 ${pi/12} 0"/>
   </joint>
   <!-- ===================== LEFT ROCKER ===================== -->

Commit message: feat: 'working' navigation

File: src/rover_description/urdf/rover.urdf.xacro (robot description, xacro)
@@ -45,9 +45,9 @@
     </collision>
   </link>
-  <joint name="suspension_base_axii_joint" type="fixed">
-    <parent link="base_link"/>
-    <child link="suspension_base_axii_link"/>
-    <origin xyz="0 0 0" rpy="0 0 0"/>
-  </joint>
+<joint name="suspension_base_axii_joint" type="fixed">
+  <parent link="suspension_base_axii_link"/>
+  <child link="base_link"/>
+  <origin xyz="0 0 0" rpy="0 0 0"/>
+</joint>
   <!-- ===================== MAIN BODY ===================== -->
   <link name="main_body_link">
@@ -72,7 +72,7 @@
   </link>
   <joint name="main_body_joint" type="fixed">
-    <parent link="suspension_base_axii_link"/>
-    <child link="main_body_link"/>
-    <origin xyz="-0.04 0 0.05" rpy="0 0 0"/>
+    <parent link="main_body_link"/>
+    <child link="suspension_base_axii_link"/>
+    <origin xyz="0.04 0 -0.05" rpy="0 0 0"/>
   </joint>
   <!-- ===================== ZED2i STEREO CAMERA ===================== -->
@@ -84,7 +84,7 @@
   </xacro:zed_camera>
   <joint name="zed2i_base_joint" type="fixed">
-    <parent link="main_body_link"/>
-    <child link="zed2i_camera_link"/>
-    <origin xyz="0.35 0 0.18" rpy="0 ${pi/12} 0"/>
+    <parent link="zed2i_camera_link"/>
+    <child link="main_body_link"/>
+    <origin xyz="-0.2915 0 -0.2644" rpy="0 ${-pi/12} 0"/>
   </joint>
   <!-- ===================== LEFT ROCKER ===================== -->

Commit message: feat: rever urdf updated to include zed2i stereo camera

File: src/rover_description/urdf/rover.urdf.xacro (robot description, xacro)
@@ -45,9 +45,9 @@
     </collision>
   </link>
-  <joint name="suspension_base_axii_joint" type="fixed">
-    <parent link="base_link"/>
-    <child link="suspension_base_axii_link"/>
-    <origin xyz="0 0 0" rpy="0 0 0"/>
-  </joint>
+<joint name="suspension_base_axii_joint" type="fixed">
+  <parent link="suspension_base_axii_link"/>
+  <child link="base_link"/>
+  <origin xyz="0 0 0" rpy="0 0 0"/>
+</joint>
   <!-- ===================== MAIN BODY ===================== -->
   <link name="main_body_link">
@@ -72,11 +72,20 @@
   </link>
   <joint name="main_body_joint" type="fixed">
-    <parent link="suspension_base_axii_link"/>
+    <parent link="main_body_link"/>
+    <child link="suspension_base_axii_link"/>
+    <origin xyz="0.04 0 -0.05" rpy="0 0 0"/>
+  </joint>
+  <!-- ===================== ZED2i STEREO CAMERA ===================== -->
+  <xacro:include filename="$(find zed_description)/urdf/zed_macro.urdf.xacro" />
+  <xacro:zed_camera name="zed2i" model="zed2i">
+      <gnss_origin>
+          <origin xyz="0 0 0" rpy="0 0 0" />
+      </gnss_origin>
+  </xacro:zed_camera>
+  <joint name="zed2i_base_joint" type="fixed">
+    <parent link="zed2i_camera_link"/>
     <child link="main_body_link"/>
-    <origin xyz="-0.04 0 0.05" rpy="0 0 0"/>
-  </joint>
-  <!-- ===================== CAMERA ===================== -->
-  <xacro:include filename="$(find rover_description)/urdf/camera.xacro"/>
-  <xacro:camera/>
+    <origin xyz="-0.2915 0 -0.2644" rpy="0 ${-pi/12} 0"/>
+  </joint>
   <!-- ===================== LEFT ROCKER ===================== -->
   <link name="l_rocker_link">

Commit message: feat: imu added to the simulation; all topics of zed2i remaped to more readable names

File: src/rover_description/urdf/rover.urdf.xacro (robot description, xacro)
@@ -82,4 +82,5 @@
     simulate_rgb="$(arg stereo_camera_simulate_rgb)"
     simulate_pointcloud="$(arg stereo_camera_simulate_pointcloud)"
+    simulate_imu="$(arg stereo_camera_simulate_imu)"
   />
   <joint name="zed2i_base_joint" type="fixed">

File: src/rover_description/urdf/rover.xacro (robot description, xacro)
@@ -9,4 +9,5 @@
   <xacro:arg name="stereo_camera_simulate_rgb" default="false"/>
   <xacro:arg name="stereo_camera_simulate_pointcloud" default="false"/>
+  <xacro:arg name="stereo_camera_simulate_imu" default="false"/>
   <!-- Main robot description -->
   <xacro:include filename="$(find rover_description)/urdf/rover.urdf.xacro"/>

File: src/rover_description/urdf/stereo_camera.xacro (robot description, xacro)
@@ -5,5 +5,11 @@
     The visual/collision geometry and joint are always added.
   -->
-  <xacro:macro name="stereo_camera" params="use_sim:=false simulate_rgb:=false simulate_pointcloud:=false">
+  <xacro:macro
+    name="stereo_camera"
+    params="use_sim:=false
+            simulate_rgb:=false
+            simulate_pointcloud:=false
+            simulate_imu:=false"
+  >
     <xacro:include filename="$(find zed_description)/urdf/zed_macro.urdf.xacro" />
     <xacro:zed_camera name="zed2i" model="zed2i">
@@ -12,4 +18,5 @@
       </gnss_origin>
     </xacro:zed_camera>
+    <!-- RGB CAMERA PLUGIN -->
     <xacro:if value="${use_sim and simulate_rgb}">
       <gazebo reference="zed2i_left_camera_frame">
@@ -41,4 +48,5 @@
       </gazebo>
     </xacro:if>
+    <!-- DEPTH & POINTCLOUD PLUGIN -->
     <xacro:if value="${use_sim and simulate_pointcloud}">
       <gazebo reference="zed2i_left_camera_frame">
@@ -54,6 +62,6 @@
             </image>
             <clip>
-              <near>0.3</near>
-              <far>20.0</far>
+              <near>0.01</near>
+              <far>15.0</far>
             </clip>
           </camera>
@@ -68,6 +76,22 @@
             <camera_name>depth</camera_name>
             <frame_name>zed2i_left_camera_optical_frame</frame_name>
-            <min_depth>0.3</min_depth>
-            <max_depth>20.0</max_depth>
+            <min_depth>0.01</min_depth>
+            <max_depth>15.0</max_depth>
+          </plugin>
+        </sensor>
+      </gazebo>
+    </xacro:if>
+    <!-- IMU PLUGIN -->
+    <xacro:if value="${use_sim and simulate_imu}">
+      <gazebo reference="zed2i_left_camera_frame">
+        <sensor name="zed2i_imu_sensor" type="imu">
+          <always_on>true</always_on>
+          <update_rate>100.0</update_rate>
+          <plugin name="zed2i_imu_plugin" filename="libgazebo_ros_imu_sensor.so">
+            <ros>
+              <namespace>zed2i</namespace>
+              <remapping>~/out:=imu/data</remapping>
+            </ros>
+            <initial_orientation_as_reference>false</initial_orientation_as_reference>
           </plugin>
         </sensor>

Commit message: feat: base_footprint frame added as the new root

File: src/rover_description/urdf/rover.urdf.xacro (robot description, xacro)
@@ -17,4 +17,11 @@
     <color rgba="0.4 0.4 0.4 1"/>
   </material>
+  <!-- ===================== BASE FOOTPRINT ===================== -->
+  <link name="base_footprint"/>
+  <joint name="base_footprint_joint" type="fixed">
+    <parent link="base_footprint"/>
+    <child link="base_link"/>
+    <origin xyz="0 0 0.42" rpy="0 0 0"/>
+  </joint>
   <!-- ===================== BASE ===================== -->
   <link name="base_link">
@@ -45,9 +52,9 @@
     </collision>
   </link>
-<joint name="suspension_base_axii_joint" type="fixed">
-  <parent link="suspension_base_axii_link"/>
-  <child link="base_link"/>
-  <origin xyz="0 0 0" rpy="0 0 0"/>
-</joint>
+  <joint name="suspension_base_axii_joint" type="fixed">
+    <parent link="base_link"/>
+    <child link="suspension_base_axii_link"/>
+    <origin xyz="0 0 0" rpy="0 0 0"/>
+  </joint>
   <!-- ===================== MAIN BODY ===================== -->
   <link name="main_body_link">
@@ -72,7 +79,7 @@
   </link>
   <joint name="main_body_joint" type="fixed">
-    <parent link="main_body_link"/>
-    <child link="suspension_base_axii_link"/>
-    <origin xyz="0.04 0 -0.05" rpy="0 0 0"/>
+    <parent link="suspension_base_axii_link"/>
+    <child link="main_body_link"/>
+    <origin xyz="-0.04 0 0.05" rpy="0 0 0"/>
   </joint>
   <!-- ===================== ZED2i STEREO CAMERA ===================== -->
@@ -85,7 +92,7 @@
   />
   <joint name="zed2i_base_joint" type="fixed">
-    <parent link="zed2i_camera_link"/>
-    <child link="main_body_link"/>
-    <origin xyz="-0.2915 0 -0.2644" rpy="0 ${-pi/12} 0"/>
+    <parent link="main_body_link"/>
+    <child link="zed2i_camera_link"/>
+    <origin xyz="0.350039 0 0.179931" rpy="0 ${pi/12} 0"/>
   </joint>
   <!-- ===================== RPLIDAR S2 ===================== -->

File: src/rover_description/urdf/stereo_camera.xacro (robot description, xacro)
@@ -19,5 +19,6 @@
           <update_rate>20.0</update_rate>
           <topic>/zed2i/rgb/image_rect_color</topic>
-          <gz_frame_id>zed2i_left_camera_optical_frame</gz_frame_id>
+          <ignition_frame_id>zed2i_left_camera_frame_optical</ignition_frame_id>
+          <gz_frame_id>zed2i_left_camera_frame_optical</gz_frame_id>
           <camera>
             <camera_info_topic>/zed2i/rgb/camera_info</camera_info_topic>
@@ -41,17 +42,18 @@
         <sensor type="depth_camera" name="zed2i_depth_sensor">
           <always_on>true</always_on>
-          <update_rate>15.0</update_rate>
+          <update_rate>10.0</update_rate>
           <topic>/zed2i/depth/depth_registered</topic>
-          <gz_frame_id>zed2i_left_camera_optical_frame</gz_frame_id>
+          <ignition_frame_id>zed2i_left_camera_frame</ignition_frame_id>
+          <gz_frame_id>zed2i_left_camera_frame</gz_frame_id>
           <camera>
             <camera_info_topic>/zed2i/depth/camera_info</camera_info_topic>
             <horizontal_fov>1.91986</horizontal_fov>
             <image>
-              <width>640</width>
-              <height>360</height>
+              <width>320</width>
+              <height>180</height>
               <format>R_FLOAT32</format>
             </image>
             <clip>
-              <near>0.01</near>
+              <near>0.3</near>
               <far>15.0</far>
             </clip>

Commit message: chore: minor changes in the rover urdf

File: src/rover_description/urdf/rover.urdf.xacro (robot description, xacro)
@@ -94,5 +94,5 @@
     <parent link="main_body_link"/>
     <child link="zed2i_camera_link"/>
-    <origin xyz="0.350039 0 0.179931" rpy="0 ${pi/12} 0"/>
+    <origin xyz="0.35 0 0.19" rpy="0 ${pi/12} 0"/>
   </joint>
   <!-- ===================== RPLIDAR S2 ===================== -->
@@ -105,5 +105,5 @@
     <parent link="main_body_link"/>
     <child link="laser_link"/>
-    <origin xyz="0 0 0.17" rpy="0 0 0"/>
+    <origin xyz="0 0 0.1" rpy="0 0 0"/>
   </joint>
   <!-- ===================== LEFT ROCKER ===================== -->

Commit message: fix: lidar position fixed in the rover urdf

File: src/rover_description/urdf/rover.urdf.xacro (robot description, xacro)
@@ -105,5 +105,5 @@
     <parent link="main_body_link"/>
     <child link="laser_link"/>
-    <origin xyz="0 0 0.1" rpy="0 0 0"/>
+    <origin xyz="0 0 0.17" rpy="0 0 0"/>
   </joint>
   <!-- ===================== LEFT ROCKER ===================== -->

File: src/rover_description/urdf/stereo_camera.xacro (robot description, xacro)
@@ -61,5 +61,5 @@
             </image>
             <clip>
-              <near>0.4</near>
+              <near>0.45</near>
               <far>15.0</far>
             </clip>

Commit message: chore: minor change in the zed2i position on the rover

File: src/rover_description/urdf/rover.urdf.xacro (robot description, xacro)
@@ -94,5 +94,5 @@
     <parent link="main_body_link"/>
     <child link="zed2i_camera_link"/>
-    <origin xyz="0.35 0 0.19" rpy="0 ${pi/12} 0"/>
+    <origin xyz="0.365 0 0.19" rpy="0 ${pi/12} 0"/>
   </joint>
   <!-- ===================== RPLIDAR S2 ===================== -->
