Commit message: feat(rover_description): match simulated lidar to real RPLIDAR S2 spec & use official RPLIDAR S2 STL

File: src/rover_description/urdf/lidar_sim.xacro (robot description, xacro)
@@ -1,22 +1,27 @@
 <?xml version="1.0"?>
 <robot xmlns:xacro="http://www.ros.org/wiki/xacro">
-  <!-- Simulated 2-D lidar for Gazebo (nav2 testing only). -->
+  <!--
+    Simulated RPLIDAR S2 (Gazebo, nav2 testing only).
+  -->
+  <material name="lidar_black">
+    <color rgba="0.05 0.05 0.05 1.0"/>
+  </material>
   <link name="laser_link">
     <inertial>
       <origin xyz="0 0 0" rpy="0 0 0"/>
-      <mass value="0.2"/>
+      <mass value="0.19"/>
       <inertia ixx="0.0001" iyy="0.0001" izz="0.0002" ixy="0" ixz="0" iyz="0"/>
     </inertial>
     <visual>
-      <origin xyz="0 0 0" rpy="0 0 0"/>
+      <origin xyz="0 0 -0.057" rpy="-1.5708 0 3.1416"/>
       <geometry>
-        <cylinder radius="0.05" length="0.04"/>
+        <mesh filename="package://rover_description/meshes/navigation/lidar/rplidar_s2.stl" scale="0.001 0.001 0.001"/>
       </geometry>
-      <material name="orange_mount"/>
+      <material name="lidar_black"/>
     </visual>
     <collision>
       <origin xyz="0 0 0" rpy="0 0 0"/>
       <geometry>
-        <cylinder radius="0.05" length="0.04"/>
+        <cylinder radius="0.0385" length="0.039"/>
       </geometry>
     </collision>
@@ -25,5 +30,5 @@
     <parent link="main_body_link"/>
     <child link="laser_link"/>
-    <origin xyz="0.2 0 0.12" rpy="0 0 0"/>
+    <origin xyz="0 0 0.17" rpy="0 0 0"/>
   </joint>
   <gazebo reference="laser_link">
@@ -42,6 +47,6 @@
         </scan>
         <range>
-          <min>0.12</min>
-          <max>10.0</max>
+          <min>0.05</min>
+          <max>18.0</max>
           <resolution>0.01</resolution>
         </range>

Commit message: refactore: only one of the dublicating sim xacro files kept, publishing of the scan topic in the simulation made conditional

File: src/rover_description/urdf/lidar_sim.xacro (robot description, xacro)
@@ -2,55 +2,62 @@
 <robot xmlns:xacro="http://www.ros.org/wiki/xacro">
   <!--
-    Simulated RPLIDAR S2 (Gazebo, nav2 testing only).
+    RPLIDAR S2 fragment as a macro. Call `lidar_sim simulate_scan="true|false"` to
+    include the simulated sensor (topic publishing). The visual/collision
+    geometry and joint are always added so the model is visible in the GUI.
   -->
-  <material name="lidar_black">
-    <color rgba="0.05 0.05 0.05 1.0"/>
-  </material>
-  <link name="laser_link">
-    <inertial>
-      <origin xyz="0 0 0" rpy="0 0 0"/>
-      <mass value="0.19"/>
-      <inertia ixx="0.0001" iyy="0.0001" izz="0.0002" ixy="0" ixz="0" iyz="0"/>
-    </inertial>
-    <visual>
-      <origin xyz="0 0 -0.057" rpy="-1.5708 0 3.1416"/>
-      <geometry>
-        <mesh filename="package://rover_description/meshes/navigation/lidar/rplidar_s2.stl" scale="0.001 0.001 0.001"/>
-      </geometry>
-      <material name="lidar_black"/>
-    </visual>
-    <collision>
-      <origin xyz="0 0 0" rpy="0 0 0"/>
-      <geometry>
-        <cylinder radius="0.0385" length="0.039"/>
-      </geometry>
-    </collision>
-  </link>
-  <joint name="laser_joint" type="fixed">
-    <parent link="main_body_link"/>
-    <child link="laser_link"/>
-    <origin xyz="0 0 0.17" rpy="0 0 0"/>
-  </joint>
-  <gazebo reference="laser_link">
-    <sensor type="gpu_lidar" name="generic_laser">
-      <update_rate>10.0</update_rate>
-      <topic>/scan</topic>
-      <gz_frame_id>laser_link</gz_frame_id>
-      <lidar>
-        <scan>
-          <horizontal>
-            <samples>360</samples>
-            <resolution>1</resolution>
-            <min_angle>-3.141592</min_angle>
-            <max_angle>3.141592</max_angle>
-          </horizontal>
-        </scan>
-        <range>
-          <min>0.05</min>
-          <max>18.0</max>
-          <resolution>0.01</resolution>
-        </range>
-      </lidar>
-    </sensor>
-  </gazebo>
+  <xacro:macro name="lidar_sim" params="simulate_scan:false">
+    <material name="lidar_black">
+      <color rgba="0.05 0.05 0.05 1.0"/>
+    </material>
+    <link name="laser_link">
+      <inertial>
+        <origin xyz="0 0 0" rpy="0 0 0"/>
+        <mass value="0.19"/>
+        <inertia ixx="0.0001" iyy="0.0001" izz="0.0002" ixy="0" ixz="0" iyz="0"/>
+      </inertial>
+      <visual>
+        <origin xyz="0 0 -0.057" rpy="-1.5708 0 3.1416"/>
+        <geometry>
+          <mesh filename="package://rover_description/meshes/navigation/lidar/rplidar_s2.stl" scale="0.001 0.001 0.001"/>
+        </geometry>
+        <material name="lidar_black"/>
+      </visual>
+      <collision>
+        <origin xyz="0 0 0" rpy="0 0 0"/>
+        <geometry>
+          <cylinder radius="0.0385" length="0.039"/>
+        </geometry>
+      </collision>
+    </link>
+    <joint name="laser_joint" type="fixed">
+      <parent link="main_body_link"/>
+      <child link="laser_link"/>
+      <origin xyz="0 0 0.17" rpy="0 0 0"/>
+    </joint>
+    <!-- Only include the Gazebo sensor block when simulation/publishing is desired -->
+    <xacro:if value="${simulate_scan}">
+      <gazebo reference="laser_link">
+        <sensor type="gpu_lidar" name="generic_laser">
+          <update_rate>10.0</update_rate>
+          <topic>/scan</topic>
+          <gz_frame_id>laser_link</gz_frame_id>
+          <lidar>
+            <scan>
+              <horizontal>
+                <samples>360</samples>
+                <resolution>1</resolution>
+                <min_angle>-3.141592</min_angle>
+                <max_angle>3.141592</max_angle>
+              </horizontal>
+            </scan>
+            <range>
+              <min>0.05</min>
+              <max>18.0</max>
+              <resolution>0.01</resolution>
+            </range>
+          </lidar>
+        </sensor>
+      </gazebo>
+    </xacro:if>
+  </xacro:macro>
 </robot>

File: src/rover_sim/urdf/rover_sim.urdf.xacro (robot description, xacro)
@@ -1,9 +1,10 @@
 <?xml version="1.0"?>
+<!-- Parameter defines whether to add simulation of the topics used by the navigational stack -->
+<xacro:arg name="use_nav" default="false"/>
 <robot name="indomitus_rover" xmlns:xacro="http://www.ros.org/wiki/xacro">
-  <!-- Main robot description -->
   <xacro:include filename="$(find rover_description)/urdf/rover.urdf.xacro"/>
-  <!-- Simulation ros2_control -->
   <xacro:include filename="$(find rover_description)/urdf/ros2_control_sim.xacro"/>
-  <!-- gz_ros2_control plugin -->
+  <xacro:include filename="$(find rover_description)/urdf/lidar_sim.xacro"/>
+  <xacro:lidar_sim simulate_scan="${use_nav}"/>
   <gazebo>
     <plugin filename="gz_ros2_control-system"
