Commit message: refactore: rover description refactored; stereo camera topic conditionaly added to simulation

File: src/rover_description/urdf/lidar.xacro (robot description, xacro)
@@ -2,9 +2,9 @@
 <robot xmlns:xacro="http://www.ros.org/wiki/xacro">
   <!--
-    RPLIDAR S2 fragment as a macro. Call `lidar_sim simulate_scan="true|false"` to
+    RPLIDAR S2 fragment as a macro. Call `lidar simulate_scan="true|false"` to
     include the simulated sensor (topic publishing). The visual/collision
     geometry and joint are always added so the model is visible in the GUI.
   -->
-  <xacro:macro name="lidar_sim" params="simulate_scan:false">
+  <xacro:macro name="lidar" params="use_sim:=false simulate_scan:=false">
     <material name="lidar_black">
       <color rgba="0.05 0.05 0.05 1.0"/>
@@ -35,6 +35,5 @@
       <origin xyz="0 0 0.17" rpy="0 0 0"/>
     </joint>
-    <!-- Only include the Gazebo sensor block when simulation/publishing is desired -->
-    <xacro:if value="${simulate_scan}">
+    <xacro:if value="${use_sim and simulate_scan}">
       <gazebo reference="laser_link">
         <sensor type="gpu_lidar" name="generic_laser">

File: src/rover_description/urdf/rover.urdf.xacro (robot description, xacro)
@@ -77,10 +77,10 @@
   </joint>
   <!-- ===================== ZED2i STEREO CAMERA ===================== -->
-  <xacro:include filename="$(find zed_description)/urdf/zed_macro.urdf.xacro" />
-  <xacro:zed_camera name="zed2i" model="zed2i">
-      <gnss_origin>
-          <origin xyz="0 0 0" rpy="0 0 0" />
-      </gnss_origin>
-  </xacro:zed_camera>
+  <xacro:include filename="$(find rover_description)/urdf/stereo_camera.xacro" />
+  <xacro:stereo_camera
+    use_sim="$(arg use_sim)"
+    simulate_rgb="$(arg stereo_camera_simulate_rgb)"
+    simulate_pointcloud="$(arg stereo_camera_simulate_pointcloud)"
+  />
   <joint name="zed2i_base_joint" type="fixed">
     <parent link="zed2i_camera_link"/>
@@ -88,4 +88,10 @@
     <origin xyz="-0.2915 0 -0.2644" rpy="0 ${-pi/12} 0"/>
   </joint>
+  <!-- ===================== RPLIDAR S2 ===================== -->
+  <xacro:include filename="$(find rover_description)/urdf/lidar.xacro" />
+  <xacro:lidar
+    use_sim="$(arg use_sim)"
+    simulate_scan="$(arg lidar_simulate_scan)"
+  />
   <!-- ===================== LEFT ROCKER ===================== -->
   <link name="l_rocker_link">

File: src/rover_description/urdf/rover.xacro (robot description, xacro)
@@ -1,7 +1,12 @@
 <?xml version="1.0"?>
 <robot name="indomitus_s1" xmlns:xacro="http://www.ros.org/wiki/xacro">
+<!-- Global / Top-Level Arguments -->
   <xacro:arg name="use_sim" default="false"/>
   <xacro:arg name="can_interface" default="can0"/>
   <xacro:arg name="controllers_yaml_path" default=""/>
+  <!-- Sensor Simulation Arguments -->
+  <xacro:arg name="lidar_simulate_scan" default="false"/>
+  <xacro:arg name="stereo_camera_simulate_rgb" default="false"/>
+  <xacro:arg name="stereo_camera_simulate_pointcloud" default="false"/>
   <!-- Main robot description -->
   <xacro:include filename="$(find rover_description)/urdf/rover.urdf.xacro"/>

Commit message: fix: stereo camera xacro fixed to use moder gazebo plugins; alwaays_on tag added to the lidar xacro

File: src/rover_description/urdf/lidar.xacro (robot description, xacro)
@@ -38,4 +38,5 @@
       <gazebo reference="laser_link">
         <sensor type="gpu_lidar" name="generic_laser">
+          <always_on>true</always_on>
           <update_rate>10.0</update_rate>
           <topic>/rplidar/scan</topic>

File: src/rover_description/urdf/stereo_camera.xacro (robot description, xacro)
@@ -1,15 +1,9 @@
 <?xml version="1.0"?>
 <robot xmlns:xacro="http://www.ros.org/wiki/xacro">
-  <!--
-    ZED 2i stereo camera fragment as a macro.
-    The visual/collision geometry and joint are always added.
-  -->
-  <xacro:macro
-    name="stereo_camera"
-    params="use_sim:=false
-            simulate_rgb:=false
-            simulate_pointcloud:=false
-            simulate_imu:=false"
-  >
+  <xacro:macro name="stereo_camera"
+               params="use_sim:=false
+                       simulate_rgb:=false
+                       simulate_pointcloud:=false
+                       simulate_imu:=false">
     <xacro:include filename="$(find zed_description)/urdf/zed_macro.urdf.xacro" />
     <xacro:zed_camera name="zed2i" model="zed2i">
@@ -18,11 +12,14 @@
       </gnss_origin>
     </xacro:zed_camera>
-    <!-- RGB CAMERA PLUGIN -->
+    <!-- RGB CAMERA -->
     <xacro:if value="${use_sim and simulate_rgb}">
       <gazebo reference="zed2i_left_camera_frame">
         <sensor type="camera" name="zed2i_rgb_sensor">
-          <update_rate>30.0</update_rate>
           <always_on>true</always_on>
-          <camera name="zed2i_rgb">
+          <update_rate>20.0</update_rate>
+          <topic>/zed2i/rgb/image_rect_color</topic>
+          <gz_frame_id>zed2i_left_camera_optical_frame</gz_frame_id>
+          <camera>
+            <camera_info_topic>/zed2i/rgb/camera_info</camera_info_topic>
             <horizontal_fov>1.91986</horizontal_fov>
             <image>
@@ -36,23 +33,17 @@
             </clip>
           </camera>
-          <plugin name="zed2i_rgb_plugin" filename="libgazebo_ros_camera.so">
-            <ros>
-              <namespace>zed2i</namespace>
-              <remapping>image_raw:=rgb/image_rect_color</remapping>
-              <remapping>camera_info:=rgb/camera_info</remapping>
-            </ros>
-            <camera_name>rgb</camera_name>
-            <frame_name>zed2i_left_camera_optical_frame</frame_name>
-          </plugin>
         </sensor>
       </gazebo>
     </xacro:if>
-    <!-- DEPTH & POINTCLOUD PLUGIN -->
+    <!-- DEPTH CAMERA -->
     <xacro:if value="${use_sim and simulate_pointcloud}">
       <gazebo reference="zed2i_left_camera_frame">
-        <sensor type="depth" name="zed2i_depth_sensor">
+        <sensor type="depth_camera" name="zed2i_depth_sensor">
+          <always_on>true</always_on>
           <update_rate>15.0</update_rate>
-          <always_on>true</always_on>
-          <camera name="zed2i_depth">
+          <topic>/zed2i/depth/depth_registered</topic>
+          <gz_frame_id>zed2i_left_camera_optical_frame</gz_frame_id>
+          <camera>
+            <camera_info_topic>/zed2i/depth/camera_info</camera_info_topic>
             <horizontal_fov>1.91986</horizontal_fov>
             <image>
@@ -66,21 +57,8 @@
             </clip>
           </camera>
-          <plugin name="zed2i_pointcloud_plugin" filename="libgazebo_ros_camera.so">
-            <ros>
-              <namespace>zed2i</namespace>
-              <remapping>points:=points</remapping>
-              <remapping>depth/image_raw:=depth/depth_registered</remapping>
-              <remapping>camera_info:=depth/camera_info</remapping>
-              <remapping>image_raw:=depth/image_rect_color</remapping>
-            </ros>
-            <camera_name>depth</camera_name>
-            <frame_name>zed2i_left_camera_optical_frame</frame_name>
-            <min_depth>0.01</min_depth>
-            <max_depth>15.0</max_depth>
-          </plugin>
         </sensor>
       </gazebo>
     </xacro:if>
-    <!-- IMU PLUGIN -->
+    <!-- IMU -->
     <xacro:if value="${use_sim and simulate_imu}">
       <gazebo reference="zed2i_left_camera_frame">
@@ -88,11 +66,6 @@
           <always_on>true</always_on>
           <update_rate>100.0</update_rate>
-          <plugin name="zed2i_imu_plugin" filename="libgazebo_ros_imu_sensor.so">
-            <ros>
-              <namespace>zed2i</namespace>
-              <remapping>~/out:=imu/data</remapping>
-            </ros>
-            <initial_orientation_as_reference>false</initial_orientation_as_reference>
-          </plugin>
+          <topic>/zed2i/imu/data</topic>
+          <gz_frame_id>zed2i_left_camera_frame</gz_frame_id>
         </sensor>
       </gazebo>

Commit message: chore: minor changes in the xacros of the rover, stereo camera and lidar

File: src/rover_description/urdf/lidar.xacro (robot description, xacro)
@@ -2,7 +2,8 @@
 <robot xmlns:xacro="http://www.ros.org/wiki/xacro">
   <!--
-    RPLIDAR S2 fragment as a macro. Call `lidar simulate_scan="true|false"` to
-    include the simulated sensor (topic publishing). The visual/collision
-    geometry and joint are always added so the model is visible in the GUI.
+    RPLIDAR S2 fragment as a macro.
+    Parameters: `use_sim`, `simulate_scan` (booleans).
+    Enables Gazebo GPU lidar plugin and topic publishing when set to true.
+    Defines the sensor link, visual, and collision geometries.
   -->
   <xacro:macro name="lidar" params="use_sim:=false simulate_scan:=false">
@@ -30,9 +31,4 @@
       </collision>
     </link>
-    <joint name="laser_joint" type="fixed">
-      <parent link="main_body_link"/>
-      <child link="laser_link"/>
-      <origin xyz="0 0 0.17" rpy="0 0 0"/>
-    </joint>
     <xacro:if value="${use_sim and simulate_scan}">
       <gazebo reference="laser_link">

File: src/rover_description/urdf/rover.urdf.xacro (robot description, xacro)
@@ -102,4 +102,9 @@
     simulate_scan="$(arg lidar_simulate_scan)"
   />
+  <joint name="laser_joint" type="fixed">
+    <parent link="main_body_link"/>
+    <child link="laser_link"/>
+    <origin xyz="0 0 0.17" rpy="0 0 0"/>
+  </joint>
   <!-- ===================== LEFT ROCKER ===================== -->
   <link name="l_rocker_link">

File: src/rover_description/urdf/stereo_camera.xacro (robot description, xacro)
@@ -1,4 +1,10 @@
 <?xml version="1.0"?>
 <robot xmlns:xacro="http://www.ros.org/wiki/xacro">
+  <!--
+    ZED2i Stereo Camera fragment as a macro.
+    Parameters: `use_sim`, `simulate_rgb`, `simulate_depth`, `simulate_imu` (booleans).
+    Enables Gazebo camera and IMU plugins and topic publishing when set to true.
+    Defines the sensor links, visual, and collision geometries.
+  -->
   <xacro:macro name="stereo_camera"
                params="use_sim:=false
