Commit message: Feature/navigation/nav core (#469)
* SLAM added.

* Nav2 added.

* EKF now fuses ZED 2i odometry (only in real launches) and wheel odometry.

* Launch file and config for the ZED 2i added.

* Launch file and config for the RPLIDAR S2 added.

* Launch file for Scan filter node to filter out rover from lidar scans added

* Dockerfile updated to include a separate hardware workspace, with improved caching.

* Docker Compose files unified.

* Simulation launch files and configs updated

File: src/rover_description/urdf/properties.xacro (robot description, xacro)
@@ -60,3 +60,14 @@
   <xacro:property name="wheel_kp" value="1000000.0"/>
   <xacro:property name="wheel_kd" value="1.0"/>
+  <!-- ===================== ZED2I POSSITION ===================== -->
+  <xacro:property name="zed2i_x" value="${body_length / 2.0 + 0.05}"/>
+  <xacro:property name="zed2i_y" value="0.0"/>
+  <xacro:property name="zed2i_z" value="${body_height / 2.0 + 0.05}"/>
+  <xacro:property name="zed2i_rx" value="0.0"/>
+  <xacro:property name="zed2i_ry" value="${pi/12}"/>
+  <xacro:property name="zed2i_rz" value="0.0"/>
+  <!-- ===================== LIDAR POSSITION ===================== -->
+  <xacro:property name="lidar_x" value="0.0"/>
+  <xacro:property name="lidar_y" value="0.0"/>
+  <xacro:property name="lidar_z" value="${body_height / 2.0 + 0.07}"/>
 </robot>

File: src/rover_description/urdf/rover.urdf.xacro (robot description, xacro)
@@ -5,5 +5,6 @@
   <xacro:include filename="$(find rover_description)/urdf/macros/rocker_assembly.xacro"/>
   <xacro:include filename="$(find rover_description)/urdf/macros/accessories.xacro"/>
-  <xacro:include filename="$(find rover_description)/urdf/camera.xacro"/>
+  <xacro:include filename="$(find rover_description)/urdf/macros/stereo_camera.xacro"/>
+  <xacro:include filename="$(find rover_description)/urdf/macros/lidar.xacro"/>
   <!-- mount_arm:=true bolts the indomitus_arm (arm_description) onto
        main_body_link, matching the real hardware where the arm is
@@ -38,4 +39,11 @@
     <color rgba="0.7 0.05 0.05 1"/>
   </material>
+  <!-- ===================== BASE FOOTPRINT ===================== -->
+  <link name="base_footprint"/>
+  <joint name="base_footprint_joint" type="fixed">
+    <parent link="base_footprint"/>
+    <child link="base_link"/>
+    <origin xyz="0 0 0.42" rpy="0 0 0"/>
+  </joint>
   <!-- ===================== BASE ===================== -->
   <link name="base_link">
@@ -97,6 +105,26 @@
     <origin xyz="0 0 0.02" rpy="0 0 0"/>
   </joint>
-  <!-- ===================== CAMERA ===================== -->
-  <xacro:camera/>
+  <!-- ===================== ZED2i STEREO CAMERA ===================== -->
+  <xacro:stereo_camera
+    use_sim="$(arg use_sim)"
+    simulate_rgb="$(arg stereo_camera_simulate_rgb)"
+    simulate_depth="$(arg stereo_camera_simulate_depth)"
+    simulate_imu="$(arg stereo_camera_simulate_imu)"
+  />
+  <joint name="zed2i_base_joint" type="fixed">
+    <parent link="main_body_link"/>
+    <child link="zed2i_camera_link"/>
+    <origin xyz="${zed2i_x} ${zed2i_y} ${zed2i_z}" rpy="${zed2i_rx} ${zed2i_ry} ${zed2i_rz}"/>
+  </joint>
+  <!-- ===================== RPLIDAR S2 ===================== -->
+  <xacro:lidar
+    use_sim="$(arg use_sim)"
+    simulate_scan="$(arg lidar_simulate_scan)"
+  />
+  <joint name="laser_joint" type="fixed">
+    <parent link="main_body_link"/>
+    <child link="laser_link"/>
+    <origin xyz="${lidar_x} ${lidar_y} ${lidar_z}" rpy="0 0 0"/>
+  </joint>
   <!-- ===================== ROCKERS + WHEELS ===================== -->
   <xacro:rocker_assembly side="l" y_sign="1"/>

File: src/rover_description/urdf/rover.xacro (robot description, xacro)
@@ -1,7 +1,13 @@
 <?xml version="1.0"?>
 <robot name="indomitus_s1" xmlns:xacro="http://www.ros.org/wiki/xacro">
+<!-- Global / Top-Level Arguments -->
   <xacro:arg name="use_sim" default="false"/>
   <xacro:arg name="can_interface" default="can0"/>
   <xacro:arg name="controllers_yaml_path" default=""/>
+  <!-- Sensor Simulation Arguments -->
+  <xacro:arg name="lidar_simulate_scan" default="false"/>
+  <xacro:arg name="stereo_camera_simulate_rgb" default="false"/>
+  <xacro:arg name="stereo_camera_simulate_depth" default="false"/>
+  <xacro:arg name="stereo_camera_simulate_imu" default="false"/>
   <!-- Main robot description -->
   <xacro:include filename="$(find rover_description)/urdf/rover.urdf.xacro"/>

Commit message: feat(rover_localization): add ekf_tilt_node for base_link tilt fusion, base_link_ground_ref frame

File: src/rover_description/urdf/properties.xacro (robot description, xacro)
@@ -49,4 +49,11 @@
   <!-- Mesh alignment: centers wheel.stl on the wheel link's own origin -->
   <xacro:property name="wheel_hub_offset" value="0.151"/>
+  <!-- ===================== BASE GROUND CLEARANCE ===================== -->
+  <!-- Height of base_link above ground level (base_footprint / base_link_ground_ref),
+       derived from the suspension/wheel stack-up at the nominal rest pose (rocker
+       angle = 0, steering angle = 0): rocker pivot -> wheel-mount hub (-rocker_hub_z),
+       wheel-mount hub -> axle (wheel_mount_drop), axle -> ground (wheel_radius).
+       If this value changes, change initial_state z seed in the rover_localization/config/ekf_tilt.yaml's-->
+  <xacro:property name="base_link_ground_height" value="${wheel_radius - rocker_hub_z + wheel_mount_drop}"/>
   <!-- ===================== JOINT LIMITS ===================== -->
   <xacro:property name="steering_limit" value="${3.0 * pi / 2.0}"/>  <!-- +/-270 deg -->

File: src/rover_description/urdf/rover.urdf.xacro (robot description, xacro)
@@ -7,14 +7,5 @@
   <xacro:include filename="$(find rover_description)/urdf/macros/stereo_camera.xacro"/>
   <xacro:include filename="$(find rover_description)/urdf/macros/lidar.xacro"/>
-  <!-- mount_arm:=true bolts the indomitus_arm (arm_description) onto
-       main_body_link, matching the real hardware where the arm is
-       physically attached to the rover chassis. Defaults to false so
-       existing rover-only bringup/sim behavior is unchanged unless a
-       launch file opts in. The include is unconditional (it only defines
-       the indomitus_arm macro; no links/joints are created until it is
-       invoked below), so arm_description must be present in the overlay
-       the same way it already is for arm_bringup/arm_hardware_interface. -->
   <xacro:include filename="$(find arm_description)/urdf/arm_macro.xacro"/>
-  <xacro:arg name="mount_arm" default="false"/>
   <!-- ===================== MATERIALS ===================== -->
   <material name="blue_body">
@@ -39,11 +30,4 @@
     <color rgba="0.7 0.05 0.05 1"/>
   </material>
-  <!-- ===================== BASE FOOTPRINT ===================== -->
-  <link name="base_footprint"/>
-  <joint name="base_footprint_joint" type="fixed">
-    <parent link="base_footprint"/>
-    <child link="base_link"/>
-    <origin xyz="0 0 0.42" rpy="0 0 0"/>
-  </joint>
   <!-- ===================== BASE ===================== -->
   <link name="base_link">
@@ -53,4 +37,10 @@
     </inertial>
   </link>
+  <link name="base_link_ground_ref"/>
+  <joint name="base_link_ground_ref_joint" type="fixed">
+    <parent link="base_link"/>
+    <child link="base_link_ground_ref"/>
+    <origin xyz="0 0 -${base_link_ground_height}" rpy="0 0 0"/>
+  </joint>
   <!-- ===================== SUSPENSION BASE AXII ===================== -->
   <link name="suspension_base_axii_link">

File: src/rover_description/urdf/rover.xacro (robot description, xacro)
@@ -9,5 +9,7 @@
   <xacro:arg name="stereo_camera_simulate_rgb" default="false"/>
   <xacro:arg name="stereo_camera_simulate_depth" default="false"/>
-  <xacro:arg name="stereo_camera_simulate_imu" default="false"/>
+  <xacro:arg name="stereo_camera_simulate_imu" default="true"/>
+  <!-- mount_arm:=true bolts the indomitus_arm onto main_body_link.-->
+  <xacro:arg name="mount_arm" default="false"/>
   <!-- Main robot description -->
   <xacro:include filename="$(find rover_description)/urdf/rover.urdf.xacro"/>

Commit message: fix: base_link_ground_ref frame removed, base_frame for the slope_layer changed to rover_footprint

File: src/rover_description/urdf/properties.xacro (robot description, xacro)
@@ -50,10 +50,12 @@
   <xacro:property name="wheel_hub_offset" value="0.151"/>
   <!-- ===================== BASE GROUND CLEARANCE ===================== -->
-  <!-- Height of base_link above ground level (base_footprint / base_link_ground_ref),
-       derived from the suspension/wheel stack-up at the nominal rest pose (rocker
-       angle = 0, steering angle = 0): rocker pivot -> wheel-mount hub (-rocker_hub_z),
+  <!-- Height of base_link above ground level (base_footprint), derived from the
+       suspension/wheel stack-up at the nominal rest pose (rocker angle = 0,
+       steering angle = 0): rocker pivot -> wheel-mount hub (-rocker_hub_z),
        wheel-mount hub -> axle (wheel_mount_drop), axle -> ground (wheel_radius).
-       If this value changes, update the `ground_height` parameter passed to
-       tilt_broadcaster_node in rover_localization/launch/ekf.launch.py to match. -->
+       Not consumed anywhere in this xacro tree; it's the source of truth for
+       the `ground_height` parameter passed to tilt_broadcaster_node in
+       rover_localization/launch/ekf.launch.py; update that parameter to match
+       if this value changes. -->
   <xacro:property name="base_link_ground_height" value="${wheel_radius - rocker_hub_z + wheel_mount_drop}"/>
   <!-- ===================== JOINT LIMITS ===================== -->

File: src/rover_description/urdf/rover.urdf.xacro (robot description, xacro)
@@ -37,10 +37,4 @@
     </inertial>
   </link>
-  <link name="base_link_ground_ref"/>
-  <joint name="base_link_ground_ref_joint" type="fixed">
-    <parent link="base_link"/>
-    <child link="base_link_ground_ref"/>
-    <origin xyz="0 0 -${base_link_ground_height}" rpy="0 0 0"/>
-  </joint>
   <!-- ===================== SUSPENSION BASE AXII ===================== -->
   <link name="suspension_base_axii_link">

Commit message: fix: wheel parameters updated for all controllers

File: src/rover_description/urdf/properties.xacro (robot description, xacro)
@@ -5,6 +5,6 @@
   <xacro:property name="M_PI_2" value="${pi / 2.0}"/>
   <!-- ===================== CHASSIS LAYOUT ===================== -->
-  <xacro:property name="wheelbase" value="0.842"/>     <!-- front-to-rear axle distance -->
-  <xacro:property name="track_width" value="0.682"/>   <!-- left-to-right rocker pivot distance -->
+  <xacro:property name="wheelbase" value="0.797"/>     <!-- front-to-rear axle distance -->
+  <xacro:property name="track_width" value="0.644"/>   <!-- left-to-right rocker pivot distance -->
   <!-- ===================== MAIN BODY ===================== -->
   <xacro:property name="body_length" value="0.603"/>   <!-- X -->
@@ -44,5 +44,5 @@
   <!-- ===================== WHEEL ===================== -->
   <!-- Geometry -->
-  <xacro:property name="wheel_radius" value="0.16"/>
+  <xacro:property name="wheel_radius" value="0.156"/>
   <xacro:property name="wheel_width" value="0.12"/>
   <xacro:property name="wheel_mass" value="0.5"/>

Commit message: chore: something removed

File: src/rover_description/urdf/properties.xacro (robot description, xacro)
@@ -70,14 +70,3 @@
   <xacro:property name="wheel_kp" value="1000000.0"/>
   <xacro:property name="wheel_kd" value="1.0"/>
-  <!-- ===================== ZED2I POSSITION ===================== -->
-  <xacro:property name="zed2i_x" value="${body_length / 2.0 + 0.05}"/>
-  <xacro:property name="zed2i_y" value="0.0"/>
-  <xacro:property name="zed2i_z" value="${body_height / 2.0 + 0.05}"/>
-  <xacro:property name="zed2i_rx" value="0.0"/>
-  <xacro:property name="zed2i_ry" value="${pi/12}"/>
-  <xacro:property name="zed2i_rz" value="0.0"/>
-  <!-- ===================== LIDAR POSSITION ===================== -->
-  <xacro:property name="lidar_x" value="0.0"/>
-  <xacro:property name="lidar_y" value="0.0"/>
-  <xacro:property name="lidar_z" value="${body_height / 2.0 + 0.07}"/>
 </robot>

File: src/rover_description/urdf/rover.urdf.xacro (robot description, xacro)
@@ -4,7 +4,4 @@
   <xacro:include filename="$(find rover_description)/urdf/macros/inertia_macros.xacro"/>
   <xacro:include filename="$(find rover_description)/urdf/macros/rocker_assembly.xacro"/>
-  <xacro:include filename="$(find rover_description)/urdf/macros/accessories.xacro"/>
-  <xacro:include filename="$(find rover_description)/urdf/macros/stereo_camera.xacro"/>
-  <xacro:include filename="$(find rover_description)/urdf/macros/lidar.xacro"/>
   <xacro:include filename="$(find arm_description)/urdf/arm_macro.xacro"/>
   <!-- ===================== MATERIALS ===================== -->
@@ -23,10 +20,4 @@
   <material name="red_axii">
     <color rgba="0.55 0.56 0.58 1"/>
-  </material>
-  <material name="beacon_light">
-    <color rgba="0.9 0.35 0.05 1"/>
-  </material>
-  <material name="button_red">
-    <color rgba="0.7 0.05 0.05 1"/>
   </material>
   <!-- ===================== BASE ===================== -->
@@ -89,34 +80,7 @@
     <origin xyz="0 0 0.02" rpy="0 0 0"/>
   </joint>
-  <!-- ===================== ZED2i STEREO CAMERA ===================== -->
-  <xacro:stereo_camera
-    use_sim="$(arg use_sim)"
-    simulate_rgb="$(arg stereo_camera_simulate_rgb)"
-    simulate_depth="$(arg stereo_camera_simulate_depth)"
-    simulate_imu="$(arg stereo_camera_simulate_imu)"
-  />
-  <joint name="zed2i_base_joint" type="fixed">
-    <parent link="main_body_link"/>
-    <child link="zed2i_camera_link"/>
-    <origin xyz="${zed2i_x} ${zed2i_y} ${zed2i_z}" rpy="${zed2i_rx} ${zed2i_ry} ${zed2i_rz}"/>
-  </joint>
-  <!-- ===================== RPLIDAR S2 ===================== -->
-  <xacro:lidar
-    use_sim="$(arg use_sim)"
-    simulate_scan="$(arg lidar_simulate_scan)"
-  />
-  <joint name="laser_joint" type="fixed">
-    <parent link="main_body_link"/>
-    <child link="laser_link"/>
-    <origin xyz="${lidar_x} ${lidar_y} ${lidar_z}" rpy="0 0 0"/>
-  </joint>
   <!-- ===================== ROCKERS + WHEELS ===================== -->
   <xacro:rocker_assembly side="l" y_sign="1"/>
   <xacro:rocker_assembly side="r" y_sign="-1"/>
-  <!-- ===================== ACCESSORIES ===================== -->
-  <xacro:towerlight_accessory suffix="l" y_sign="1"/>
-  <xacro:towerlight_accessory suffix="r" y_sign="-1"/>
-  <xacro:stop_button_accessory suffix="l" y_sign="1"/>
-  <xacro:stop_button_accessory suffix="r" y_sign="-1"/>
   <!-- ===================== ARM (OPTIONAL) ===================== -->
   <!-- Placeholder mount pose; update once the real MR_ARM_ATT attachment

File: src/rover_description/urdf/rover.xacro (robot description, xacro)
@@ -5,9 +5,4 @@
   <xacro:arg name="can_interface" default="can0"/>
   <xacro:arg name="controllers_yaml_path" default=""/>
-  <!-- Sensor Simulation Arguments -->
-  <xacro:arg name="lidar_simulate_scan" default="false"/>
-  <xacro:arg name="stereo_camera_simulate_rgb" default="false"/>
-  <xacro:arg name="stereo_camera_simulate_depth" default="false"/>
-  <xacro:arg name="stereo_camera_simulate_imu" default="true"/>
   <!-- mount_arm:=true bolts the indomitus_arm onto main_body_link.-->
   <xacro:arg name="mount_arm" default="false"/>
