Commit message: feat(arm): add camera_link, servo camera-frame control, keyboard teleop node

File: src/arm/arm_description/urdf/arm_macro.xacro (robot description, xacro)
@@ -124,4 +124,20 @@
     <!-- TCP (Tool Center Point) is a virtual point -->
     <link name="arm_tcp_link"/>
+    <!-- Camera mounted on wrist_2 -->
+    <joint name="arm_camera_joint" type="fixed">
+      <parent link="arm_wrist_2_link"/>
+      <child link="arm_camera_link"/>
+      <origin xyz="0.05 0 0" rpy="0 0 0"/>
+    </joint>
+    <link name="arm_camera_link">
+      <visual>
+        <geometry>
+          <box size="0.06 0.06 0.03"/>
+        </geometry>
+        <material name="camera_blue">
+          <color rgba="0.0 0.0 1.0 1.0"/>
+        </material>
+      </visual>
+    </link>
     <!-- ROS 2 Control Configuration -->
     <ros2_control name="ArmSystem" type="system">

Commit message: fix(arm): reposition camera_link

File: src/arm/arm_description/urdf/arm_macro.xacro (robot description, xacro)
@@ -128,5 +128,5 @@
       <parent link="arm_wrist_2_link"/>
       <child link="arm_camera_link"/>
-      <origin xyz="0.05 0 0" rpy="0 0 0"/>
+      <origin xyz="-0.13286 -0.01058 0.00685" rpy="0 ${pi/2} 0"/>
     </joint>
     <link name="arm_camera_link">

Commit message: feat(arm): update keyboard servo axes and camera orientation

File: src/arm/arm_description/urdf/arm_macro.xacro (robot description, xacro)
@@ -128,5 +128,5 @@
       <parent link="arm_wrist_2_link"/>
       <child link="arm_camera_link"/>
-      <origin xyz="-0.13286 -0.01058 0.00685" rpy="0 ${pi/2} 0"/>
+      <origin xyz="-0.13286 -0.01058 0.00685" rpy="0 ${-pi/2} 0"/>
     </joint>
     <link name="arm_camera_link">

Commit message: feature: added jaw gripper

File: src/arm/arm_description/urdf/arm_macro.xacro (robot description, xacro)
@@ -2,4 +2,5 @@
 <robot xmlns:xacro="http://www.ros.org/wiki/xacro">
   <xacro:arg name="use_fake_hardware" default="true"/>
+  <xacro:arg name="end_effector" default="jaw"/>
   <xacro:macro name="indomitus_arm" params="parent_link *origin">
     <xacro:property name="mesh_path" value="package://arm_description/meshes"/>
@@ -110,9 +111,19 @@
       <parent link="arm_wrist_2_link"/>
       <child link="arm_end_effector_link"/>
-      <origin xyz="0 0 0.05" rpy="0 0 0"/>
+      <origin xyz="-0.067825 0 0.0353" rpy="${-pi/2} 0 ${-pi/2}"/>
       <axis xyz="0 0 1"/>
       <limit lower="${-pi}" upper="${pi}" effort="100.0" velocity="1.0"/>
     </joint>
     <link name="arm_end_effector_link">
+      <xacro:if value="${'$(arg end_effector)' == 'jaw'}">
+        <visual>
+          <geometry><mesh filename="${mesh_path}/jaw_gripper.stl" scale="${stl_scale}"/></geometry>
+        </visual>
+        <collision>
+          <geometry><mesh filename="${mesh_path}/jaw_gripper.stl" scale="${stl_scale}"/></geometry>
+        </collision>
+      </xacro:if>
+      <xacro:if value="${'$(arg end_effector)' == 'other_tool'}">
+        </xacro:if>
       <xacro:dummy_inertia mass="0.2"/>
     </link>
@@ -120,7 +131,11 @@
       <parent link="arm_end_effector_link"/>
       <child link="arm_tcp_link"/>
-      <origin xyz="0 0 0.02" rpy="0 0 0"/>
+      <xacro:if value="${'$(arg end_effector)' == 'jaw'}">
+        <origin xyz="0 -0.23 0" rpy="0 0 0"/>
+      </xacro:if>
+      <xacro:if value="${'$(arg end_effector)' != 'jaw'}">
+        <origin xyz="0 -0.23 0" rpy="0 0 0"/>
+      </xacro:if>
     </joint>
-    <!-- TCP (Tool Center Point) is a virtual point -->
     <link name="arm_tcp_link"/>
     <!-- Camera mounted on wrist_2 -->

Commit message: feat(arm): command servo relative to gripper-mounted camera frame

File: src/arm/arm_description/urdf/arm_macro.xacro (robot description, xacro)
@@ -6,5 +6,4 @@
     <xacro:property name="mesh_path" value="package://arm_description/meshes"/>
     <xacro:property name="stl_scale" value="0.001 0.001 0.001"/>
-    <!-- Dummy macro for mass and inertia (required for physical simulations) -->
     <xacro:macro name="dummy_inertia" params="mass">
       <inertial>
@@ -125,5 +124,5 @@
       </xacro:if>
       <xacro:if value="${'$(arg end_effector)' == 'other_tool'}">
-        </xacro:if>
+      </xacro:if>
       <xacro:dummy_inertia mass="0.2"/>
     </link>
@@ -139,9 +138,8 @@
     </joint>
     <link name="arm_tcp_link"/>
-    <!-- Camera mounted on wrist_2 -->
     <joint name="arm_camera_joint" type="fixed">
-      <parent link="arm_wrist_2_link"/>
+      <parent link="arm_end_effector_link"/>
       <child link="arm_camera_link"/>
-      <origin xyz="-0.13286 -0.01058 0.00685" rpy="0 ${-pi/2} 0"/>
+      <origin xyz="-0.00110236 -0.0683370 -0.0340064" rpy="${pi} 0 ${-pi/2}"/>
     </joint>
     <link name="arm_camera_link">
@@ -154,6 +152,10 @@
         </material>
       </visual>
+      <collision>
+        <geometry>
+          <box size="0.06 0.06 0.03"/>
+        </geometry>
+      </collision>
     </link>
-    <!-- ROS 2 Control Configuration -->
     <ros2_control name="ArmSystem" type="system">
       <hardware>
@@ -162,5 +164,4 @@
         </xacro:if>
         <xacro:unless value="$(arg use_fake_hardware)">
-          <!-- TODO: replace with the real plugin name once arm_hardware_interface is implemented -->
           <plugin>arm_hardware_interface/ArmCanSystem</plugin>
           <param name="can_interface">can0</param>

Commit message: old testing

File: src/arm/arm_description/urdf/arm_macro.xacro (robot description, xacro)
@@ -46,5 +46,5 @@
       <parent link="arm_base_link"/>
       <child link="arm_shoulder_link"/>
-      <origin xyz="0 0.013 0.0945" rpy="0 0 ${-pi/2}"/>
+      <origin xyz="0 0.013 0.0945" rpy="${-pi/2} 0 ${-pi/2}"/>
       <axis xyz="1 0 0"/>
       <limit lower="${-pi/2}" upper="${pi}" effort="100.0" velocity="1.0"/>

Commit message: fix(arm): correct wrist end-effector joint axis and invert pitch direction

File: src/arm/arm_description/urdf/arm_macro.xacro (robot description, xacro)
@@ -111,5 +111,5 @@
       <child link="arm_end_effector_link"/>
       <origin xyz="-0.067825 0 0.0353" rpy="${-pi/2} 0 ${-pi/2}"/>
-      <axis xyz="0 0 1"/>
+      <axis xyz="0 1 0"/>
       <limit lower="${-pi}" upper="${pi}" effort="100.0" velocity="1.0"/>
     </joint>

Commit message: feat(arm): add camera_link, servo camera-frame control, keyboard tele… (#490)
* feat(arm): add camera_link, servo camera-frame control, keyboard teleop node

* feat(arm):add logging to keyboard servo node

* fix(arm): reposition camera_link

* fix(arm): correct axis orientation

* feat(arm): update keyboard servo axes and camera orientation

* feature: added jaw gripper

* refactor(arm): fix ROS parameters, relative topics, and servo shutdown

* feat(arm): command servo relative to gripper-mounted camera frame

* fix(arm): replace TTY auto-repeat with evdev press/release events

* fix(launch): start servo_node on arm_controller spawner exit event

* fix(arm): fix servo_node race condition and document servo readiness

* docs(arm): clean up trailing placeholder in servo status docstring

* fix(arm): comment out warehouse_ros_mongo dependency to fix CI build

* fix(arm): add missing exec_depends in arm_moveit_config and arm_tasks package.xml

* fix(arm): correct wrist end-effector joint axis and invert pitch direction

---------

Co-authored-by: Martik-k <kosiv.marta@gmail.com>

File: src/arm/arm_description/urdf/arm_macro.xacro (robot description, xacro)
@@ -2,8 +2,8 @@
 <robot xmlns:xacro="http://www.ros.org/wiki/xacro">
   <xacro:arg name="use_fake_hardware" default="true"/>
+  <xacro:arg name="end_effector" default="jaw"/>
   <xacro:macro name="indomitus_arm" params="parent_link *origin">
     <xacro:property name="mesh_path" value="package://arm_description/meshes"/>
     <xacro:property name="stl_scale" value="0.001 0.001 0.001"/>
-    <!-- Dummy macro for mass and inertia (required for physical simulations) -->
     <xacro:macro name="dummy_inertia" params="mass">
       <inertial>
@@ -110,9 +110,19 @@
       <parent link="arm_wrist_2_link"/>
       <child link="arm_end_effector_link"/>
-      <origin xyz="0 0 0.05" rpy="0 0 0"/>
-      <axis xyz="0 0 1"/>
+      <origin xyz="-0.067825 0 0.0353" rpy="${-pi/2} 0 ${-pi/2}"/>
+      <axis xyz="0 1 0"/>
       <limit lower="${-pi}" upper="${pi}" effort="100.0" velocity="1.0"/>
     </joint>
     <link name="arm_end_effector_link">
+      <xacro:if value="${'$(arg end_effector)' == 'jaw'}">
+        <visual>
+          <geometry><mesh filename="${mesh_path}/jaw_gripper.stl" scale="${stl_scale}"/></geometry>
+        </visual>
+        <collision>
+          <geometry><mesh filename="${mesh_path}/jaw_gripper.stl" scale="${stl_scale}"/></geometry>
+        </collision>
+      </xacro:if>
+      <xacro:if value="${'$(arg end_effector)' == 'other_tool'}">
+      </xacro:if>
       <xacro:dummy_inertia mass="0.2"/>
     </link>
@@ -120,9 +130,32 @@
       <parent link="arm_end_effector_link"/>
       <child link="arm_tcp_link"/>
-      <origin xyz="0 0 0.02" rpy="0 0 0"/>
+      <xacro:if value="${'$(arg end_effector)' == 'jaw'}">
+        <origin xyz="0 -0.23 0" rpy="0 0 0"/>
+      </xacro:if>
+      <xacro:if value="${'$(arg end_effector)' != 'jaw'}">
+        <origin xyz="0 -0.23 0" rpy="0 0 0"/>
+      </xacro:if>
     </joint>
-    <!-- TCP (Tool Center Point) is a virtual point -->
     <link name="arm_tcp_link"/>
-    <!-- ROS 2 Control Configuration -->
+    <joint name="arm_camera_joint" type="fixed">
+      <parent link="arm_end_effector_link"/>
+      <child link="arm_camera_link"/>
+      <origin xyz="-0.00110236 -0.0683370 -0.0340064" rpy="${pi} 0 ${-pi/2}"/>
+    </joint>
+    <link name="arm_camera_link">
+      <visual>
+        <geometry>
+          <box size="0.06 0.06 0.03"/>
+        </geometry>
+        <material name="camera_blue">
+          <color rgba="0.0 0.0 1.0 1.0"/>
+        </material>
+      </visual>
+      <collision>
+        <geometry>
+          <box size="0.06 0.06 0.03"/>
+        </geometry>
+      </collision>
+    </link>
     <ros2_control name="ArmSystem" type="system">
       <hardware>
@@ -131,5 +164,4 @@
         </xacro:if>
         <xacro:unless value="$(arg use_fake_hardware)">
-          <!-- TODO: replace with the real plugin name once arm_hardware_interface is implemented -->
           <plugin>arm_hardware_interface/ArmCanSystem</plugin>
           <param name="can_interface">can0</param>

Commit message: feature: synchronized 20-23 motors in visualization and in reality, made a safe launch of the launch file

File: src/arm/arm_description/urdf/arm_macro.xacro (robot description, xacro)
@@ -46,5 +46,5 @@
       <parent link="arm_base_link"/>
       <child link="arm_shoulder_link"/>
-      <origin xyz="0 0.013 0.0945" rpy="${-pi/2} 0 ${-pi/2}"/>
+      <origin xyz="0 0.013 0.0945" rpy="${-pi/3} 0 ${-pi/2}"/>
       <axis xyz="1 0 0"/>
       <limit lower="${-pi/2}" upper="${pi}" effort="100.0" velocity="1.0"/>
@@ -62,5 +62,5 @@
       <parent link="arm_shoulder_link"/>
       <child link="arm_forearm_link"/>
-      <origin xyz="-0.057 0 0.5" rpy="0 0 0"/>
+      <origin xyz="-0.057 0 0.5" rpy="${5*pi/6} 0 0"/>
       <axis xyz="1 0 0"/>
       <limit lower="${-pi/2}" upper="${pi/2}" effort="100.0" velocity="1.0"/>
@@ -131,10 +131,29 @@
         </xacro:if>
         <xacro:unless value="$(arg use_fake_hardware)">
-          <!-- TODO: replace with the real plugin name once arm_hardware_interface is implemented -->
           <plugin>arm_hardware_interface/ArmCanSystem</plugin>
           <param name="can_interface">can0</param>
+          <!-- Stiffness ramps 0 -> 100% over this many seconds after activation -->
+          <param name="gain_ramp_secs">6.0</param>
+          <!-- Hard rate limiter on outgoing position commands (rad/s).
+               Even a wrong/hostile command cannot move a joint faster than this.
+               Keep at 0.3 for the very first powered tests, raise later. -->
+          <param name="max_cmd_speed_rad_s">1.0</param>
+          <!-- Activation aborts if any motor is silent for this long -->
+          <param name="feedback_timeout_secs">2.0</param>
         </xacro:unless>
       </hardware>
-      <xacro:macro name="arm_joint_control" params="joint_name">
+      <!-- ======================= CALIBRATION =======================
+           direction : +1 if pushing the joint in its URDF-positive direction
+                       (right-hand rule about the <axis>) makes the RAW motor
+                       angle increase; -1 otherwise.
+           offset    : the RAW motor angle (rad) measured when the arm is
+                       physically in the URDF zero pose. If you save the motor
+                       zero (0xB1 / FF..FE) at that pose, offset = 0.0.
+           kp / kd   : MIT gains — starting values are the proven ones from
+                       play_arm_waypoints.py. Halve kp for first powered tests.
+           Determine direction & offset with scripts/check_calibration.py
+           (torqueless) — see CALIBRATION_GUIDE.md.
+           ============================================================= -->
+      <xacro:macro name="arm_joint_control" params="joint_name motor_id direction offset kp kd">
         <joint name="${joint_name}">
           <command_interface name="position">
@@ -142,14 +161,21 @@
             <param name="max">${pi}</param>
           </command_interface>
-          <command_interface name="velocity"/> <state_interface name="position"/>
+          <command_interface name="velocity"/>
+          <state_interface name="position"/>
           <state_interface name="velocity"/>
+          <param name="motor_id">${motor_id}</param>
+          <param name="direction">${direction}</param>
+          <param name="offset">${offset}</param>
+          <param name="kp">${kp}</param>
+          <param name="kd">${kd}</param>
         </joint>
       </xacro:macro>
-      <xacro:arm_joint_control joint_name="arm_mount_base_joint"/>
-      <xacro:arm_joint_control joint_name="arm_base_shoulder_joint"/>
-      <xacro:arm_joint_control joint_name="arm_shoulder_forearm_joint"/>
-      <xacro:arm_joint_control joint_name="arm_forearm_wrist_1_joint"/>
-      <xacro:arm_joint_control joint_name="arm_wrist_1_wrist_2_joint"/>
-      <xacro:arm_joint_control joint_name="arm_wrist_2_end_effector_joint"/>
+      <!-- TODO: replace direction/offset with YOUR measured calibration values -->
+      <xacro:arm_joint_control joint_name="arm_mount_base_joint"          motor_id="20" direction="-1" offset="1.9746" kp="15.0" kd="1.5"/>
+      <xacro:arm_joint_control joint_name="arm_base_shoulder_joint"       motor_id="21" direction="-1" offset="1.7093" kp="100.0" kd="3.5"/>
+      <xacro:arm_joint_control joint_name="arm_shoulder_forearm_joint"    motor_id="22" direction="1"  offset="-0.7155" kp="50.0" kd="2.0"/>
+      <xacro:arm_joint_control joint_name="arm_forearm_wrist_1_joint"     motor_id="23" direction="-1" offset="1.0378" kp="10.0" kd="1.0"/>
+      <xacro:arm_joint_control joint_name="arm_wrist_1_wrist_2_joint"     motor_id="24" direction="1"  offset="0.0" kp="30.0"  kd="1.0"/>
+      <xacro:arm_joint_control joint_name="arm_wrist_2_end_effector_joint" motor_id="25" direction="1" offset="0.0" kp="15.0"  kd="0.5"/>
     </ros2_control>
   </xacro:macro>

Commit message: feat(arm): update camera orientation and set gazebo visual colors

File: src/arm/arm_description/urdf/arm_macro.xacro (robot description, xacro)
@@ -7,4 +7,7 @@
     <xacro:property name="mesh_path" value="package://arm_description/meshes"/>
     <xacro:property name="stl_scale" value="0.001 0.001 0.001"/>
+    <material name="light_grey">
+      <color rgba="0.7 0.7 0.7 1.0"/>
+    </material>
     <xacro:macro name="dummy_inertia" params="mass">
       <inertial>
@@ -22,4 +25,5 @@
       <visual>
         <geometry><mesh filename="${mesh_path}/arm_mount.stl" scale="${stl_scale}"/></geometry>
+        <material name="light_grey"/>
       </visual>
       <collision>
@@ -38,4 +42,5 @@
       <visual>
         <geometry><mesh filename="${mesh_path}/arm_base.stl" scale="${stl_scale}"/></geometry>
+        <material name="light_grey"/>
       </visual>
       <collision>
@@ -54,4 +59,5 @@
       <visual>
         <geometry><mesh filename="${mesh_path}/arm_shoulder.stl" scale="${stl_scale}"/></geometry>
+        <material name="light_grey"/>
       </visual>
       <collision>
@@ -70,4 +76,5 @@
       <visual>
         <geometry><mesh filename="${mesh_path}/arm_forearm.stl" scale="${stl_scale}"/></geometry>
+        <material name="light_grey"/>
       </visual>
       <collision>
@@ -86,4 +93,5 @@
       <visual>
         <geometry><mesh filename="${mesh_path}/arm_wrist_1.stl" scale="${stl_scale}"/></geometry>
+        <material name="light_grey"/>
       </visual>
       <collision>
@@ -102,4 +110,5 @@
       <visual>
         <geometry><mesh filename="${mesh_path}/arm_wrist_2.stl" scale="${stl_scale}"/></geometry>
+        <material name="light_grey"/>
       </visual>
       <collision>
@@ -119,4 +128,5 @@
         <visual>
           <geometry><mesh filename="${mesh_path}/jaw_gripper.stl" scale="${stl_scale}"/></geometry>
+          <material name="light_grey"/>
         </visual>
         <collision>
@@ -197,7 +207,70 @@
         </plugin>
       </gazebo>
+      <gazebo reference="arm_mount_link">
+        <visual>
+          <material>
+            <ambient>0.7 0.7 0.7 1.0</ambient>
+            <diffuse>0.7 0.7 0.7 1.0</diffuse>
+            <specular>0.3 0.3 0.3 1.0</specular>
+          </material>
+        </visual>
+      </gazebo>
+      <gazebo reference="arm_base_link">
+        <visual>
+          <material>
+            <ambient>0.7 0.7 0.7 1.0</ambient>
+            <diffuse>0.7 0.7 0.7 1.0</diffuse>
+            <specular>0.3 0.3 0.3 1.0</specular>
+          </material>
+        </visual>
+      </gazebo>
+      <gazebo reference="arm_shoulder_link">
+        <visual>
+          <material>
+            <ambient>0.7 0.7 0.7 1.0</ambient>
+            <diffuse>0.7 0.7 0.7 1.0</diffuse>
+            <specular>0.3 0.3 0.3 1.0</specular>
+          </material>
+        </visual>
+      </gazebo>
+      <gazebo reference="arm_forearm_link">
+        <visual>
+          <material>
+            <ambient>0.7 0.7 0.7 1.0</ambient>
+            <diffuse>0.7 0.7 0.7 1.0</diffuse>
+            <specular>0.3 0.3 0.3 1.0</specular>
+          </material>
+        </visual>
+      </gazebo>
+      <gazebo reference="arm_wrist_1_link">
+        <visual>
+          <material>
+            <ambient>0.7 0.7 0.7 1.0</ambient>
+            <diffuse>0.7 0.7 0.7 1.0</diffuse>
+            <specular>0.3 0.3 0.3 1.0</specular>
+          </material>
+        </visual>
+      </gazebo>
+      <gazebo reference="arm_wrist_2_link">
+        <visual>
+          <material>
+            <ambient>0.7 0.7 0.7 1.0</ambient>
+            <diffuse>0.7 0.7 0.7 1.0</diffuse>
+            <specular>0.3 0.3 0.3 1.0</specular>
+          </material>
+        </visual>
+      </gazebo>
+      <gazebo reference="arm_end_effector_link">
+        <visual>
+          <material>
+            <ambient>0.7 0.7 0.7 1.0</ambient>
+            <diffuse>0.7 0.7 0.7 1.0</diffuse>
+            <specular>0.3 0.3 0.3 1.0</specular>
+          </material>
+        </visual>
+      </gazebo>
       <gazebo reference="arm_camera_link">
         <sensor name="arm_camera" type="camera">
-          <pose>0 0 0 0 0 0</pose>
+          <pose>0 0 0.03 0 0 0</pose>
           <camera>
             <horizontal_fov>1.047</horizontal_fov>

Commit message: fix(arm): add camera optical frame and fix camera_info bridge topic

File: src/arm/arm_description/urdf/arm_macro.xacro (robot description, xacro)
@@ -169,4 +169,10 @@
       </collision>
     </link>
+    <joint name="arm_camera_optical_joint" type="fixed">
+      <parent link="arm_camera_link"/>
+      <child link="arm_camera_optical_frame"/>
+      <origin xyz="0 0 0.03" rpy="${-pi/2} 0 ${-pi/2}"/>
+    </joint>
+    <link name="arm_camera_optical_frame"/>
     <ros2_control name="ArmSystem" type="system">
       <hardware>
@@ -274,4 +280,5 @@
           <pose>0 0 0.03 0 0 0</pose>
           <camera>
+            <optical_frame_id>arm_camera_optical_frame</optical_frame_id>
             <horizontal_fov>1.047</horizontal_fov>
             <image>

File: src/arm/arm_description/urdf/arm_macro_simple.xacro (robot description, xacro)
@@ -4,7 +4,4 @@
   <xacro:arg name="end_effector" default="jaw"/>
   <xacro:arg name="sim" default="false"/>
-  <!-- camera:=false drops the simulated camera sensor (the URDF link and
-       frames stay). Camera rendering is the main real-time-factor cost
-       when the GPU isn't doing the rendering. -->
   <xacro:arg name="camera" default="true"/>
   <xacro:macro name="indomitus_arm" params="parent_link *origin">
@@ -19,9 +16,4 @@
       </inertial>
     </xacro:macro>
-    <!-- Visual + collision as a primitive placed to span the link's extent
-         between its joint frames. Primitives instead of the CAD meshes keep
-         rendering cheap (the STLs were ~500k triangles, which software
-         rendering of the simulated camera could not sustain); joints,
-         masses and inertias fully define the physics and are unaffected. -->
     <xacro:macro name="box_geometry" params="size xyz">
       <visual>
@@ -156,4 +148,10 @@
       </collision>
     </link>
+    <joint name="arm_camera_optical_joint" type="fixed">
+      <parent link="arm_camera_link"/>
+      <child link="arm_camera_optical_frame"/>
+      <origin xyz="0 0 0.03" rpy="${-pi/2} 0 ${-pi/2}"/>
+    </joint>
+    <link name="arm_camera_optical_frame"/>
     <ros2_control name="ArmSystem" type="system">
       <hardware>
@@ -262,4 +260,5 @@
           <pose>0 0 0.03 0 0 0</pose>
           <camera>
+            <optical_frame_id>arm_camera_optical_frame</optical_frame_id>
             <horizontal_fov>1.047</horizontal_fov>
             <image>
