Commit message: Feature/arm/gazebo moveit camera sim (#501)
* feat(arm): integrate Gazebo sim, ros2_control and MoveIt for arm

* feat(arm): update camera orientation and set gazebo visual colors

* feat(arm): integrate servo teleop with Gazebo sim time

* feat(arm): add combined Gazebo+RViz launch and raise teleop speeds

* feat(arm): add primitive-geometry arm variant and use it in Gazebo sim

* chore(arm): strip explanatory comments from sim launch files

* fix(arm): verify safe-pose result with timeout, restore hw teleop speeds with sim override, clock-only bridge when camera off

* fix(arm): shut down sim launch on spawn/controller failure, declare missing arm_sim runtime deps

* fix(arm): add camera optical frame and fix camera_info bridge topic

* fix(sim): adjust spawn height for arm_mount mesh origin

* docs(arm): document sim teleop invocation in node and params file

* fix(arm): safe-pose servo gating, camera arg fix, drop unused geometry variant

---------

Co-authored-by: Martik-k <kosiv.marta@gmail.com>

File: src/arm/arm_description/urdf/arm_macro.xacro (robot description, xacro)
@@ -3,7 +3,15 @@
   <xacro:arg name="use_fake_hardware" default="true"/>
   <xacro:arg name="end_effector" default="jaw"/>
+  <xacro:arg name="sim" default="false"/>
+  <!-- camera:=false drops the simulated camera sensor (the URDF link and
+       frames stay). Camera rendering is the main real-time-factor cost
+       when the GPU isn't doing the rendering. -->
+  <xacro:arg name="camera" default="true"/>
   <xacro:macro name="indomitus_arm" params="parent_link *origin">
     <xacro:property name="mesh_path" value="package://arm_description/meshes"/>
     <xacro:property name="stl_scale" value="0.001 0.001 0.001"/>
+    <material name="light_grey">
+      <color rgba="0.7 0.7 0.7 1.0"/>
+    </material>
     <xacro:macro name="dummy_inertia" params="mass">
       <inertial>
@@ -21,4 +29,5 @@
       <visual>
         <geometry><mesh filename="${mesh_path}/arm_mount.stl" scale="${stl_scale}"/></geometry>
+        <material name="light_grey"/>
       </visual>
       <collision>
@@ -37,4 +46,5 @@
       <visual>
         <geometry><mesh filename="${mesh_path}/arm_base.stl" scale="${stl_scale}"/></geometry>
+        <material name="light_grey"/>
       </visual>
       <collision>
@@ -53,4 +63,5 @@
       <visual>
         <geometry><mesh filename="${mesh_path}/arm_shoulder.stl" scale="${stl_scale}"/></geometry>
+        <material name="light_grey"/>
       </visual>
       <collision>
@@ -69,4 +80,5 @@
       <visual>
         <geometry><mesh filename="${mesh_path}/arm_forearm.stl" scale="${stl_scale}"/></geometry>
+        <material name="light_grey"/>
       </visual>
       <collision>
@@ -85,4 +97,5 @@
       <visual>
         <geometry><mesh filename="${mesh_path}/arm_wrist_1.stl" scale="${stl_scale}"/></geometry>
+        <material name="light_grey"/>
       </visual>
       <collision>
@@ -101,4 +114,5 @@
       <visual>
         <geometry><mesh filename="${mesh_path}/arm_wrist_2.stl" scale="${stl_scale}"/></geometry>
+        <material name="light_grey"/>
       </visual>
       <collision>
@@ -118,4 +132,5 @@
         <visual>
           <geometry><mesh filename="${mesh_path}/jaw_gripper.stl" scale="${stl_scale}"/></geometry>
+          <material name="light_grey"/>
         </visual>
         <collision>
@@ -158,12 +173,23 @@
       </collision>
     </link>
+    <joint name="arm_camera_optical_joint" type="fixed">
+      <parent link="arm_camera_link"/>
+      <child link="arm_camera_optical_frame"/>
+      <origin xyz="0 0 0.03" rpy="${-pi/2} 0 ${-pi/2}"/>
+    </joint>
+    <link name="arm_camera_optical_frame"/>
     <ros2_control name="ArmSystem" type="system">
       <hardware>
-        <xacro:if value="$(arg use_fake_hardware)">
-          <plugin>mock_components/GenericSystem</plugin>
+        <xacro:if value="$(arg sim)">
+          <plugin>gz_ros2_control/GazeboSimSystem</plugin>
         </xacro:if>
-        <xacro:unless value="$(arg use_fake_hardware)">
-          <plugin>arm_hardware_interface/ArmCanSystem</plugin>
-          <param name="can_interface">can0</param>
+        <xacro:unless value="$(arg sim)">
+          <xacro:if value="$(arg use_fake_hardware)">
+            <plugin>mock_components/GenericSystem</plugin>
+          </xacro:if>
+          <xacro:unless value="$(arg use_fake_hardware)">
+            <plugin>arm_hardware_interface/ArmCanSystem</plugin>
+            <param name="can_interface">can0</param>
+          </xacro:unless>
         </xacro:unless>
       </hardware>
@@ -185,4 +211,98 @@
       <xacro:arm_joint_control joint_name="arm_wrist_2_end_effector_joint"/>
     </ros2_control>
+    <xacro:if value="$(arg sim)">
+      <gazebo>
+        <plugin filename="gz_ros2_control-system" name="gz_ros2_control::GazeboSimROS2ControlPlugin">
+          <parameters>$(find arm_sim)/config/ros2_controllers.yaml</parameters>
+        </plugin>
+      </gazebo>
+      <gazebo reference="arm_mount_link">
+        <visual>
+          <material>
+            <ambient>0.7 0.7 0.7 1.0</ambient>
+            <diffuse>0.7 0.7 0.7 1.0</diffuse>
+            <specular>0.3 0.3 0.3 1.0</specular>
+          </material>
+        </visual>
+      </gazebo>
+      <gazebo reference="arm_base_link">
+        <visual>
+          <material>
+            <ambient>0.7 0.7 0.7 1.0</ambient>
+            <diffuse>0.7 0.7 0.7 1.0</diffuse>
+            <specular>0.3 0.3 0.3 1.0</specular>
+          </material>
+        </visual>
+      </gazebo>
+      <gazebo reference="arm_shoulder_link">
+        <visual>
+          <material>
+            <ambient>0.7 0.7 0.7 1.0</ambient>
+            <diffuse>0.7 0.7 0.7 1.0</diffuse>
+            <specular>0.3 0.3 0.3 1.0</specular>
+          </material>
+        </visual>
+      </gazebo>
+      <gazebo reference="arm_forearm_link">
+        <visual>
+          <material>
+            <ambient>0.7 0.7 0.7 1.0</ambient>
+            <diffuse>0.7 0.7 0.7 1.0</diffuse>
+            <specular>0.3 0.3 0.3 1.0</specular>
+          </material>
+        </visual>
+      </gazebo>
+      <gazebo reference="arm_wrist_1_link">
+        <visual>
+          <material>
+            <ambient>0.7 0.7 0.7 1.0</ambient>
+            <diffuse>0.7 0.7 0.7 1.0</diffuse>
+            <specular>0.3 0.3 0.3 1.0</specular>
+          </material>
+        </visual>
+      </gazebo>
+      <gazebo reference="arm_wrist_2_link">
+        <visual>
+          <material>
+            <ambient>0.7 0.7 0.7 1.0</ambient>
+            <diffuse>0.7 0.7 0.7 1.0</diffuse>
+            <specular>0.3 0.3 0.3 1.0</specular>
+          </material>
+        </visual>
+      </gazebo>
+      <gazebo reference="arm_end_effector_link">
+        <visual>
+          <material>
+            <ambient>0.7 0.7 0.7 1.0</ambient>
+            <diffuse>0.7 0.7 0.7 1.0</diffuse>
+            <specular>0.3 0.3 0.3 1.0</specular>
+          </material>
+        </visual>
+      </gazebo>
+      <xacro:if value="$(arg camera)">
+      <gazebo reference="arm_camera_link">
+        <sensor name="arm_camera" type="camera">
+          <pose>0 0 0.03 0 0 0</pose>
+          <camera>
+            <optical_frame_id>arm_camera_optical_frame</optical_frame_id>
+            <horizontal_fov>1.047</horizontal_fov>
+            <image>
+              <width>640</width>
+              <height>480</height>
+              <format>R8G8B8</format>
+            </image>
+            <clip>
+              <near>0.05</near>
+              <far>15</far>
+            </clip>
+          </camera>
+          <always_on>1</always_on>
+          <update_rate>30</update_rate>
+          <visualize>true</visualize>
+          <topic>arm_camera/image_raw</topic>
+        </sensor>
+      </gazebo>
+      </xacro:if>
+    </xacro:if>
   </xacro:macro>
 </robot>

Commit message: feat(panel): switch panel description, bringup and sim packages

File: src/arm/arm_description/urdf/arm_macro.xacro (robot description, xacro)
@@ -4,4 +4,12 @@
   <xacro:arg name="end_effector" default="jaw"/>
   <xacro:arg name="sim" default="false"/>
+  <!-- When the arm is mounted into another robot's URDF (e.g. the rover, see
+       rover_description's mount_arm arg) that outer URDF already adds its
+       own single gz_ros2_control-system plugin covering every <ros2_control>
+       block in the combined model. Set this to false in that case so the
+       arm doesn't register a second, redundant controller_manager plugin
+       for the same Gazebo model. Standalone arm sim (arm_sim) leaves this
+       at the default so it keeps adding its own plugin as before. -->
+  <xacro:arg name="standalone_gz_plugin" default="true"/>
   <!-- camera:=false drops the simulated camera sensor (the URDF link and
        frames stay). Camera rendering is the main real-time-factor cost
@@ -212,9 +220,11 @@
     </ros2_control>
     <xacro:if value="$(arg sim)">
-      <gazebo>
-        <plugin filename="gz_ros2_control-system" name="gz_ros2_control::GazeboSimROS2ControlPlugin">
-          <parameters>$(find arm_sim)/config/ros2_controllers.yaml</parameters>
-        </plugin>
-      </gazebo>
+      <xacro:if value="$(arg standalone_gz_plugin)">
+        <gazebo>
+          <plugin filename="gz_ros2_control-system" name="gz_ros2_control::GazeboSimROS2ControlPlugin">
+            <parameters>$(find arm_sim)/config/ros2_controllers.yaml</parameters>
+          </plugin>
+        </gazebo>
+      </xacro:if>
       <gazebo reference="arm_mount_link">
         <visual>

File: src/rover_description/urdf/rover.urdf.xacro (robot description, xacro)
@@ -1,4 +1,14 @@
 <?xml version="1.0"?>
 <robot name="indomitus_s1" xmlns:xacro="http://www.ros.org/wiki/xacro">
+  <!-- mount_arm:=true bolts the indomitus_arm (arm_description) onto
+       main_body_link, matching the real hardware where the arm is
+       physically attached to the rover chassis. Defaults to false so
+       existing rover-only bringup/sim behavior is unchanged unless a
+       launch file opts in. The include is unconditional (it only defines
+       the indomitus_arm macro; no links/joints are created until it is
+       invoked below), so arm_description must be present in the overlay
+       the same way it already is for arm_bringup/arm_hardware_interface. -->
+  <xacro:include filename="$(find arm_description)/urdf/arm_macro.xacro"/>
+  <xacro:arg name="mount_arm" default="false"/>
   <!-- ===================== MATERIALS ===================== -->
   <material name="blue_body">
@@ -365,3 +375,11 @@
     <limit effort="100" velocity="10"/>
   </joint>
+  <!-- ===================== ARM (OPTIONAL) ===================== -->
+  <!-- Placeholder mount pose; update once the real MR_ARM_ATT attachment
+       point from CAD is known. -->
+  <xacro:if value="$(arg mount_arm)">
+    <xacro:indomitus_arm parent_link="main_body_link">
+      <origin xyz="0.2 0 0.1" rpy="0 0 0"/>
+    </xacro:indomitus_arm>
+  </xacro:if>
 </robot>

Commit message: feat: replace arm meshes

File: src/arm/arm_description/urdf/arm_macro.xacro (robot description, xacro)
@@ -28,9 +28,9 @@
     <link name="arm_mount_link">
       <visual>
-        <geometry><mesh filename="${mesh_path}/arm_mount.stl" scale="${stl_scale}"/></geometry>
-        <material name="light_grey"/>
-      </visual>
-      <collision>
-        <geometry><mesh filename="${mesh_path}/arm_mount.stl" scale="${stl_scale}"/></geometry>
+        <geometry><mesh filename="${mesh_path}/arm_mount_v2.stl" scale="${stl_scale}"/></geometry>
+        <material name="light_grey"/>
+      </visual>
+      <collision>
+        <geometry><mesh filename="${mesh_path}/arm_mount_v2.stl" scale="${stl_scale}"/></geometry>
       </collision>
       <xacro:dummy_inertia mass="1.0"/>
@@ -39,5 +39,5 @@
       <parent link="arm_mount_link"/>
       <child link="arm_base_link"/>
-      <origin xyz="0 0 0.018" rpy="0 0 0"/>
+      <origin xyz="0.06 0 0.021" rpy="0 0 0"/>
       <axis xyz="0 0 1"/>
       <limit lower="${-pi}" upper="${pi}" effort="100.0" velocity="1.0"/>
@@ -45,9 +45,9 @@
     <link name="arm_base_link">
       <visual>
-        <geometry><mesh filename="${mesh_path}/arm_base.stl" scale="${stl_scale}"/></geometry>
-        <material name="light_grey"/>
-      </visual>
-      <collision>
-        <geometry><mesh filename="${mesh_path}/arm_base.stl" scale="${stl_scale}"/></geometry>
+        <geometry><mesh filename="${mesh_path}/arm_base_v2.stl" scale="${stl_scale}"/></geometry>
+        <material name="light_grey"/>
+      </visual>
+      <collision>
+        <geometry><mesh filename="${mesh_path}/arm_base_v2.stl" scale="${stl_scale}"/></geometry>
       </collision>
       <xacro:dummy_inertia mass="2.0"/>
@@ -56,15 +56,15 @@
       <parent link="arm_base_link"/>
       <child link="arm_shoulder_link"/>
-      <origin xyz="0 0.013 0.0945" rpy="0 0 ${-pi/2}"/>
+      <origin xyz="-0.040366 -0.000325 0.103" rpy="${pi/6} 0 ${-pi}"/>
       <axis xyz="1 0 0"/>
-      <limit lower="${-pi/2}" upper="${pi}" effort="100.0" velocity="1.0"/>
+      <limit lower="${-pi}" upper="${pi}" effort="100.0" velocity="1.0"/>
     </joint>
     <link name="arm_shoulder_link">
       <visual>
-        <geometry><mesh filename="${mesh_path}/arm_shoulder.stl" scale="${stl_scale}"/></geometry>
-        <material name="light_grey"/>
-      </visual>
-      <collision>
-        <geometry><mesh filename="${mesh_path}/arm_shoulder.stl" scale="${stl_scale}"/></geometry>
+        <geometry><mesh filename="${mesh_path}/arm_shoulder_v2.stl" scale="${stl_scale}"/></geometry>
+        <material name="light_grey"/>
+      </visual>
+      <collision>
+        <geometry><mesh filename="${mesh_path}/arm_shoulder_v2.stl" scale="${stl_scale}"/></geometry>
       </collision>
       <xacro:dummy_inertia mass="1.5"/>
@@ -73,5 +73,5 @@
       <parent link="arm_shoulder_link"/>
       <child link="arm_forearm_link"/>
-      <origin xyz="-0.057 0 0.5" rpy="0 0 0"/>
+      <origin xyz="0 0.3 0" rpy="${5*pi/6} 0 0"/>
       <axis xyz="1 0 0"/>
       <limit lower="${-pi/2}" upper="${pi/2}" effort="100.0" velocity="1.0"/>
@@ -79,9 +79,9 @@
     <link name="arm_forearm_link">
       <visual>
-        <geometry><mesh filename="${mesh_path}/arm_forearm.stl" scale="${stl_scale}"/></geometry>
-        <material name="light_grey"/>
-      </visual>
-      <collision>
-        <geometry><mesh filename="${mesh_path}/arm_forearm.stl" scale="${stl_scale}"/></geometry>
+        <geometry><mesh filename="${mesh_path}/arm_forearm_v2.stl" scale="${stl_scale}"/></geometry>
+        <material name="light_grey"/>
+      </visual>
+      <collision>
+        <geometry><mesh filename="${mesh_path}/arm_forearm_v2.stl" scale="${stl_scale}"/></geometry>
       </collision>
       <xacro:dummy_inertia mass="1.0"/>
@@ -90,15 +90,15 @@
       <parent link="arm_forearm_link"/>
       <child link="arm_wrist_1_link"/>
-      <origin xyz="0.002175 0 0.4" rpy="${pi} ${pi} 0"/>
-      <axis xyz="1 0 0"/>
+      <origin xyz="-0.0173 0.3 0" rpy="0 ${pi/2} 0"/>
+      <axis xyz="0 0 1"/>
       <limit lower="${-pi/2}" upper="${pi/2}" effort="100.0" velocity="1.0"/>
     </joint>
     <link name="arm_wrist_1_link">
       <visual>
-        <geometry><mesh filename="${mesh_path}/arm_wrist_1.stl" scale="${stl_scale}"/></geometry>
-        <material name="light_grey"/>
-      </visual>
-      <collision>
-        <geometry><mesh filename="${mesh_path}/arm_wrist_1.stl" scale="${stl_scale}"/></geometry>
+        <geometry><mesh filename="${mesh_path}/arm_wrist_v2.stl" scale="${stl_scale}"/></geometry>
+        <material name="light_grey"/>
+      </visual>
+      <collision>
+        <geometry><mesh filename="${mesh_path}/arm_wrist_v2.stl" scale="${stl_scale}"/></geometry>
       </collision>
       <xacro:dummy_inertia mass="0.5"/>
@@ -107,15 +107,15 @@
       <parent link="arm_wrist_1_link"/>
       <child link="arm_wrist_2_link"/>
-      <origin xyz="-0.067825 0 0.0353" rpy="0 ${pi/2} 0"/>
-      <axis xyz="1 0 0"/>
+      <origin xyz="0.0323 0 -0.035" rpy="${-pi/2} 0 ${pi/2}"/>
+      <axis xyz="0 0 1"/>
       <limit lower="${-pi}" upper="${pi}" effort="100.0" velocity="1.0"/>
     </joint>
     <link name="arm_wrist_2_link">
       <visual>
-        <geometry><mesh filename="${mesh_path}/arm_wrist_2.stl" scale="${stl_scale}"/></geometry>
-        <material name="light_grey"/>
-      </visual>
-      <collision>
-        <geometry><mesh filename="${mesh_path}/arm_wrist_2.stl" scale="${stl_scale}"/></geometry>
+        <geometry><mesh filename="${mesh_path}/arm_wrist_v2.stl" scale="${stl_scale}"/></geometry>
+        <material name="light_grey"/>
+      </visual>
+      <collision>
+        <geometry><mesh filename="${mesh_path}/arm_wrist_v2.stl" scale="${stl_scale}"/></geometry>
       </collision>
       <xacro:dummy_inertia mass="0.3"/>
@@ -124,6 +124,6 @@
       <parent link="arm_wrist_2_link"/>
       <child link="arm_end_effector_link"/>
-      <origin xyz="-0.067825 0 0.0353" rpy="${-pi/2} 0 ${-pi/2}"/>
-      <axis xyz="0 1 0"/>
+      <origin xyz="0.0323 0 -0.035" rpy="${-pi/2} 0 ${-pi/2}"/>
+      <axis xyz="0 0 1"/>
       <limit lower="${-pi}" upper="${pi}" effort="100.0" velocity="1.0"/>
     </joint>
@@ -131,9 +131,9 @@
       <xacro:if value="${'$(arg end_effector)' == 'jaw'}">
         <visual>
-          <geometry><mesh filename="${mesh_path}/jaw_gripper.stl" scale="${stl_scale}"/></geometry>
+          <geometry><mesh filename="${mesh_path}/arm_jaw_gripper_v2.stl" scale="${stl_scale}"/></geometry>
           <material name="light_grey"/>
         </visual>
         <collision>
-          <geometry><mesh filename="${mesh_path}/jaw_gripper.stl" scale="${stl_scale}"/></geometry>
+          <geometry><mesh filename="${mesh_path}/arm_jaw_gripper_v2.stl" scale="${stl_scale}"/></geometry>
         </collision>
       </xacro:if>
@@ -142,4 +142,42 @@
       <xacro:dummy_inertia mass="0.2"/>
     </link>
+    <xacro:if value="${'$(arg end_effector)' == 'jaw'}">
+      <!-- From CAD, origin of each finger relative to gripper origin (mm):
+           finger 1 (right): closed (3.5, -10.72, 122.133)  -> open (15.5, -10.72, 122.133)
+           finger 2 (left):  closed (-3.5, 13.78, 122.133)  -> open (-15.5, 13.78, 122.133)
+           X is symmetric (+-3.5mm closed, +-12mm stroke); Y is NOT mirrored between the two
+           fingers on purpose (offset so the finger pads clear each other near full close). -->
+      <xacro:property name="finger_x_closed" value="-0.0035"/>
+      <xacro:property name="finger_stroke" value="0.012"/>
+      <xacro:property name="finger_z" value="0.122133"/>
+      <xacro:property name="finger_right_y" value="0.01072"/>
+      <xacro:property name="finger_left_y" value="-0.01378"/>
+      <xacro:macro name="jaw_gripper_finger" params="side x_closed y yaw axis_sign">
+        <joint name="arm_jaw_gripper_finger_${side}_joint" type="prismatic">
+          <parent link="arm_end_effector_link"/>
+          <child link="arm_jaw_gripper_finger_${side}_link"/>
+          <origin xyz="${x_closed} ${y} ${finger_z}" rpy="0 0 ${yaw}"/>
+          <axis xyz="${axis_sign} 0 0"/>
+          <limit lower="0" upper="${finger_stroke}" effort="20.0" velocity="0.05"/>
+          <xacro:unless value="${side == 'right'}">
+            <mimic joint="arm_jaw_gripper_finger_right_joint" multiplier="-1.0" offset="0.0"/>
+          </xacro:unless>
+        </joint>
+        <link name="arm_jaw_gripper_finger_${side}_link">
+          <visual>
+            <geometry><mesh filename="${mesh_path}/arm_jaw_gripper_finger_v2.stl" scale="${stl_scale}"/></geometry>
+            <material name="light_grey"/>
+          </visual>
+          <collision>
+            <geometry><mesh filename="${mesh_path}/arm_jaw_gripper_finger_v2.stl" scale="${stl_scale}"/></geometry>
+          </collision>
+          <xacro:dummy_inertia mass="0.05"/>
+        </link>
+      </xacro:macro>
+      <!-- Same part mounted twice: "left" is the "right" finger rotated 180 deg about Z,
+           so both slide outward along their own local +X (axis) to open — no mirrored mesh needed. -->
+      <xacro:jaw_gripper_finger side="right" x_closed="${finger_x_closed}"  y="${finger_right_y}" yaw="0"      axis_sign="-1"/>
+      <xacro:jaw_gripper_finger side="left"  x_closed="${-finger_x_closed}" y="${finger_left_y}"  yaw="${pi}" axis_sign="1"/>
+    </xacro:if>
     <joint name="arm_tcp_joint" type="fixed">
       <parent link="arm_end_effector_link"/>
@@ -280,4 +318,24 @@
         </visual>
       </gazebo>
+      <xacro:if value="${'$(arg end_effector)' == 'jaw'}">
+        <gazebo reference="arm_jaw_gripper_finger_right_link">
+          <visual>
+            <material>
+              <ambient>0.7 0.7 0.7 1.0</ambient>
+              <diffuse>0.7 0.7 0.7 1.0</diffuse>
+              <specular>0.3 0.3 0.3 1.0</specular>
+            </material>
+          </visual>
+        </gazebo>
+        <gazebo reference="arm_jaw_gripper_finger_left_link">
+          <visual>
+            <material>
+              <ambient>0.7 0.7 0.7 1.0</ambient>
+              <diffuse>0.7 0.7 0.7 1.0</diffuse>
+              <specular>0.3 0.3 0.3 1.0</specular>
+            </material>
+          </visual>
+        </gazebo>
+      </xacro:if>
       <xacro:if value="$(arg camera)">
       <gazebo reference="arm_camera_link">
