Commit message: fix(arm): unblock Servo motion and fix camera/roll behavior

File: src/arm/arm_description/urdf/arm_macro.xacro (robot description, xacro)
@@ -194,5 +194,5 @@
       <parent link="arm_end_effector_link"/>
       <child link="arm_camera_link"/>
-      <origin xyz="-0.00110236 -0.0683370 -0.0340064" rpy="${pi} 0 ${-pi/2}"/>
+      <origin xyz="0.0012919902801513672 0.07102805376052856 0.03884565830230713" rpy="0 ${-pi/2} ${-pi/2}"/>
     </joint>
     <link name="arm_camera_link">
@@ -248,4 +248,23 @@
       <xacro:arm_joint_control joint_name="arm_wrist_1_wrist_2_joint"/>
       <xacro:arm_joint_control joint_name="arm_wrist_2_end_effector_joint"/>
+      <!-- Only the right finger joint needs a ros2_control interface: the
+           left one is a <mimic> of it, computed automatically (by
+           robot_state_publisher for TF, and by the planning scene monitor
+           for collision state) from the right joint's reported position —
+           it doesn't need its own state/command interface. Without this,
+           joint_state_broadcaster never reports arm_jaw_gripper_finger_right_joint
+           at all, and the planning scene monitor (used by both move_group
+           and Servo) considers the robot's state permanently incomplete,
+           which silently blocks all motion. -->
+      <xacro:if value="${'$(arg end_effector)' == 'jaw'}">
+        <joint name="arm_jaw_gripper_finger_right_joint">
+          <command_interface name="position">
+            <param name="min">0</param>
+            <param name="max">${finger_stroke}</param>
+          </command_interface>
+          <state_interface name="position"/>
+          <state_interface name="velocity"/>
+        </joint>
+      </xacro:if>
     </ros2_control>
     <xacro:if value="$(arg sim)">

Commit message: fix(arm): flip gripper 180°, reposition camera, fix camera self-view

File: src/arm/arm_description/urdf/arm_macro.xacro (robot description, xacro)
@@ -124,5 +124,5 @@
       <parent link="arm_wrist_2_link"/>
       <child link="arm_end_effector_link"/>
-      <origin xyz="0.0323 0 -0.035" rpy="${-pi/2} 0 ${-pi/2}"/>
+      <origin xyz="0.0323 0 -0.035" rpy="${pi/2} 0 ${pi/2}"/>
       <axis xyz="0 0 1"/>
       <limit lower="${-pi}" upper="${pi}" effort="100.0" velocity="1.0"/>
@@ -194,10 +194,10 @@
       <parent link="arm_end_effector_link"/>
       <child link="arm_camera_link"/>
-      <origin xyz="0.0012919902801513672 0.07102805376052856 0.03884565830230713" rpy="0 ${-pi/2} ${-pi/2}"/>
+      <origin xyz="0.0012604892253875732 -0.045 0.07839690148830414" rpy="0 ${-pi/2} ${pi/2}"/>
     </joint>
     <link name="arm_camera_link">
       <visual>
         <geometry>
-          <box size="0.06 0.06 0.03"/>
+          <box size="0.06 0.06 0.06"/>
         </geometry>
         <material name="camera_blue">
@@ -207,5 +207,5 @@
       <collision>
         <geometry>
-          <box size="0.06 0.06 0.03"/>
+          <box size="0.06 0.06 0.06"/>
         </geometry>
       </collision>
@@ -214,5 +214,5 @@
       <parent link="arm_camera_link"/>
       <child link="arm_camera_optical_frame"/>
-      <origin xyz="0 0 0.03" rpy="${-pi/2} 0 ${-pi/2}"/>
+      <origin xyz="0 0 0" rpy="${-pi/2} 0 ${-pi/2}"/>
     </joint>
     <link name="arm_camera_optical_frame"/>
@@ -360,5 +360,5 @@
       <gazebo reference="arm_camera_link">
         <sensor name="arm_camera" type="camera">
-          <pose>0 0 0.03 0 0 0</pose>
+          <pose>0.045 0 0 0 0 0</pose>
           <camera>
             <optical_frame_id>arm_camera_optical_frame</optical_frame_id>

Commit message: fix(arm): fix gripper mimic limits and camera optical-frame TF

File: src/arm/arm_description/urdf/arm_macro.xacro (robot description, xacro)
@@ -153,5 +153,5 @@
       <xacro:property name="finger_right_y" value="0.01072"/>
       <xacro:property name="finger_left_y" value="-0.01378"/>
-      <xacro:macro name="jaw_gripper_finger" params="side x_closed y yaw axis_sign">
+      <xacro:macro name="jaw_gripper_finger" params="side x_closed y yaw axis_sign limit_lower limit_upper">
         <joint name="arm_jaw_gripper_finger_${side}_joint" type="prismatic">
           <parent link="arm_end_effector_link"/>
@@ -159,6 +159,13 @@
           <origin xyz="${x_closed} ${y} ${finger_z}" rpy="0 0 ${yaw}"/>
           <axis xyz="${axis_sign} 0 0"/>
-          <limit lower="0" upper="${finger_stroke}" effort="20.0" velocity="0.05"/>
+          <limit lower="${limit_lower}" upper="${limit_upper}" effort="20.0" velocity="0.05"/>
           <xacro:unless value="${side == 'right'}">
+            <!-- Right and left are mirror images (180 deg about Z), so their axes
+                 point opposite ways in the parent frame — multiplier=-1.0 makes
+                 them slide apart symmetrically as the right joint opens, rather
+                 than translating together with a fixed gap. Left's own range is
+                 shifted negative to match, since its opening motion is the
+                 mirror of right's (mimic must stay within the child's own
+                 declared limits). -->
             <mimic joint="arm_jaw_gripper_finger_right_joint" multiplier="-1.0" offset="0.0"/>
           </xacro:unless>
@@ -177,6 +184,6 @@
       <!-- Same part mounted twice: "left" is the "right" finger rotated 180 deg about Z,
            so both slide outward along their own local +X (axis) to open — no mirrored mesh needed. -->
-      <xacro:jaw_gripper_finger side="right" x_closed="${finger_x_closed}"  y="${finger_right_y}" yaw="0"      axis_sign="-1"/>
-      <xacro:jaw_gripper_finger side="left"  x_closed="${-finger_x_closed}" y="${finger_left_y}"  yaw="${pi}" axis_sign="1"/>
+      <xacro:jaw_gripper_finger side="right" x_closed="${finger_x_closed}"  y="${finger_right_y}" yaw="0"      axis_sign="-1" limit_lower="0"                limit_upper="${finger_stroke}"/>
+      <xacro:jaw_gripper_finger side="left"  x_closed="${-finger_x_closed}" y="${finger_left_y}"  yaw="${pi}" axis_sign="1"  limit_lower="${-finger_stroke}" limit_upper="0"/>
     </xacro:if>
     <joint name="arm_tcp_joint" type="fixed">
@@ -214,5 +221,9 @@
       <parent link="arm_camera_link"/>
       <child link="arm_camera_optical_frame"/>
-      <origin xyz="0 0 0" rpy="${-pi/2} 0 ${-pi/2}"/>
+      <!-- Matches the Gazebo <sensor>'s own <pose> offset below (both push the
+           optical center 0.045m forward along arm_camera_link's local X, past
+           the placeholder box's front face) so the published TF and the
+           actual render origin agree. -->
+      <origin xyz="0.045 0 0" rpy="${-pi/2} 0 ${-pi/2}"/>
     </joint>
     <link name="arm_camera_optical_frame"/>

Commit message: fix(arm): estimate TCP offset from v2 gripper mesh geometry

File: src/arm/arm_description/urdf/arm_macro.xacro (robot description, xacro)
@@ -191,5 +191,5 @@
       <child link="arm_tcp_link"/>
       <xacro:if value="${'$(arg end_effector)' == 'jaw'}">
-        <origin xyz="0 -0.23 0" rpy="0 0 0"/>
+        <origin xyz="0 -0.0015 0.2072" rpy="0 0 0"/>
       </xacro:if>
       <xacro:if value="${'$(arg end_effector)' != 'jaw'}">
@@ -221,8 +221,4 @@
       <parent link="arm_camera_link"/>
       <child link="arm_camera_optical_frame"/>
-      <!-- Matches the Gazebo <sensor>'s own <pose> offset below (both push the
-           optical center 0.045m forward along arm_camera_link's local X, past
-           the placeholder box's front face) so the published TF and the
-           actual render origin agree. -->
       <origin xyz="0.045 0 0" rpy="${-pi/2} 0 ${-pi/2}"/>
     </joint>
