Commit message: feat(arm): adopt new mesh set — geometry, jaw gripper, camera

File: src/arm/arm_description/urdf/arm_macro.xacro (robot description, xacro)
@@ -2,8 +2,16 @@
 <robot xmlns:xacro="http://www.ros.org/wiki/xacro">
   <xacro:arg name="use_fake_hardware" default="true"/>
+  <xacro:arg name="end_effector" default="jaw"/>
+  <xacro:arg name="sim" default="false"/>
+  <!-- camera:=false drops the simulated camera sensor (the URDF link and
+       frames stay). Camera rendering is the main real-time-factor cost
+       when the GPU isn't doing the rendering. -->
+  <xacro:arg name="camera" default="true"/>
   <xacro:macro name="indomitus_arm" params="parent_link *origin">
     <xacro:property name="mesh_path" value="package://arm_description/meshes"/>
     <xacro:property name="stl_scale" value="0.001 0.001 0.001"/>
-    <!-- Dummy macro for mass and inertia (required for physical simulations) -->
+    <material name="light_grey">
+      <color rgba="0.7 0.7 0.7 1.0"/>
+    </material>
     <xacro:macro name="dummy_inertia" params="mass">
       <inertial>
@@ -20,8 +28,9 @@
     <link name="arm_mount_link">
       <visual>
-        <geometry><mesh filename="${mesh_path}/arm_mount.stl" scale="${stl_scale}"/></geometry>
-      </visual>
-      <collision>
-        <geometry><mesh filename="${mesh_path}/arm_mount.stl" scale="${stl_scale}"/></geometry>
+        <geometry><mesh filename="${mesh_path}/arm_mount_v2.stl" scale="${stl_scale}"/></geometry>
+        <material name="light_grey"/>
+      </visual>
+      <collision>
+        <geometry><mesh filename="${mesh_path}/arm_mount_v2.stl" scale="${stl_scale}"/></geometry>
       </collision>
       <xacro:dummy_inertia mass="1.0"/>
@@ -30,5 +39,5 @@
       <parent link="arm_mount_link"/>
       <child link="arm_base_link"/>
-      <origin xyz="0 0 0.018" rpy="0 0 0"/>
+      <origin xyz="0.06 0 0.021" rpy="0 0 0"/>
       <axis xyz="0 0 1"/>
       <limit lower="${-pi}" upper="${pi}" effort="100.0" velocity="1.0"/>
@@ -36,8 +45,9 @@
     <link name="arm_base_link">
       <visual>
-        <geometry><mesh filename="${mesh_path}/arm_base.stl" scale="${stl_scale}"/></geometry>
-      </visual>
-      <collision>
-        <geometry><mesh filename="${mesh_path}/arm_base.stl" scale="${stl_scale}"/></geometry>
+        <geometry><mesh filename="${mesh_path}/arm_base_v2.stl" scale="${stl_scale}"/></geometry>
+        <material name="light_grey"/>
+      </visual>
+      <collision>
+        <geometry><mesh filename="${mesh_path}/arm_base_v2.stl" scale="${stl_scale}"/></geometry>
       </collision>
       <xacro:dummy_inertia mass="2.0"/>
@@ -46,14 +56,15 @@
       <parent link="arm_base_link"/>
       <child link="arm_shoulder_link"/>
-      <origin xyz="0 0.013 0.0945" rpy="${-pi/3} 0 ${-pi/2}"/>
+      <origin xyz="-0.040366 -0.000325 0.103" rpy="${pi/3} 0 ${-pi}"/>
       <axis xyz="1 0 0"/>
-      <limit lower="${-pi/2}" upper="${pi}" effort="100.0" velocity="1.0"/>
+      <limit lower="${-pi}" upper="${pi}" effort="100.0" velocity="1.0"/>
     </joint>
     <link name="arm_shoulder_link">
       <visual>
-        <geometry><mesh filename="${mesh_path}/arm_shoulder.stl" scale="${stl_scale}"/></geometry>
-      </visual>
-      <collision>
-        <geometry><mesh filename="${mesh_path}/arm_shoulder.stl" scale="${stl_scale}"/></geometry>
+        <geometry><mesh filename="${mesh_path}/arm_shoulder_v2.stl" scale="${stl_scale}"/></geometry>
+        <material name="light_grey"/>
+      </visual>
+      <collision>
+        <geometry><mesh filename="${mesh_path}/arm_shoulder_v2.stl" scale="${stl_scale}"/></geometry>
       </collision>
       <xacro:dummy_inertia mass="1.5"/>
@@ -62,5 +73,5 @@
       <parent link="arm_shoulder_link"/>
       <child link="arm_forearm_link"/>
-      <origin xyz="-0.057 0 0.5" rpy="${5*pi/6} 0 0"/>
+      <origin xyz="0 0.3 0" rpy="${5*pi/12} 0 0"/>
       <axis xyz="1 0 0"/>
       <limit lower="${-pi/2}" upper="${pi/2}" effort="100.0" velocity="1.0"/>
@@ -68,8 +79,9 @@
     <link name="arm_forearm_link">
       <visual>
-        <geometry><mesh filename="${mesh_path}/arm_forearm.stl" scale="${stl_scale}"/></geometry>
-      </visual>
-      <collision>
-        <geometry><mesh filename="${mesh_path}/arm_forearm.stl" scale="${stl_scale}"/></geometry>
+        <geometry><mesh filename="${mesh_path}/arm_forearm_v2.stl" scale="${stl_scale}"/></geometry>
+        <material name="light_grey"/>
+      </visual>
+      <collision>
+        <geometry><mesh filename="${mesh_path}/arm_forearm_v2.stl" scale="${stl_scale}"/></geometry>
       </collision>
       <xacro:dummy_inertia mass="1.0"/>
@@ -78,14 +90,15 @@
       <parent link="arm_forearm_link"/>
       <child link="arm_wrist_1_link"/>
-      <origin xyz="0.002175 0 0.4" rpy="${pi} ${pi} 0"/>
-      <axis xyz="1 0 0"/>
+      <origin xyz="-0.0173 0.3 0" rpy="0 ${pi/2} 0"/>
+      <axis xyz="0 0 1"/>
       <limit lower="${-pi/2}" upper="${pi/2}" effort="100.0" velocity="1.0"/>
     </joint>
     <link name="arm_wrist_1_link">
       <visual>
-        <geometry><mesh filename="${mesh_path}/arm_wrist_1.stl" scale="${stl_scale}"/></geometry>
-      </visual>
-      <collision>
-        <geometry><mesh filename="${mesh_path}/arm_wrist_1.stl" scale="${stl_scale}"/></geometry>
+        <geometry><mesh filename="${mesh_path}/arm_wrist_v2.stl" scale="${stl_scale}"/></geometry>
+        <material name="light_grey"/>
+      </visual>
+      <collision>
+        <geometry><mesh filename="${mesh_path}/arm_wrist_v2.stl" scale="${stl_scale}"/></geometry>
       </collision>
       <xacro:dummy_inertia mass="0.5"/>
@@ -94,14 +107,15 @@
       <parent link="arm_wrist_1_link"/>
       <child link="arm_wrist_2_link"/>
-      <origin xyz="-0.067825 0 0.0353" rpy="0 ${pi/2} 0"/>
-      <axis xyz="1 0 0"/>
+      <origin xyz="0.0323 0 -0.035" rpy="${-pi/2} 0 ${pi/2}"/>
+      <axis xyz="0 0 1"/>
       <limit lower="${-pi}" upper="${pi}" effort="100.0" velocity="1.0"/>
     </joint>
     <link name="arm_wrist_2_link">
       <visual>
-        <geometry><mesh filename="${mesh_path}/arm_wrist_2.stl" scale="${stl_scale}"/></geometry>
-      </visual>
-      <collision>
-        <geometry><mesh filename="${mesh_path}/arm_wrist_2.stl" scale="${stl_scale}"/></geometry>
+        <geometry><mesh filename="${mesh_path}/arm_wrist_v2.stl" scale="${stl_scale}"/></geometry>
+        <material name="light_grey"/>
+      </visual>
+      <collision>
+        <geometry><mesh filename="${mesh_path}/arm_wrist_v2.stl" scale="${stl_scale}"/></geometry>
       </collision>
       <xacro:dummy_inertia mass="0.3"/>
@@ -110,50 +124,113 @@
       <parent link="arm_wrist_2_link"/>
       <child link="arm_end_effector_link"/>
-      <origin xyz="0 0 0.05" rpy="0 0 0"/>
+      <origin xyz="0.0323 0 -0.035" rpy="${-pi/2} ${pi/2} ${-pi/2}"/>
       <axis xyz="0 0 1"/>
       <limit lower="${-pi}" upper="${pi}" effort="100.0" velocity="1.0"/>
     </joint>
     <link name="arm_end_effector_link">
+      <xacro:if value="${'$(arg end_effector)' == 'jaw'}">
+        <visual>
+          <geometry><mesh filename="${mesh_path}/arm_jaw_gripper_v2.stl" scale="${stl_scale}"/></geometry>
+          <material name="light_grey"/>
+        </visual>
+        <collision>
+          <geometry><mesh filename="${mesh_path}/arm_jaw_gripper_v2.stl" scale="${stl_scale}"/></geometry>
+        </collision>
+      </xacro:if>
+      <xacro:if value="${'$(arg end_effector)' == 'other_tool'}">
+      </xacro:if>
       <xacro:dummy_inertia mass="0.2"/>
     </link>
+    <xacro:if value="${'$(arg end_effector)' == 'jaw'}">
+      <!-- From CAD, origin of each finger relative to gripper origin (mm):
+           finger 1 (right): closed (3.5, -10.72, 122.133)  -> open (15.5, -10.72, 122.133)
+           finger 2 (left):  closed (-3.5, 13.78, 122.133)  -> open (-15.5, 13.78, 122.133)
+           X is symmetric (+-3.5mm closed, +-12mm stroke); Y is NOT mirrored between the two
+           fingers on purpose (offset so the finger pads clear each other near full close). -->
+      <xacro:property name="finger_x_closed" value="-0.0035"/>
+      <xacro:property name="finger_stroke" value="0.012"/>
+      <xacro:property name="finger_z" value="0.122133"/>
+      <xacro:property name="finger_right_y" value="0.01072"/>
+      <xacro:property name="finger_left_y" value="-0.01378"/>
+      <xacro:macro name="jaw_gripper_finger" params="side x_closed y yaw axis_sign">
+        <joint name="arm_jaw_gripper_finger_${side}_joint" type="prismatic">
+          <parent link="arm_end_effector_link"/>
+          <child link="arm_jaw_gripper_finger_${side}_link"/>
+          <origin xyz="${x_closed} ${y} ${finger_z}" rpy="0 0 ${yaw}"/>
+          <axis xyz="${axis_sign} 0 0"/>
+          <limit lower="0" upper="${finger_stroke}" effort="20.0" velocity="0.05"/>
+          <xacro:unless value="${side == 'right'}">
+            <mimic joint="arm_jaw_gripper_finger_right_joint" multiplier="-1.0" offset="0.0"/>
+          </xacro:unless>
+        </joint>
+        <link name="arm_jaw_gripper_finger_${side}_link">
+          <visual>
+            <geometry><mesh filename="${mesh_path}/arm_jaw_gripper_finger_v2.stl" scale="${stl_scale}"/></geometry>
+            <material name="light_grey"/>
+          </visual>
+          <collision>
+            <geometry><mesh filename="${mesh_path}/arm_jaw_gripper_finger_v2.stl" scale="${stl_scale}"/></geometry>
+          </collision>
+          <xacro:dummy_inertia mass="0.05"/>
+        </link>
+      </xacro:macro>
+      <!-- Same part mounted twice: "left" is the "right" finger rotated 180 deg about Z,
+           so both slide outward along their own local +X (axis) to open — no mirrored mesh needed. -->
+      <xacro:jaw_gripper_finger side="right" x_closed="${finger_x_closed}"  y="${finger_right_y}" yaw="0"      axis_sign="-1"/>
+      <xacro:jaw_gripper_finger side="left"  x_closed="${-finger_x_closed}" y="${finger_left_y}"  yaw="${pi}" axis_sign="1"/>
+    </xacro:if>
     <joint name="arm_tcp_joint" type="fixed">
       <parent link="arm_end_effector_link"/>
       <child link="arm_tcp_link"/>
-      <origin xyz="0 0 0.02" rpy="0 0 0"/>
-    </joint>
-    <!-- TCP (Tool Center Point) is a virtual point -->
+      <xacro:if value="${'$(arg end_effector)' == 'jaw'}">
+        <origin xyz="0 -0.23 0" rpy="0 0 0"/>
+      </xacro:if>
+      <xacro:if value="${'$(arg end_effector)' != 'jaw'}">
+        <origin xyz="0 -0.23 0" rpy="0 0 0"/>
+      </xacro:if>
+    </joint>
     <link name="arm_tcp_link"/>
-    <!-- ROS 2 Control Configuration -->
+    <joint name="arm_camera_joint" type="fixed">
+      <parent link="arm_end_effector_link"/>
+      <child link="arm_camera_link"/>
+      <origin xyz="0.0012919902801513672 0.07102805376052856 0.03884565830230713" rpy="0 ${-pi/2} ${-pi/2}"/>
+    </joint>
+    <link name="arm_camera_link">
+      <visual>
+        <geometry>
+          <box size="0.06 0.06 0.03"/>
+        </geometry>
+        <material name="camera_blue">
+          <color rgba="0.0 0.0 1.0 1.0"/>
+        </material>
+      </visual>
+      <collision>
+        <geometry>
+          <box size="0.06 0.06 0.03"/>
+        </geometry>
+      </collision>
+    </link>
+    <joint name="arm_camera_optical_joint" type="fixed">
+      <parent link="arm_camera_link"/>
+      <child link="arm_camera_optical_frame"/>
+      <origin xyz="0 0 0.03" rpy="${-pi/2} 0 ${-pi/2}"/>
+    </joint>
+    <link name="arm_camera_optical_frame"/>
     <ros2_control name="ArmSystem" type="system">
       <hardware>
-        <xacro:if value="$(arg use_fake_hardware)">
-          <plugin>mock_components/GenericSystem</plugin>
+        <xacro:if value="$(arg sim)">
+          <plugin>gz_ros2_control/GazeboSimSystem</plugin>
         </xacro:if>
-        <xacro:unless value="$(arg use_fake_hardware)">
-          <plugin>arm_hardware_interface/ArmCanSystem</plugin>
-          <param name="can_interface">can0</param>
-          <!-- Stiffness ramps 0 -> 100% over this many seconds after activation -->
-          <param name="gain_ramp_secs">6.0</param>
-          <!-- Hard rate limiter on outgoing position commands (rad/s).
-               Even a wrong/hostile command cannot move a joint faster than this.
-               Keep at 0.3 for the very first powered tests, raise later. -->
-          <param name="max_cmd_speed_rad_s">1.0</param>
-          <!-- Activation aborts if any motor is silent for this long -->
-          <param name="feedback_timeout_secs">2.0</param>
+        <xacro:unless value="$(arg sim)">
+          <xacro:if value="$(arg use_fake_hardware)">
+            <plugin>mock_components/GenericSystem</plugin>
+          </xacro:if>
+          <xacro:unless value="$(arg use_fake_hardware)">
+            <plugin>arm_hardware_interface/ArmCanSystem</plugin>
+            <param name="can_interface">can0</param>
+          </xacro:unless>
         </xacro:unless>
       </hardware>
-      <!-- ======================= CALIBRATION =======================
-           direction : +1 if pushing the joint in its URDF-positive direction
-                       (right-hand rule about the <axis>) makes the RAW motor
-                       angle increase; -1 otherwise.
-           offset    : the RAW motor angle (rad) measured when the arm is
-                       physically in the URDF zero pose. If you save the motor
-                       zero (0xB1 / FF..FE) at that pose, offset = 0.0.
-           kp / kd   : MIT gains — starting values are the proven ones from
-                       play_arm_waypoints.py. Halve kp for first powered tests.
-           Determine direction & offset with scripts/check_calibration.py
-           (torqueless) — see CALIBRATION_GUIDE.md.
-           ============================================================= -->
-      <xacro:macro name="arm_joint_control" params="joint_name motor_id direction offset kp kd">
+      <xacro:macro name="arm_joint_control" params="joint_name">
         <joint name="${joint_name}">
           <command_interface name="position">
@@ -161,22 +238,148 @@
             <param name="max">${pi}</param>
           </command_interface>
-          <command_interface name="velocity"/>
           <state_interface name="position"/>
           <state_interface name="velocity"/>
-          <param name="motor_id">${motor_id}</param>
-          <param name="direction">${direction}</param>
-          <param name="offset">${offset}</param>
-          <param name="kp">${kp}</param>
-          <param name="kd">${kd}</param>
         </joint>
       </xacro:macro>
-      <!-- TODO: replace direction/offset with YOUR measured calibration values -->
-      <xacro:arm_joint_control joint_name="arm_mount_base_joint"          motor_id="20" direction="-1" offset="1.9746" kp="15.0" kd="1.5"/>
-      <xacro:arm_joint_control joint_name="arm_base_shoulder_joint"       motor_id="21" direction="-1" offset="1.7093" kp="120.0" kd="4.0"/>
-      <xacro:arm_joint_control joint_name="arm_shoulder_forearm_joint" motor_id="22" direction="1" offset="-0.7155" kp="75.0" kd="2.75"/>
-      <xacro:arm_joint_control joint_name="arm_forearm_wrist_1_joint"     motor_id="23" direction="-1" offset="1.0378" kp="10.0" kd="1.0"/>
-      <xacro:arm_joint_control joint_name="arm_wrist_1_wrist_2_joint"     motor_id="24" direction="1"  offset="0.0" kp="30.0"  kd="1.0"/>
-      <xacro:arm_joint_control joint_name="arm_wrist_2_end_effector_joint" motor_id="25" direction="1" offset="0.0" kp="15.0"  kd="0.5"/>
+      <xacro:arm_joint_control joint_name="arm_mount_base_joint"/>
+      <xacro:arm_joint_control joint_name="arm_base_shoulder_joint"/>
+      <xacro:arm_joint_control joint_name="arm_shoulder_forearm_joint"/>
+      <xacro:arm_joint_control joint_name="arm_forearm_wrist_1_joint"/>
+      <xacro:arm_joint_control joint_name="arm_wrist_1_wrist_2_joint"/>
+      <xacro:arm_joint_control joint_name="arm_wrist_2_end_effector_joint"/>
+      <!-- Only the right finger joint needs a ros2_control interface: the
+           left one is a <mimic> of it, computed automatically (by
+           robot_state_publisher for TF, and by the planning scene monitor
+           for collision state) from the right joint's reported position —
+           it doesn't need its own state/command interface. Without this,
+           joint_state_broadcaster never reports arm_jaw_gripper_finger_right_joint
+           at all, and the planning scene monitor (used by both move_group
+           and Servo) considers the robot's state permanently incomplete,
+           which silently blocks all motion. -->
+      <xacro:if value="${'$(arg end_effector)' == 'jaw'}">
+        <joint name="arm_jaw_gripper_finger_right_joint">
+          <command_interface name="position">
+            <param name="min">0</param>
+            <param name="max">${finger_stroke}</param>
+          </command_interface>
+          <state_interface name="position"/>
+          <state_interface name="velocity"/>
+        </joint>
+      </xacro:if>
     </ros2_control>
+    <xacro:if value="$(arg sim)">
+      <gazebo>
+        <plugin filename="gz_ros2_control-system" name="gz_ros2_control::GazeboSimROS2ControlPlugin">
+          <parameters>$(find arm_sim)/config/ros2_controllers.yaml</parameters>
+        </plugin>
+      </gazebo>
+      <gazebo reference="arm_mount_link">
+        <visual>
+          <material>
+            <ambient>0.7 0.7 0.7 1.0</ambient>
+            <diffuse>0.7 0.7 0.7 1.0</diffuse>
+            <specular>0.3 0.3 0.3 1.0</specular>
+          </material>
+        </visual>
+      </gazebo>
+      <gazebo reference="arm_base_link">
+        <visual>
+          <material>
+            <ambient>0.7 0.7 0.7 1.0</ambient>
+            <diffuse>0.7 0.7 0.7 1.0</diffuse>
+            <specular>0.3 0.3 0.3 1.0</specular>
+          </material>
+        </visual>
+      </gazebo>
+      <gazebo reference="arm_shoulder_link">
+        <visual>
+          <material>
+            <ambient>0.7 0.7 0.7 1.0</ambient>
+            <diffuse>0.7 0.7 0.7 1.0</diffuse>
+            <specular>0.3 0.3 0.3 1.0</specular>
+          </material>
+        </visual>
+      </gazebo>
+      <gazebo reference="arm_forearm_link">
+        <visual>
+          <material>
+            <ambient>0.7 0.7 0.7 1.0</ambient>
+            <diffuse>0.7 0.7 0.7 1.0</diffuse>
+            <specular>0.3 0.3 0.3 1.0</specular>
+          </material>
+        </visual>
+      </gazebo>
+      <gazebo reference="arm_wrist_1_link">
+        <visual>
+          <material>
+            <ambient>0.7 0.7 0.7 1.0</ambient>
+            <diffuse>0.7 0.7 0.7 1.0</diffuse>
+            <specular>0.3 0.3 0.3 1.0</specular>
+          </material>
+        </visual>
+      </gazebo>
+      <gazebo reference="arm_wrist_2_link">
+        <visual>
+          <material>
+            <ambient>0.7 0.7 0.7 1.0</ambient>
+            <diffuse>0.7 0.7 0.7 1.0</diffuse>
+            <specular>0.3 0.3 0.3 1.0</specular>
+          </material>
+        </visual>
+      </gazebo>
+      <gazebo reference="arm_end_effector_link">
+        <visual>
+          <material>
+            <ambient>0.7 0.7 0.7 1.0</ambient>
+            <diffuse>0.7 0.7 0.7 1.0</diffuse>
+            <specular>0.3 0.3 0.3 1.0</specular>
+          </material>
+        </visual>
+      </gazebo>
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