Commit message: chore(arm): recalibrate direction/offset/kp/kd for new mesh; enable gravity_ff params.

File: src/arm/arm_description/urdf/arm_macro.xacro (robot description, xacro)
@@ -229,8 +229,28 @@
             <plugin>arm_hardware_interface/ArmCanSystem</plugin>
             <param name="can_interface">can0</param>
+            <!-- Stiffness ramps 0 -> 100% over this many seconds after activation -->
+            <param name="gain_ramp_secs">15.0</param>
+            <!-- Hard rate limiter on outgoing position commands (rad/s) —
+                 even a wrong/hostile command can't move a joint faster than this. -->
+            <param name="max_cmd_speed_rad_s">1.0</param>
+            <!-- Activation aborts if any motor is silent for this long -->
+            <param name="feedback_timeout_secs">2.0</param>
+            <param name="gravity_ff_enabled">true</param>
+            <param name="gravity_ff_max_nm">8.0</param>
           </xacro:unless>
         </xacro:unless>
       </hardware>
-      <xacro:macro name="arm_joint_control" params="joint_name">
+      <!-- ======================= CALIBRATION =======================
+           direction : +1 if pushing the joint in its URDF-positive direction
+                       (right-hand rule about the <axis>) makes the RAW motor
+                       angle increase; -1 otherwise.
+           offset    : the RAW motor angle (rad) measured when the arm is
+                       physically in the URDF zero pose. If you save the motor
+                       zero (0xB1 / FF..FE) at that pose, offset = 0.0.
+           kp / kd   : MIT gains, tuned on real hardware.
+           Re-verify with scripts/check_calibration.py (torqueless) after any
+           mesh/geometry change that alters a joint's <axis>.
+           ============================================================= -->
+      <xacro:macro name="arm_joint_control" params="joint_name motor_id direction offset kp kd">
         <joint name="${joint_name}">
           <command_interface name="position">
@@ -238,24 +258,25 @@
             <param name="max">${pi}</param>
           </command_interface>
+          <command_interface name="velocity"/>
           <state_interface name="position"/>
           <state_interface name="velocity"/>
+          <param name="motor_id">${motor_id}</param>
+          <param name="direction">${direction}</param>
+          <param name="offset">${offset}</param>
+          <param name="kp">${kp}</param>
+          <param name="kd">${kd}</param>
         </joint>
       </xacro:macro>
-      <xacro:arm_joint_control joint_name="arm_mount_base_joint"/>
-      <xacro:arm_joint_control joint_name="arm_base_shoulder_joint"/>
-      <xacro:arm_joint_control joint_name="arm_shoulder_forearm_joint"/>
-      <xacro:arm_joint_control joint_name="arm_forearm_wrist_1_joint"/>
-      <xacro:arm_joint_control joint_name="arm_wrist_1_wrist_2_joint"/>
-      <xacro:arm_joint_control joint_name="arm_wrist_2_end_effector_joint"/>
-      <!-- Only the right finger joint needs a ros2_control interface: the
-           left one is a <mimic> of it, computed automatically (by
-           robot_state_publisher for TF, and by the planning scene monitor
-           for collision state) from the right joint's reported position —
-           it doesn't need its own state/command interface. Without this,
-           joint_state_broadcaster never reports arm_jaw_gripper_finger_right_joint
-           at all, and the planning scene monitor (used by both move_group
-           and Servo) considers the robot's state permanently incomplete,
-           which silently blocks all motion. -->
-      <xacro:if value="${'$(arg end_effector)' == 'jaw'}">
+      <xacro:arm_joint_control joint_name="arm_mount_base_joint"          motor_id="20" direction="-1" offset="0.0"  kp="60.0"  kd="4.0"/>
+      <xacro:arm_joint_control joint_name="arm_base_shoulder_joint"       motor_id="21" direction="1" offset="0.0"  kp="80.0" kd="5.0"/>
+      <xacro:arm_joint_control joint_name="arm_shoulder_forearm_joint"    motor_id="22" direction="-1"  offset="0.0" kp="60.0" kd="4.0"/>
+      <xacro:arm_joint_control joint_name="arm_forearm_wrist_1_joint"     motor_id="23" direction="-1" offset="0.0"  kp="15.0"  kd="3.0"/>
+      <xacro:arm_joint_control joint_name="arm_wrist_1_wrist_2_joint"     motor_id="24" direction="-1"  offset="0.0"     kp="15.0"  kd="3.0"/>
+      <xacro:arm_joint_control joint_name="arm_wrist_2_end_effector_joint" motor_id="25" direction="1" offset="0.0"     kp="10.0"  kd="3.0"/>
+      <!-- Only the right finger needs an interface: left is a <mimic> of it.
+           sim/fake only — ArmCanSystem hardcodes NUM_JOINTS=6 and has no
+           motor for the gripper yet; claiming this joint on real hardware
+           causes "Expected 6 joints, got 7" and a crash on activation. -->
+      <xacro:if value="${('$(arg end_effector)' == 'jaw') and (('$(arg sim)' == 'true') or ('$(arg use_fake_hardware)' == 'true'))}">
         <joint name="arm_jaw_gripper_finger_right_joint">
           <command_interface name="position">

Commit message: Feature/arm/replace meshes (#516)
* feat: replace arm meshes

* fix(arm): unblock Servo motion and fix camera/roll behavior

* fix(arm): flip gripper 180°, reposition camera, fix camera self-view

* fix(arm): fix gripper mimic limits and camera optical-frame TF

* fix(arm): estimate TCP offset from v2 gripper mesh geometry

---------

Co-authored-by: Martik-k <kosiv.marta@gmail.com>

File: src/arm/arm_description/urdf/arm_macro.xacro (robot description, xacro)
@@ -28,9 +28,9 @@
     <link name="arm_mount_link">
       <visual>
-        <geometry><mesh filename="${mesh_path}/arm_mount.stl" scale="${stl_scale}"/></geometry>
-        <material name="light_grey"/>
-      </visual>
-      <collision>
-        <geometry><mesh filename="${mesh_path}/arm_mount.stl" scale="${stl_scale}"/></geometry>
+        <geometry><mesh filename="${mesh_path}/arm_mount_v2.stl" scale="${stl_scale}"/></geometry>
+        <material name="light_grey"/>
+      </visual>
+      <collision>
+        <geometry><mesh filename="${mesh_path}/arm_mount_v2.stl" scale="${stl_scale}"/></geometry>
       </collision>
       <xacro:dummy_inertia mass="1.0"/>
@@ -39,5 +39,5 @@
       <parent link="arm_mount_link"/>
       <child link="arm_base_link"/>
-      <origin xyz="0 0 0.018" rpy="0 0 0"/>
+      <origin xyz="0.06 0 0.021" rpy="0 0 0"/>
       <axis xyz="0 0 1"/>
       <limit lower="${-pi}" upper="${pi}" effort="100.0" velocity="1.0"/>
@@ -45,9 +45,9 @@
     <link name="arm_base_link">
       <visual>
-        <geometry><mesh filename="${mesh_path}/arm_base.stl" scale="${stl_scale}"/></geometry>
-        <material name="light_grey"/>
-      </visual>
-      <collision>
-        <geometry><mesh filename="${mesh_path}/arm_base.stl" scale="${stl_scale}"/></geometry>
+        <geometry><mesh filename="${mesh_path}/arm_base_v2.stl" scale="${stl_scale}"/></geometry>
+        <material name="light_grey"/>
+      </visual>
+      <collision>
+        <geometry><mesh filename="${mesh_path}/arm_base_v2.stl" scale="${stl_scale}"/></geometry>
       </collision>
       <xacro:dummy_inertia mass="2.0"/>
@@ -56,15 +56,15 @@
       <parent link="arm_base_link"/>
       <child link="arm_shoulder_link"/>
-      <origin xyz="0 0.013 0.0945" rpy="0 0 ${-pi/2}"/>
+      <origin xyz="-0.040366 -0.000325 0.103" rpy="${pi/6} 0 ${-pi}"/>
       <axis xyz="1 0 0"/>
-      <limit lower="${-pi/2}" upper="${pi}" effort="100.0" velocity="1.0"/>
+      <limit lower="${-pi}" upper="${pi}" effort="100.0" velocity="1.0"/>
     </joint>
     <link name="arm_shoulder_link">
       <visual>
-        <geometry><mesh filename="${mesh_path}/arm_shoulder.stl" scale="${stl_scale}"/></geometry>
-        <material name="light_grey"/>
-      </visual>
-      <collision>
-        <geometry><mesh filename="${mesh_path}/arm_shoulder.stl" scale="${stl_scale}"/></geometry>
+        <geometry><mesh filename="${mesh_path}/arm_shoulder_v2.stl" scale="${stl_scale}"/></geometry>
+        <material name="light_grey"/>
+      </visual>
+      <collision>
+        <geometry><mesh filename="${mesh_path}/arm_shoulder_v2.stl" scale="${stl_scale}"/></geometry>
       </collision>
       <xacro:dummy_inertia mass="1.5"/>
@@ -73,5 +73,5 @@
       <parent link="arm_shoulder_link"/>
       <child link="arm_forearm_link"/>
-      <origin xyz="-0.057 0 0.5" rpy="0 0 0"/>
+      <origin xyz="0 0.3 0" rpy="${5*pi/6} 0 0"/>
       <axis xyz="1 0 0"/>
       <limit lower="${-pi/2}" upper="${pi/2}" effort="100.0" velocity="1.0"/>
@@ -79,9 +79,9 @@
     <link name="arm_forearm_link">
       <visual>
-        <geometry><mesh filename="${mesh_path}/arm_forearm.stl" scale="${stl_scale}"/></geometry>
-        <material name="light_grey"/>
-      </visual>
-      <collision>
-        <geometry><mesh filename="${mesh_path}/arm_forearm.stl" scale="${stl_scale}"/></geometry>
+        <geometry><mesh filename="${mesh_path}/arm_forearm_v2.stl" scale="${stl_scale}"/></geometry>
+        <material name="light_grey"/>
+      </visual>
+      <collision>
+        <geometry><mesh filename="${mesh_path}/arm_forearm_v2.stl" scale="${stl_scale}"/></geometry>
       </collision>
       <xacro:dummy_inertia mass="1.0"/>
@@ -90,15 +90,15 @@
       <parent link="arm_forearm_link"/>
       <child link="arm_wrist_1_link"/>
-      <origin xyz="0.002175 0 0.4" rpy="${pi} ${pi} 0"/>
-      <axis xyz="1 0 0"/>
+      <origin xyz="-0.0173 0.3 0" rpy="0 ${pi/2} 0"/>
+      <axis xyz="0 0 1"/>
       <limit lower="${-pi/2}" upper="${pi/2}" effort="100.0" velocity="1.0"/>
     </joint>
     <link name="arm_wrist_1_link">
       <visual>
-        <geometry><mesh filename="${mesh_path}/arm_wrist_1.stl" scale="${stl_scale}"/></geometry>
-        <material name="light_grey"/>
-      </visual>
-      <collision>
-        <geometry><mesh filename="${mesh_path}/arm_wrist_1.stl" scale="${stl_scale}"/></geometry>
+        <geometry><mesh filename="${mesh_path}/arm_wrist_v2.stl" scale="${stl_scale}"/></geometry>
+        <material name="light_grey"/>
+      </visual>
+      <collision>
+        <geometry><mesh filename="${mesh_path}/arm_wrist_v2.stl" scale="${stl_scale}"/></geometry>
       </collision>
       <xacro:dummy_inertia mass="0.5"/>
@@ -107,15 +107,15 @@
       <parent link="arm_wrist_1_link"/>
       <child link="arm_wrist_2_link"/>
-      <origin xyz="-0.067825 0 0.0353" rpy="0 ${pi/2} 0"/>
-      <axis xyz="1 0 0"/>
+      <origin xyz="0.0323 0 -0.035" rpy="${-pi/2} 0 ${pi/2}"/>
+      <axis xyz="0 0 1"/>
       <limit lower="${-pi}" upper="${pi}" effort="100.0" velocity="1.0"/>
     </joint>
     <link name="arm_wrist_2_link">
       <visual>
-        <geometry><mesh filename="${mesh_path}/arm_wrist_2.stl" scale="${stl_scale}"/></geometry>
-        <material name="light_grey"/>
-      </visual>
-      <collision>
-        <geometry><mesh filename="${mesh_path}/arm_wrist_2.stl" scale="${stl_scale}"/></geometry>
+        <geometry><mesh filename="${mesh_path}/arm_wrist_v2.stl" scale="${stl_scale}"/></geometry>
+        <material name="light_grey"/>
+      </visual>
+      <collision>
+        <geometry><mesh filename="${mesh_path}/arm_wrist_v2.stl" scale="${stl_scale}"/></geometry>
       </collision>
       <xacro:dummy_inertia mass="0.3"/>
@@ -124,6 +124,6 @@
       <parent link="arm_wrist_2_link"/>
       <child link="arm_end_effector_link"/>
-      <origin xyz="-0.067825 0 0.0353" rpy="${-pi/2} 0 ${-pi/2}"/>
-      <axis xyz="0 1 0"/>
+      <origin xyz="0.0323 0 -0.035" rpy="${pi/2} 0 ${pi/2}"/>
+      <axis xyz="0 0 1"/>
       <limit lower="${-pi}" upper="${pi}" effort="100.0" velocity="1.0"/>
     </joint>
@@ -131,9 +131,9 @@
       <xacro:if value="${'$(arg end_effector)' == 'jaw'}">
         <visual>
-          <geometry><mesh filename="${mesh_path}/jaw_gripper.stl" scale="${stl_scale}"/></geometry>
+          <geometry><mesh filename="${mesh_path}/arm_jaw_gripper_v2.stl" scale="${stl_scale}"/></geometry>
           <material name="light_grey"/>
         </visual>
         <collision>
-          <geometry><mesh filename="${mesh_path}/jaw_gripper.stl" scale="${stl_scale}"/></geometry>
+          <geometry><mesh filename="${mesh_path}/arm_jaw_gripper_v2.stl" scale="${stl_scale}"/></geometry>
         </collision>
       </xacro:if>
@@ -142,9 +142,54 @@
       <xacro:dummy_inertia mass="0.2"/>
     </link>
+    <xacro:if value="${'$(arg end_effector)' == 'jaw'}">
+      <!-- From CAD, origin of each finger relative to gripper origin (mm):
+           finger 1 (right): closed (3.5, -10.72, 122.133)  -> open (15.5, -10.72, 122.133)
+           finger 2 (left):  closed (-3.5, 13.78, 122.133)  -> open (-15.5, 13.78, 122.133)
+           X is symmetric (+-3.5mm closed, +-12mm stroke); Y is NOT mirrored between the two
+           fingers on purpose (offset so the finger pads clear each other near full close). -->
+      <xacro:property name="finger_x_closed" value="-0.0035"/>
+      <xacro:property name="finger_stroke" value="0.012"/>
+      <xacro:property name="finger_z" value="0.122133"/>
+      <xacro:property name="finger_right_y" value="0.01072"/>
+      <xacro:property name="finger_left_y" value="-0.01378"/>
+      <xacro:macro name="jaw_gripper_finger" params="side x_closed y yaw axis_sign limit_lower limit_upper">
+        <joint name="arm_jaw_gripper_finger_${side}_joint" type="prismatic">
+          <parent link="arm_end_effector_link"/>
+          <child link="arm_jaw_gripper_finger_${side}_link"/>
+          <origin xyz="${x_closed} ${y} ${finger_z}" rpy="0 0 ${yaw}"/>
+          <axis xyz="${axis_sign} 0 0"/>
+          <limit lower="${limit_lower}" upper="${limit_upper}" effort="20.0" velocity="0.05"/>
+          <xacro:unless value="${side == 'right'}">
+            <!-- Right and left are mirror images (180 deg about Z), so their axes
+                 point opposite ways in the parent frame — multiplier=-1.0 makes
+                 them slide apart symmetrically as the right joint opens, rather
+                 than translating together with a fixed gap. Left's own range is
+                 shifted negative to match, since its opening motion is the
+                 mirror of right's (mimic must stay within the child's own
+                 declared limits). -->
+            <mimic joint="arm_jaw_gripper_finger_right_joint" multiplier="-1.0" offset="0.0"/>
+          </xacro:unless>
+        </joint>
+        <link name="arm_jaw_gripper_finger_${side}_link">
+          <visual>
+            <geometry><mesh filename="${mesh_path}/arm_jaw_gripper_finger_v2.stl" scale="${stl_scale}"/></geometry>
+            <material name="light_grey"/>
+          </visual>
+          <collision>
+            <geometry><mesh filename="${mesh_path}/arm_jaw_gripper_finger_v2.stl" scale="${stl_scale}"/></geometry>
+          </collision>
+          <xacro:dummy_inertia mass="0.05"/>
+        </link>
+      </xacro:macro>
+      <!-- Same part mounted twice: "left" is the "right" finger rotated 180 deg about Z,
+           so both slide outward along their own local +X (axis) to open — no mirrored mesh needed. -->
+      <xacro:jaw_gripper_finger side="right" x_closed="${finger_x_closed}"  y="${finger_right_y}" yaw="0"      axis_sign="-1" limit_lower="0"                limit_upper="${finger_stroke}"/>
+      <xacro:jaw_gripper_finger side="left"  x_closed="${-finger_x_closed}" y="${finger_left_y}"  yaw="${pi}" axis_sign="1"  limit_lower="${-finger_stroke}" limit_upper="0"/>
+    </xacro:if>
     <joint name="arm_tcp_joint" type="fixed">
       <parent link="arm_end_effector_link"/>
       <child link="arm_tcp_link"/>
       <xacro:if value="${'$(arg end_effector)' == 'jaw'}">
-        <origin xyz="0 -0.23 0" rpy="0 0 0"/>
+        <origin xyz="0 -0.0015 0.2072" rpy="0 0 0"/>
       </xacro:if>
       <xacro:if value="${'$(arg end_effector)' != 'jaw'}">
@@ -156,10 +201,10 @@
       <parent link="arm_end_effector_link"/>
       <child link="arm_camera_link"/>
-      <origin xyz="-0.00110236 -0.0683370 -0.0340064" rpy="${pi} 0 ${-pi/2}"/>
+      <origin xyz="0.0012604892253875732 -0.045 0.07839690148830414" rpy="0 ${-pi/2} ${pi/2}"/>
     </joint>
     <link name="arm_camera_link">
       <visual>
         <geometry>
-          <box size="0.06 0.06 0.03"/>
+          <box size="0.06 0.06 0.06"/>
         </geometry>
         <material name="camera_blue">
@@ -169,5 +214,5 @@
       <collision>
         <geometry>
-          <box size="0.06 0.06 0.03"/>
+          <box size="0.06 0.06 0.06"/>
         </geometry>
       </collision>
@@ -176,5 +221,5 @@
       <parent link="arm_camera_link"/>
       <child link="arm_camera_optical_frame"/>
-      <origin xyz="0 0 0.03" rpy="${-pi/2} 0 ${-pi/2}"/>
+      <origin xyz="0.045 0 0" rpy="${-pi/2} 0 ${-pi/2}"/>
     </joint>
     <link name="arm_camera_optical_frame"/>
@@ -210,4 +255,23 @@
       <xacro:arm_joint_control joint_name="arm_wrist_1_wrist_2_joint"/>
       <xacro:arm_joint_control joint_name="arm_wrist_2_end_effector_joint"/>
+      <!-- Only the right finger joint needs a ros2_control interface: the
+           left one is a <mimic> of it, computed automatically (by
+           robot_state_publisher for TF, and by the planning scene monitor
+           for collision state) from the right joint's reported position —
+           it doesn't need its own state/command interface. Without this,
+           joint_state_broadcaster never reports arm_jaw_gripper_finger_right_joint
+           at all, and the planning scene monitor (used by both move_group
+           and Servo) considers the robot's state permanently incomplete,
+           which silently blocks all motion. -->
+      <xacro:if value="${'$(arg end_effector)' == 'jaw'}">
+        <joint name="arm_jaw_gripper_finger_right_joint">
+          <command_interface name="position">
+            <param name="min">0</param>
+            <param name="max">${finger_stroke}</param>
+          </command_interface>
+          <state_interface name="position"/>
+          <state_interface name="velocity"/>
+        </joint>
+      </xacro:if>
     </ros2_control>
     <xacro:if value="$(arg sim)">
@@ -280,8 +344,28 @@
         </visual>
       </gazebo>
+      <xacro:if value="${'$(arg end_effector)' == 'jaw'}">
+        <gazebo reference="arm_jaw_gripper_finger_right_link">
+          <visual>
+            <material>
+              <ambient>0.7 0.7 0.7 1.0</ambient>
+              <diffuse>0.7 0.7 0.7 1.0</diffuse>
+              <specular>0.3 0.3 0.3 1.0</specular>
+            </material>
+          </visual>
+        </gazebo>
+        <gazebo reference="arm_jaw_gripper_finger_left_link">
+          <visual>
+            <material>
+              <ambient>0.7 0.7 0.7 1.0</ambient>
+              <diffuse>0.7 0.7 0.7 1.0</diffuse>
+              <specular>0.3 0.3 0.3 1.0</specular>
+            </material>
+          </visual>
+        </gazebo>
+      </xacro:if>
       <xacro:if value="$(arg camera)">
       <gazebo reference="arm_camera_link">
         <sensor name="arm_camera" type="camera">
-          <pose>0 0 0.03 0 0 0</pose>
+          <pose>0.045 0 0 0 0 0</pose>
           <camera>
             <optical_frame_id>arm_camera_optical_frame</optical_frame_id>

Commit message: fix(arm): give the jaw gripper finger its own mock hardware component

File: src/arm/arm_description/urdf/arm_macro.xacro (robot description, xacro)
@@ -282,12 +282,8 @@
       <xacro:arm_joint_control joint_name="arm_wrist_2_end_effector_joint" motor_id="25" direction="1" offset="0.0"     kp="10.0"  kd="3.0"/>
       <!-- Only the right finger needs an interface: left is a <mimic> of it.
-           sim/fake only — ArmCanSystem hardcodes NUM_JOINTS=6 and has no motor
-           for the gripper, so claiming this joint on real hardware fails with
-           "Expected 6 joints, got 7". Trade-off: on real hardware the finger is
-           then absent from joint_state_broadcaster, so the planning scene monitor
-           sees an incomplete state and silently blocks move_group/Servo motion.
-           Real-hardware Servo will need the gripper in its own
-           mock_components/GenericSystem <ros2_control> block. -->
-      <xacro:if value="${'$(arg end_effector)' == 'jaw'}">
+           Excluded on real hardware — ArmCanSystem hardcodes NUM_JOINTS=6 and
+           would fail with "Expected 6 joints, got 7"; the JawGripperStub
+           component below covers that case instead. -->
+      <xacro:if value="${('$(arg end_effector)' == 'jaw') and (('$(arg sim)' == 'true') or ('$(arg use_fake_hardware)' == 'true'))}">
         <joint name="arm_jaw_gripper_finger_right_joint">
           <command_interface name="position">
@@ -300,4 +296,28 @@
       </xacro:if>
     </ros2_control>
+    <!-- There is no gripper motor on the real arm yet, but the finger joint must
+         still report state: without it joint_state_broadcaster never publishes
+         the joint, the planning scene monitor sees an incomplete robot state,
+         and move_group/Servo silently refuse to move. GenericSystem echoes
+         commands back as state, so the joint exists for MoveIt while nothing
+         physical moves. Replace with the real gripper hardware plugin once the
+         motor is wired up. -->
+    <xacro:if value="${('$(arg end_effector)' == 'jaw') and ('$(arg sim)' == 'false') and ('$(arg use_fake_hardware)' == 'false')}">
+      <ros2_control name="JawGripperStub" type="system">
+        <hardware>
+          <plugin>mock_components/GenericSystem</plugin>
+        </hardware>
+        <joint name="arm_jaw_gripper_finger_right_joint">
+          <command_interface name="position">
+            <param name="min">0</param>
+            <param name="max">${finger_stroke}</param>
+          </command_interface>
+          <state_interface name="position">
+            <param name="initial_value">0.0</param>
+          </state_interface>
+          <state_interface name="velocity"/>
+        </joint>
+      </ros2_control>
+    </xacro:if>
     <xacro:if value="$(arg sim)">
       <gazebo>
