Commit message: fix(rover): sync rover_description with develop, keep arm mount + accessories

File: src/rover_description/urdf/rover.urdf.xacro (robot description, xacro)
@@ -1,4 +1,9 @@
 <?xml version="1.0"?>
-<robot name="indomitus_s1" xmlns:xacro="http://www.ros.org/wiki/xacro">
+<robot xmlns:xacro="http://www.ros.org/wiki/xacro">
+  <xacro:include filename="$(find rover_description)/urdf/properties.xacro"/>
+  <xacro:include filename="$(find rover_description)/urdf/macros/inertia_macros.xacro"/>
+  <xacro:include filename="$(find rover_description)/urdf/macros/rocker_assembly.xacro"/>
+  <xacro:include filename="$(find rover_description)/urdf/macros/accessories.xacro"/>
+  <xacro:include filename="$(find rover_description)/urdf/camera.xacro"/>
   <!-- mount_arm:=true bolts the indomitus_arm (arm_description) onto
        main_body_link, matching the real hardware where the arm is
@@ -13,11 +18,11 @@
   <!-- ===================== MATERIALS ===================== -->
   <material name="blue_body">
-    <color rgba="0.2 0.4 0.8 1"/>
+    <color rgba="0.55 0.56 0.58 1"/>
   </material>
   <material name="grey_structure">
-    <color rgba="0.6 0.6 0.6 1"/>
+    <color rgba="0.55 0.56 0.58 1"/>
   </material>
   <material name="orange_mount">
-    <color rgba="0.8 0.4 0.0 1"/>
+    <color rgba="0.55 0.56 0.58 1"/>
   </material>
   <material name="dark_wheel">
@@ -25,5 +30,11 @@
   </material>
   <material name="red_axii">
-    <color rgba="0.4 0.4 0.4 1"/>
+    <color rgba="0.55 0.56 0.58 1"/>
+  </material>
+  <material name="beacon_light">
+    <color rgba="0.9 0.35 0.05 1"/>
+  </material>
+  <material name="button_red">
+    <color rgba="0.7 0.05 0.05 1"/>
   </material>
   <!-- ===================== BASE ===================== -->
@@ -38,6 +49,6 @@
     <inertial>
       <origin xyz="0 0 0" rpy="0 0 0"/>
-      <mass value="0.5"/>
-      <inertia ixx="0.5" iyy="0.5" izz="1.0" ixy="0" ixz="0" iyz="0"/>
+      <mass value="${axii_mass}"/>
+      <xacro:box_inertia m="${axii_mass}" x="${axii_length}" y="${axii_width}" z="${axii_height}"/>
     </inertial>
     <visual>
@@ -51,5 +62,5 @@
       <origin xyz="0 0 0" rpy="0 0 0"/>
       <geometry>
-        <box size="0.1 0.68 0.05"/>
+        <box size="${axii_length} ${axii_width} ${axii_height}"/>
       </geometry>
     </collision>
@@ -64,11 +75,11 @@
     <inertial>
       <origin xyz="0 0 0" rpy="0 0 0"/>
-      <mass value="40.0"/>
-      <inertia ixx="0.608" iyy="1.283" izz="1.733" ixy="0" ixz="0" iyz="0"/>
+      <mass value="${body_mass}"/>
+      <xacro:box_inertia m="${body_mass}" x="${body_length}" y="${body_width}" z="${body_height}"/>
     </inertial>
     <visual>
       <origin xyz="0 0 0" rpy="0 0 0"/>
       <geometry>
-        <box size="0.6 0.4 0.2"/>
+        <box size="${body_length} ${body_width} ${body_height}"/>
       </geometry>
       <material name="blue_body"/>
@@ -77,5 +88,5 @@
       <origin xyz="0 0 0" rpy="0 0 0"/>
       <geometry>
-        <box size="0.6 0.4 0.15"/>
+        <box size="${body_length} ${body_width} ${body_height}"/>
       </geometry>
     </collision>
@@ -84,295 +95,16 @@
     <parent link="suspension_base_axii_link"/>
     <child link="main_body_link"/>
-    <origin xyz="-0.04 0 0.05" rpy="0 0 0"/>
+    <origin xyz="0 0 0.02" rpy="0 0 0"/>
   </joint>
   <!-- ===================== CAMERA ===================== -->
-  <xacro:include filename="$(find rover_description)/urdf/camera.xacro"/>
   <xacro:camera/>
-  <!-- ===================== LEFT ROCKER ===================== -->
-  <link name="l_rocker_link">
-    <inertial>
-      <origin xyz="0 0 0" rpy="0 0 0"/>
-      <mass value="1.0"/>
-      <inertia ixx="0.01" iyy="0.01" izz="0.01" ixy="0" ixz="0" iyz="0"/>
-    </inertial>
-    <visual>
-      <origin xyz="-0.55 0.02 -0.04" rpy="0 0 0"/>
-      <geometry>
-        <mesh filename="package://rover_description/meshes/suspension/rocker.stl" scale="0.001 0.001 0.001"/>
-      </geometry>
-      <material name="grey_structure"/>
-    </visual>
-    <collision>
-      <origin xyz="0 0 0" rpy="0 0 0"/>
-      <geometry>
-        <box size="1.1 0.04 0.08"/>
-      </geometry>
-    </collision>
-  </link>
-  <joint name="l_rocker_joint" type="revolute">
-    <parent link="suspension_base_axii_link"/>
-    <child link="l_rocker_link"/>
-    <origin xyz="0 0.34 0" rpy="0 0 0"/>
-    <axis xyz="0 1 0"/>
-    <limit lower="-0.5" upper="0.5" effort="100" velocity="1.0"/>
-    <dynamics damping="0.5" friction="0.1"/>
-  </joint>
-  <!-- ===================== RIGHT ROCKER ===================== -->
-  <link name="r_rocker_link">
-    <inertial>
-      <origin xyz="0 0 0" rpy="0 0 0"/>
-      <mass value="1.0"/>
-      <inertia ixx="0.01" iyy="0.01" izz="0.01" ixy="0" ixz="0" iyz="0"/>
-    </inertial>
-    <visual>
-      <origin xyz="-0.55 0.02 -0.04" rpy="0 0 0"/>
-      <geometry>
-        <mesh filename="package://rover_description/meshes/suspension/rocker.stl" scale="0.001 0.001 0.001"/>
-      </geometry>
-      <material name="grey_structure"/>
-    </visual>
-    <collision>
-      <origin xyz="0 0 0" rpy="0 0 0"/>
-      <geometry>
-        <box size="1.1 0.04 0.08"/>
-      </geometry>
-    </collision>
-  </link>
-  <joint name="r_rocker_joint" type="revolute">
-    <parent link="suspension_base_axii_link"/>
-    <child link="r_rocker_link"/>
-    <origin xyz="0 -0.34 0" rpy="0 0 0"/>
-    <axis xyz="0 1 0"/>
-    <limit lower="-0.5" upper="0.5" effort="100" velocity="1.0"/>
-    <dynamics damping="0.5" friction="0.1"/>
-  </joint>
-  <!-- ===================== FRONT LEFT WHEEL MOUNT ===================== -->
-  <link name="fl_wheel_mount_link">
-    <inertial>
-      <origin xyz="0 0 0" rpy="0 0 0"/>
-      <mass value="0.162"/>
-      <inertia ixx="0.0002" iyy="0.00012" izz="0.00012" ixy="0" ixz="0" iyz="0"/>
-    </inertial>
-    <visual>
-      <origin xyz="0 -0.06 -0.269" rpy="0 0 0"/>
-      <geometry>
-        <mesh filename="package://rover_description/meshes/suspension/wheel_mount.stl" scale="0.001 0.001 0.001"/>
-      </geometry>
-      <material name="orange_mount"/>
-    </visual>
-    <collision>
-      <origin xyz="0 0.11125 -0.18" rpy="0 0 0"/>
-      <geometry>
-        <box size="0.07 0.0625 0.25"/>
-      </geometry>
-    </collision>
-  </link>
-  <joint name="fl_wheel_mount_joint" type="revolute">
-    <parent link="l_rocker_link"/>
-    <child link="fl_wheel_mount_link"/>
-    <origin xyz="0.421 0 0" rpy="0 0 0"/>
-    <axis xyz="0 0 1"/>
-    <limit lower="-4.71238898" upper="4.71238898" effort="500" velocity="2"/>
-    <dynamics damping="0.5" friction="0.3"/>
-  </joint>
-  <!-- ===================== FRONT LEFT WHEEL ===================== -->
-  <link name="fl_wheel_link">
-    <inertial>
-      <origin xyz="0 0 0" rpy="0 0 0"/>
-      <mass value="0.5"/>
-      <inertia ixx="0.00563" iyy="0.00563" izz="0.01125" ixy="0" ixz="0" iyz="0"/>
-    </inertial>
-    <visual>
-      <origin xyz="0 -0.06 0" rpy="-1.5708 0 0"/>
-      <geometry>
-        <mesh filename="package://rover_description/meshes/suspension/wheel.stl" scale="0.001 0.001 0.001"/>
-      </geometry>
-      <material name="dark_wheel"/>
-    </visual>
-    <collision>
-      <origin xyz="0 0 0" rpy="1.5708 0 0"/>
-      <geometry>
-        <cylinder radius="0.15" length="0.12"/>
-      </geometry>
-    </collision>
-  </link>
-  <joint name="fl_wheel_joint" type="continuous">
-    <parent link="fl_wheel_mount_link"/>
-    <child link="fl_wheel_link"/>
-    <origin xyz="0 0 -0.27" rpy="0 0 0"/>
-    <axis xyz="0 1 0"/>
-    <limit effort="100" velocity="10"/>
-  </joint>
-  <!-- ===================== FRONT RIGHT WHEEL MOUNT ===================== -->
-  <link name="fr_wheel_mount_link">
-    <inertial>
-      <origin xyz="0 0 0" rpy="0 0 0"/>
-      <mass value="0.162"/>
-      <inertia ixx="0.0002" iyy="0.00012" izz="0.00012" ixy="0" ixz="0" iyz="0"/>
-    </inertial>
-    <visual>
-      <origin xyz="0 0.06 -0.269" rpy="0 0 3.14159"/>
-      <geometry>
-        <mesh filename="package://rover_description/meshes/suspension/wheel_mount.stl" scale="0.001 0.001 0.001"/>
-      </geometry>
-      <material name="orange_mount"/>
-    </visual>
-    <collision>
-      <origin xyz="0 -0.11125 -0.18" rpy="0 0 0"/>
-      <geometry>
-        <box size="0.07 0.0625 0.25"/>
-      </geometry>
-    </collision>
-  </link>
-  <joint name="fr_wheel_mount_joint" type="revolute">
-    <parent link="r_rocker_link"/>
-    <child link="fr_wheel_mount_link"/>
-    <origin xyz="0.421 0 0" rpy="0 0 0"/>
-    <axis xyz="0 0 1"/>
-    <limit lower="-4.71238898" upper="4.71238898" effort="500" velocity="2"/>
-    <dynamics damping="0.5" friction="0.3"/>
-  </joint>
-  <!-- ===================== FRONT RIGHT WHEEL ===================== -->
-  <link name="fr_wheel_link">
-    <inertial>
-      <origin xyz="0 0 0" rpy="0 0 0"/>
-      <mass value="0.5"/>
-      <inertia ixx="0.00563" iyy="0.00563" izz="0.01125" ixy="0" ixz="0" iyz="0"/>
-    </inertial>
-    <visual>
-      <origin xyz="0 0.06 0" rpy="-1.5708 0 3.14159"/>
-      <geometry>
-        <mesh filename="package://rover_description/meshes/suspension/wheel.stl" scale="0.001 0.001 0.001"/>
-      </geometry>
-      <material name="dark_wheel"/>
-    </visual>
-    <collision>
-      <origin xyz="0 0 0" rpy="-1.5708 0 0"/>
-      <geometry>
-        <cylinder radius="0.15" length="0.12"/>
-      </geometry>
-    </collision>
-  </link>
-  <joint name="fr_wheel_joint" type="continuous">
-    <parent link="fr_wheel_mount_link"/>
-    <child link="fr_wheel_link"/>
-    <origin xyz="0 0 -0.27" rpy="0 0 0"/>
-    <axis xyz="0 1 0"/>
-    <limit effort="100" velocity="10"/>
-  </joint>
-  <!-- ===================== BACK LEFT WHEEL MOUNT ===================== -->
-  <link name="bl_wheel_mount_link">
-    <inertial>
-      <origin xyz="0 0 0" rpy="0 0 0"/>
-      <mass value="0.162"/>
-      <inertia ixx="0.0002" iyy="0.00012" izz="0.00012" ixy="0" ixz="0" iyz="0"/>
-    </inertial>
-    <visual>
-      <origin xyz="0 -0.06 -0.269" rpy="0 0 0"/>
-      <geometry>
-        <mesh filename="package://rover_description/meshes/suspension/wheel_mount.stl" scale="0.001 0.001 0.001"/>
-      </geometry>
-      <material name="orange_mount"/>
-    </visual>
-    <collision>
-      <origin xyz="0 0.11125 -0.18" rpy="0 0 0"/>
-      <geometry>
-        <box size="0.07 0.0625 0.25"/>
-      </geometry>
-    </collision>
-  </link>
-  <joint name="bl_wheel_mount_joint" type="revolute">
-    <parent link="l_rocker_link"/>
-    <child link="bl_wheel_mount_link"/>
-    <origin xyz="-0.421 0 0" rpy="0 0 0"/>
-    <axis xyz="0 0 1"/>
-    <limit lower="-4.71238898" upper="4.71238898" effort="500" velocity="2"/>
-    <dynamics damping="0.5" friction="0.3"/>
-  </joint>
-  <!-- ===================== BACK LEFT WHEEL ===================== -->
-  <link name="bl_wheel_link">
-    <inertial>
-      <origin xyz="0 0 0" rpy="0 0 0"/>
-      <mass value="0.5"/>
-      <inertia ixx="0.00563" iyy="0.00563" izz="0.01125" ixy="0" ixz="0" iyz="0"/>
-    </inertial>
-    <visual>
-      <origin xyz="0 -0.06 0" rpy="-1.5708 0 0"/>
-      <geometry>
-        <mesh filename="package://rover_description/meshes/suspension/wheel.stl" scale="0.001 0.001 0.001"/>
-      </geometry>
-      <material name="dark_wheel"/>
-    </visual>
-    <collision>
-      <origin xyz="0 0 0" rpy="1.5708 0 0"/>
-      <geometry>
-        <cylinder radius="0.15" length="0.12"/>
-      </geometry>
-    </collision>
-  </link>
-  <joint name="bl_wheel_joint" type="continuous">
-    <parent link="bl_wheel_mount_link"/>
-    <child link="bl_wheel_link"/>
-    <origin xyz="0 0 -0.27" rpy="0 0 0"/>
-    <axis xyz="0 1 0"/>
-    <limit effort="100" velocity="10"/>
-  </joint>
-  <!-- ===================== BACK RIGHT WHEEL MOUNT ===================== -->
-  <link name="br_wheel_mount_link">
-    <inertial>
-      <origin xyz="0 0 0" rpy="0 0 0"/>
-      <mass value="0.162"/>
-      <inertia ixx="0.0002" iyy="0.00012" izz="0.00012" ixy="0" ixz="0" iyz="0"/>
-    </inertial>
-    <visual>
-      <origin xyz="0 0.06 -0.269" rpy="0 0 3.14159"/>
-      <geometry>
-        <mesh filename="package://rover_description/meshes/suspension/wheel_mount.stl" scale="0.001 0.001 0.001"/>
-      </geometry>
-      <material name="orange_mount"/>
-    </visual>
-    <collision>
-      <origin xyz="0 -0.11125 -0.18" rpy="0 0 0"/>
-      <geometry>
-        <box size="0.07 0.0625 0.25"/>
-      </geometry>
-    </collision>
-  </link>
-  <joint name="br_wheel_mount_joint" type="revolute">
-    <parent link="r_rocker_link"/>
-    <child link="br_wheel_mount_link"/>
-    <origin xyz="-0.421 0 0" rpy="0 0 0"/>
-    <axis xyz="0 0 1"/>
-    <limit lower="-4.71238898" upper="4.71238898" effort="500" velocity="2"/>
-    <dynamics damping="0.5" friction="0.3"/>
-  </joint>
-  <!-- ===================== BACK RIGHT WHEEL ===================== -->
-  <link name="br_wheel_link">
-    <inertial>
-      <origin xyz="0 0 0" rpy="0 0 0"/>
-      <mass value="0.5"/>
-      <inertia ixx="0.00563" iyy="0.00563" izz="0.01125" ixy="0" ixz="0" iyz="0"/>
-    </inertial>
-    <visual>
-      <origin xyz="0 0.06 0" rpy="-1.5708 0 3.14159"/>
-      <geometry>
-        <mesh filename="package://rover_description/meshes/suspension/wheel.stl" scale="0.001 0.001 0.001"/>
-      </geometry>
-      <material name="dark_wheel"/>
-    </visual>
-    <collision>
-      <origin xyz="0 0 0" rpy="-1.5708 0 0"/>
-      <geometry>
-        <cylinder radius="0.15" length="0.12"/>
-      </geometry>
-    </collision>
-  </link>
-  <joint name="br_wheel_joint" type="continuous">
-    <parent link="br_wheel_mount_link"/>
-    <child link="br_wheel_link"/>
-    <origin xyz="0 0 -0.27" rpy="0 0 0"/>
-    <axis xyz="0 1 0"/>
-    <limit effort="100" velocity="10"/>
-  </joint>
+  <!-- ===================== ROCKERS + WHEELS ===================== -->
+  <xacro:rocker_assembly side="l" y_sign="1"/>
+  <xacro:rocker_assembly side="r" y_sign="-1"/>
+  <!-- ===================== ACCESSORIES ===================== -->
+  <xacro:towerlight_accessory suffix="l" y_sign="1"/>
+  <xacro:towerlight_accessory suffix="r" y_sign="-1"/>
+  <xacro:stop_button_accessory suffix="l" y_sign="1"/>
+  <xacro:stop_button_accessory suffix="r" y_sign="-1"/>
   <!-- ===================== ARM (OPTIONAL) ===================== -->
   <!-- Placeholder mount pose; update once the real MR_ARM_ATT attachment

Commit message: Feature/arm/panel integration (#517)
* feat(panel): switch panel description, bringup and sim packages

* feat(panel): color-code panel elements and add indicators/sockets/markers

* fix(rover): sync rover_description with develop, keep arm mount + accessories

* fix(panel): sync Gazebo spawn pose with TF, add frame_prefix, fix breaker limits

---------

Co-authored-by: Martik-k <kosiv.marta@gmail.com>

File: src/arm/arm_description/urdf/arm_macro.xacro (robot description, xacro)
@@ -4,4 +4,12 @@
   <xacro:arg name="end_effector" default="jaw"/>
   <xacro:arg name="sim" default="false"/>
+  <!-- When the arm is mounted into another robot's URDF (e.g. the rover, see
+       rover_description's mount_arm arg) that outer URDF already adds its
+       own single gz_ros2_control-system plugin covering every <ros2_control>
+       block in the combined model. Set this to false in that case so the
+       arm doesn't register a second, redundant controller_manager plugin
+       for the same Gazebo model. Standalone arm sim (arm_sim) leaves this
+       at the default so it keeps adding its own plugin as before. -->
+  <xacro:arg name="standalone_gz_plugin" default="true"/>
   <!-- camera:=false drops the simulated camera sensor (the URDF link and
        frames stay). Camera rendering is the main real-time-factor cost
@@ -276,9 +284,11 @@
     </ros2_control>
     <xacro:if value="$(arg sim)">
-      <gazebo>
-        <plugin filename="gz_ros2_control-system" name="gz_ros2_control::GazeboSimROS2ControlPlugin">
-          <parameters>$(find arm_sim)/config/ros2_controllers.yaml</parameters>
-        </plugin>
-      </gazebo>
+      <xacro:if value="$(arg standalone_gz_plugin)">
+        <gazebo>
+          <plugin filename="gz_ros2_control-system" name="gz_ros2_control::GazeboSimROS2ControlPlugin">
+            <parameters>$(find arm_sim)/config/ros2_controllers.yaml</parameters>
+          </plugin>
+        </gazebo>
+      </xacro:if>
       <gazebo reference="arm_mount_link">
         <visual>

File: src/rover_description/urdf/rover.urdf.xacro (robot description, xacro)
@@ -6,4 +6,14 @@
   <xacro:include filename="$(find rover_description)/urdf/macros/accessories.xacro"/>
   <xacro:include filename="$(find rover_description)/urdf/camera.xacro"/>
+  <!-- mount_arm:=true bolts the indomitus_arm (arm_description) onto
+       main_body_link, matching the real hardware where the arm is
+       physically attached to the rover chassis. Defaults to false so
+       existing rover-only bringup/sim behavior is unchanged unless a
+       launch file opts in. The include is unconditional (it only defines
+       the indomitus_arm macro; no links/joints are created until it is
+       invoked below), so arm_description must be present in the overlay
+       the same way it already is for arm_bringup/arm_hardware_interface. -->
+  <xacro:include filename="$(find arm_description)/urdf/arm_macro.xacro"/>
+  <xacro:arg name="mount_arm" default="false"/>
   <!-- ===================== MATERIALS ===================== -->
   <material name="blue_body">
@@ -97,3 +107,11 @@
   <xacro:stop_button_accessory suffix="l" y_sign="1"/>
   <xacro:stop_button_accessory suffix="r" y_sign="-1"/>
+  <!-- ===================== ARM (OPTIONAL) ===================== -->
+  <!-- Placeholder mount pose; update once the real MR_ARM_ATT attachment
+       point from CAD is known. -->
+  <xacro:if value="$(arg mount_arm)">
+    <xacro:indomitus_arm parent_link="main_body_link">
+      <origin xyz="0.2 0 0.1" rpy="0 0 0"/>
+    </xacro:indomitus_arm>
+  </xacro:if>
 </robot>
