Commit message: Feature/arm/cartesian keyboard teleop (#525)
* feature: implement initial hardware interface for CAN motors

* fix: correct steadywin_protocol.hpp and hardware interface

* old testing

* feature: synchronized 20-23 motors in visualization and in reality, made a safe launch of the launch file

* Feature/suspension/current voltage viz (#496)

* feature: add plotjuggler for current and voltage visualization

* feature: add power node; add launch and config files for power node; rename launch in rover_viz

* fix: move luanch file to proper directory

* fix: add better layour in plotjuggler

* feature: add launch_utils.py for common code in launch files; add power_monitor.launch in bringup

* fix: minor fixes in shutdown pipeline and dependencies

* chore: little fixes

* feat(arm): adopt new mesh set — geometry, jaw gripper, camera

* fix(arm): re-flashed Damiao Master ID, boolean param parsing, clean shutdown holds instead of disabling

* feat(arm): static gravity compensation (feed-forward torque)

* chore(arm): recalibrate direction/offset/kp/kd for new mesh; enable gravity_ff params.

* feat(arm): loosen goal tolerances found too tight for real-hardware transients

* fix(arm): give the jaw gripper finger its own mock hardware component

* feat(arm): tune gains, split gravity clamps per motor family, fix velocity tolerance

* chore(arm): stable version

* fix(arm): zero-torque MIT frame in disable_motors.py, fix Steadywin T_MAX mismatch

* fix(arm): OMPL/TOTG smoothing, Servo joint limits, position deadband — still jittery

* fix(arm): rotate joystick servo about TCP, not a wrist joint

Drop the 0.005 rad command deadband that zeroed coordinated Cartesian steps, and send roll as twist.angular.x instead of JointJog on the last wrist axis.

* Revert "fix(arm): rotate joystick servo about TCP, not a wrist joint"

This reverts commit ff36058e6bd945e1d1b444f37b6cac071d7dd6a2.

* feat(arm): Cartesian keyboard/gamepad teleop with streaming Servo

Keep TCP translation in the mount frame and a large enough joint step
for +X on hardware; hold TCP attitude during Q/E without slowing XYZ.

* Add Cartesian keyboard/gamepad teleop via MoveIt Servo on the streaming controller.

Keep demo.launch and input nodes separate; document WASD/Stadia mapping and Servo/JTC switch.

* fix(arm): restore python3-evdev dependency for kayboard_servo_node

* feat(arm): view-relative EEF translation on arrows + T/G and add camera-frame translation keys to keyboard teleop

* fix(arm): view-relative gamepad teleop with configurable shift button, and round motor position packing instead of truncating

* fix(arm): close home/exit race in keyboard teleop

* fix(arm): sync Steadywin P_MAX across calibration/sim tools with steadywin_protocol.hpp

* fix(arm): refuse to run direct-CAN scripts while ros2_control is active

* docs(arm): document that Ctrl+C leaves motors holding, not disabled

* fix(arm): strict controller handoff, Gazebo/demo.launch.py parity, honest home pose

* fix(arm): sync calibration directions, teach_poses portability, doc accuracy

* fix(arm): skip STRICT switch_controller calls already in the target state

---------

Co-authored-by: Yurii Fito <fito.pn@ucu.edu.ua>
Co-authored-by: OShevchuk-UCU <o.shevchuk@ucu.edu.ua>

File: src/arm/arm_description/urdf/arm_macro.xacro (robot description, xacro)
@@ -64,5 +64,5 @@
       <parent link="arm_base_link"/>
       <child link="arm_shoulder_link"/>
-      <origin xyz="-0.040366 -0.000325 0.103" rpy="${pi/6} 0 ${-pi}"/>
+      <origin xyz="-0.040366 -0.000325 0.103" rpy="${pi/3} 0 ${-pi}"/>
       <axis xyz="1 0 0"/>
       <limit lower="${-pi}" upper="${pi}" effort="100.0" velocity="1.0"/>
@@ -81,5 +81,5 @@
       <parent link="arm_shoulder_link"/>
       <child link="arm_forearm_link"/>
-      <origin xyz="0 0.3 0" rpy="${5*pi/6} 0 0"/>
+      <origin xyz="0 0.3 0" rpy="${5*pi/12} 0 0"/>
       <axis xyz="1 0 0"/>
       <limit lower="${-pi/2}" upper="${pi/2}" effort="100.0" velocity="1.0"/>
@@ -132,5 +132,5 @@
       <parent link="arm_wrist_2_link"/>
       <child link="arm_end_effector_link"/>
-      <origin xyz="0.0323 0 -0.035" rpy="${pi/2} 0 ${pi/2}"/>
+      <origin xyz="0.0323 0 -0.035" rpy="${-pi/2} ${pi/2} ${-pi/2}"/>
       <axis xyz="0 0 1"/>
       <limit lower="${-pi}" upper="${pi}" effort="100.0" velocity="1.0"/>
@@ -244,8 +244,36 @@
             <plugin>arm_hardware_interface/ArmCanSystem</plugin>
             <param name="can_interface">can0</param>
+            <!-- Stiffness ramps 0 -> 100% over this many seconds after activation -->
+            <param name="gain_ramp_secs">15.0</param>
+            <!-- Hard rate limiter on outgoing position commands (rad/s) —
+                 even a wrong/hostile command can't move a joint faster than this. -->
+            <param name="max_cmd_speed_rad_s">1.0</param>
+            <!-- Activation aborts if any motor is silent for this long -->
+            <param name="feedback_timeout_secs">2.0</param>
+            <param name="gravity_ff_enabled">true</param>
+            <!-- ~3.8 kg hangs below the shoulder with its COM ~0.3 m out, so the
+                 holding torque there reaches ~11 Nm on extended poses. The two
+                 motor families are an order of magnitude apart: Steadywin is
+                 rated 48 Nm, Damiao only 9 Nm continuous. -->
+            <param name="gravity_ff_max_nm_steadywin">20.0</param>
+            <param name="gravity_ff_max_nm_damiao">6.0</param>
           </xacro:unless>
         </xacro:unless>
       </hardware>
-      <xacro:macro name="arm_joint_control" params="joint_name">
+      <!-- ======================= CALIBRATION =======================
+           direction : +1 if pushing the joint in its URDF-positive direction
+                       (right-hand rule about the <axis>) makes the RAW motor
+                       angle increase; -1 otherwise.
+           offset    : the RAW motor angle (rad) measured when the arm is
+                       physically in the URDF zero pose. If you save the motor
+                       zero (0xB1 / FF..FE) at that pose, offset = 0.0.
+           kp / kd   : MIT gains, tuned on real hardware. The protocol packs
+                       these into 12 bits over [0,500] and [0,5], and anything
+                       above those is clamped silently — a kd of 6 reads back
+                       as 5 with no warning anywhere.
+           Re-verify with scripts/check_calibration.py (torqueless) after any
+           mesh/geometry change that alters a joint's <axis>.
+           ============================================================= -->
+      <xacro:macro name="arm_joint_control" params="joint_name motor_id direction offset kp kd">
         <joint name="${joint_name}">
           <command_interface name="position">
@@ -253,24 +281,27 @@
             <param name="max">${pi}</param>
           </command_interface>
+          <command_interface name="velocity"/>
           <state_interface name="position"/>
           <state_interface name="velocity"/>
+          <param name="motor_id">${motor_id}</param>
+          <param name="direction">${direction}</param>
+          <param name="offset">${offset}</param>
+          <param name="kp">${kp}</param>
+          <param name="kd">${kd}</param>
         </joint>
       </xacro:macro>
-      <xacro:arm_joint_control joint_name="arm_mount_base_joint"/>
-      <xacro:arm_joint_control joint_name="arm_base_shoulder_joint"/>
-      <xacro:arm_joint_control joint_name="arm_shoulder_forearm_joint"/>
-      <xacro:arm_joint_control joint_name="arm_forearm_wrist_1_joint"/>
-      <xacro:arm_joint_control joint_name="arm_wrist_1_wrist_2_joint"/>
-      <xacro:arm_joint_control joint_name="arm_wrist_2_end_effector_joint"/>
-      <!-- Only the right finger joint needs a ros2_control interface: the
-           left one is a <mimic> of it, computed automatically (by
-           robot_state_publisher for TF, and by the planning scene monitor
-           for collision state) from the right joint's reported position —
-           it doesn't need its own state/command interface. Without this,
-           joint_state_broadcaster never reports arm_jaw_gripper_finger_right_joint
-           at all, and the planning scene monitor (used by both move_group
-           and Servo) considers the robot's state permanently incomplete,
-           which silently blocks all motion. -->
-      <xacro:if value="${'$(arg end_effector)' == 'jaw'}">
+      <!-- MIT gains: protocol max kp=500, kd=5. Steadywin at ceiling to hold
+           gravity; Damiao a step below to reduce wrist oscillation while stiff. -->
+      <xacro:arm_joint_control joint_name="arm_mount_base_joint"          motor_id="20" direction="-1" offset="0.0"  kp="500.0" kd="5.0"/>
+      <xacro:arm_joint_control joint_name="arm_base_shoulder_joint"       motor_id="21" direction="1"  offset="0.0"  kp="500.0" kd="5.0"/>
+      <xacro:arm_joint_control joint_name="arm_shoulder_forearm_joint"    motor_id="22" direction="-1" offset="0.0"  kp="500.0" kd="5.0"/>
+      <xacro:arm_joint_control joint_name="arm_forearm_wrist_1_joint"     motor_id="23" direction="-1" offset="0.0"  kp="400.0" kd="5.0"/>
+      <xacro:arm_joint_control joint_name="arm_wrist_1_wrist_2_joint"     motor_id="24" direction="-1" offset="0.0"  kp="400.0" kd="5.0"/>
+      <xacro:arm_joint_control joint_name="arm_wrist_2_end_effector_joint" motor_id="25" direction="1"  offset="0.0"  kp="350.0" kd="5.0"/>
+      <!-- Only the right finger needs an interface: left is a <mimic> of it.
+           Excluded on real hardware — ArmCanSystem hardcodes NUM_JOINTS=6 and
+           would fail with "Expected 6 joints, got 7"; the JawGripperStub
+           component below covers that case instead. -->
+      <xacro:if value="${('$(arg end_effector)' == 'jaw') and (('$(arg sim)' == 'true') or ('$(arg use_fake_hardware)' == 'true'))}">
         <joint name="arm_jaw_gripper_finger_right_joint">
           <command_interface name="position">
@@ -283,4 +314,28 @@
       </xacro:if>
     </ros2_control>
+    <!-- There is no gripper motor on the real arm yet, but the finger joint must
+         still report state: without it joint_state_broadcaster never publishes
+         the joint, the planning scene monitor sees an incomplete robot state,
+         and move_group/Servo silently refuse to move. GenericSystem echoes
+         commands back as state, so the joint exists for MoveIt while nothing
+         physical moves. Replace with the real gripper hardware plugin once the
+         motor is wired up. -->
+    <xacro:if value="${('$(arg end_effector)' == 'jaw') and ('$(arg sim)' == 'false') and ('$(arg use_fake_hardware)' == 'false')}">
+      <ros2_control name="JawGripperStub" type="system">
+        <hardware>
+          <plugin>mock_components/GenericSystem</plugin>
+        </hardware>
+        <joint name="arm_jaw_gripper_finger_right_joint">
+          <command_interface name="position">
+            <param name="min">0</param>
+            <param name="max">${finger_stroke}</param>
+          </command_interface>
+          <state_interface name="position">
+            <param name="initial_value">0.0</param>
+          </state_interface>
+          <state_interface name="velocity"/>
+        </joint>
+      </ros2_control>
+    </xacro:if>
     <xacro:if value="$(arg sim)">
       <xacro:if value="$(arg standalone_gz_plugin)">

Commit message: feat(arm): swap gripper mesh to v3, fix TCP/camera geometry to match

File: src/arm/arm_description/urdf/arm_macro.xacro (robot description, xacro)
@@ -139,9 +139,9 @@
       <xacro:if value="${'$(arg end_effector)' == 'jaw'}">
         <visual>
-          <geometry><mesh filename="${mesh_path}/arm_jaw_gripper_v2.stl" scale="${stl_scale}"/></geometry>
+          <geometry><mesh filename="${mesh_path}/arm_jaw_gripper_v3.stl" scale="${stl_scale}"/></geometry>
           <material name="light_grey"/>
         </visual>
         <collision>
-          <geometry><mesh filename="${mesh_path}/arm_jaw_gripper_v2.stl" scale="${stl_scale}"/></geometry>
+          <geometry><mesh filename="${mesh_path}/arm_jaw_gripper_v3.stl" scale="${stl_scale}"/></geometry>
         </collision>
       </xacro:if>
@@ -151,14 +151,35 @@
     </link>
     <xacro:if value="${'$(arg end_effector)' == 'jaw'}">
-      <!-- From CAD, origin of each finger relative to gripper origin (mm):
-           finger 1 (right): closed (3.5, -10.72, 122.133)  -> open (15.5, -10.72, 122.133)
-           finger 2 (left):  closed (-3.5, 13.78, 122.133)  -> open (-15.5, 13.78, 122.133)
-           X is symmetric (+-3.5mm closed, +-12mm stroke); Y is NOT mirrored between the two
-           fingers on purpose (offset so the finger pads clear each other near full close). -->
-      <xacro:property name="finger_x_closed" value="-0.0035"/>
+      <!-- v3: no CAD dimension doc available (unlike v2 above). Derived from
+           the STL geometry itself: arm_jaw_gripper_finger_v3.stl is exported
+           in the gripper's own assembly frame (same frame as
+           arm_jaw_gripper_v3.stl), not in a per-part local frame like v2 was.
+           Its bbox (X[-48.83,11] Y[-16.91,14.08] Z[53,161.52]mm) already sits
+           correctly relative to the body bbox (Z[0,76]mm, overlap 53-76mm =
+           mechanism recessed into the body, 76-161.5mm = fingers protruding)
+           when placed with a plain identity origin. Stroke has no v3 source
+           of truth yet, kept at the v2 value pending visual confirmation of
+           open/close range in sim.
+           finger_x_closed is NOT zero, unlike the rest: mirroring the mesh
+           180 deg about Z at a plain (0,0,0) origin left a real 31.55mm gap
+           between the two finger surfaces at rest (measured as the true
+           nearest-neighbor distance between arm_jaw_gripper_finger_v3.stl's
+           own vertex cloud and its mirrored copy, not just a bbox estimate,
+           which undercounted it); closed did not mean touching. Each side
+           is shifted inward by half that gap (15.775mm). A deliberate
+           overlap (0.016, ~0.45mm interference) was tried first for a
+           solid-looking contact, but under real Gazebo physics (not the
+           fake-hardware mock, which has no collision checking) the
+           interpenetrating collision meshes deadlocked the prismatic
+           joint against its own contact force and the gripper could not
+           open at all — confirmed by commanding gripper_controller with
+           the arm actually spawned in gz-sim and watching /joint_states
+           stay pinned at 0. 0.0155 leaves a ~0.55mm gap instead: visually
+           still reads as closed, but with no interpenetration to jam on. -->
+      <xacro:property name="finger_x_closed" value="0.0155"/>
       <xacro:property name="finger_stroke" value="0.012"/>
-      <xacro:property name="finger_z" value="0.122133"/>
-      <xacro:property name="finger_right_y" value="0.01072"/>
-      <xacro:property name="finger_left_y" value="-0.01378"/>
+      <xacro:property name="finger_z" value="0.0"/>
+      <xacro:property name="finger_right_y" value="0.0"/>
+      <xacro:property name="finger_left_y" value="0.0"/>
       <xacro:macro name="jaw_gripper_finger" params="side x_closed y yaw axis_sign limit_lower limit_upper">
         <joint name="arm_jaw_gripper_finger_${side}_joint" type="prismatic">
@@ -172,8 +193,5 @@
                  point opposite ways in the parent frame — multiplier=-1.0 makes
                  them slide apart symmetrically as the right joint opens, rather
-                 than translating together with a fixed gap. Left's own range is
-                 shifted negative to match, since its opening motion is the
-                 mirror of right's (mimic must stay within the child's own
-                 declared limits). -->
+                 than translating together with a fixed gap. -->
             <mimic joint="arm_jaw_gripper_finger_right_joint" multiplier="-1.0" offset="0.0"/>
           </xacro:unless>
@@ -181,9 +199,9 @@
         <link name="arm_jaw_gripper_finger_${side}_link">
           <visual>
-            <geometry><mesh filename="${mesh_path}/arm_jaw_gripper_finger_v2.stl" scale="${stl_scale}"/></geometry>
+            <geometry><mesh filename="${mesh_path}/arm_jaw_gripper_finger_v3.stl" scale="${stl_scale}"/></geometry>
             <material name="light_grey"/>
           </visual>
           <collision>
-            <geometry><mesh filename="${mesh_path}/arm_jaw_gripper_finger_v2.stl" scale="${stl_scale}"/></geometry>
+            <geometry><mesh filename="${mesh_path}/arm_jaw_gripper_finger_v3.stl" scale="${stl_scale}"/></geometry>
           </collision>
           <xacro:dummy_inertia mass="0.05"/>
@@ -199,5 +217,13 @@
       <child link="arm_tcp_link"/>
       <xacro:if value="${'$(arg end_effector)' == 'jaw'}">
-        <origin xyz="0 -0.0015 0.2072" rpy="0 0 0"/>
+        <!-- v3: X=Y=0 by construction (right/left fingers are the same mesh
+             mirrored 180 deg about Z through the shared origin, see the
+             finger properties comment above, so that origin is the natural
+             symmetric grasp centerline). Z = max Z of
+             arm_jaw_gripper_finger_v3.stl (161.5187mm, fingertip reach in
+             the shared assembly frame); same derivation the old v2 value
+             used (finger_z + finger local Z max), simplified here since
+             finger_z is now 0. -->
+        <origin xyz="0 0 0.1615" rpy="0 0 0"/>
       </xacro:if>
       <xacro:if value="${'$(arg end_effector)' != 'jaw'}">
@@ -209,10 +235,20 @@
       <parent link="arm_end_effector_link"/>
       <child link="arm_camera_link"/>
-      <origin xyz="0.0012604892253875732 -0.045 0.07839690148830414" rpy="0 ${-pi/2} ${pi/2}"/>
+      <!-- Ground truth click on the mount recess: (2.47, 21.72, 23.86)mm
+           surface point (see history above/git log for the RViz Publish
+           Point capture). Y is offset from that surface point by the
+           box's own half-extent along the axis that actually faces this
+           direction: arm_camera_link's local Z maps to global -Y here (see
+           the rpy below, unchanged throughout), and local Z is the box's
+           HEIGHT dimension (third size number below); keep this offset
+           at HALF THE CURRENT HEIGHT whenever that size number changes, or
+           the box either gaps off the surface or buries into it. Currently
+           0.05m tall -> 25mm half-extent -> Y = 21.72 + 25 = 46.72mm. -->
+      <origin xyz="0.00247 0.04672 0.02386" rpy="0 ${-pi/2} ${pi/2}"/>
     </joint>
     <link name="arm_camera_link">
       <visual>
         <geometry>
-          <box size="0.06 0.06 0.06"/>
+          <box size="0.035 0.035 0.05"/>
         </geometry>
         <material name="camera_blue">
@@ -222,5 +258,5 @@
       <collision>
         <geometry>
-          <box size="0.06 0.06 0.06"/>
+          <box size="0.035 0.035 0.05"/>
         </geometry>
       </collision>
@@ -229,5 +265,20 @@
       <parent link="arm_camera_link"/>
       <child link="arm_camera_optical_frame"/>
-      <origin xyz="0.045 0 0" rpy="${-pi/2} 0 ${-pi/2}"/>
+      <!-- 0.045 was sized for the old 60mm camera box (half-extent 30mm)
+           and never revisited when the box shrank to 35mm; it put the
+           lens 45mm out along camera_link's local +X (= +Z in
+           arm_end_effector_link), landing deep inside the v3 gripper body
+           instead of at the box's own front face. An actual captured
+           /camera/image_raw frame confirmed this: flat solid grey, the lens
+           pressed against the body's own material. Set to 0.0175, the
+           current box's half-extent, so the lens sits flush with its front
+           face instead of floating 27.5mm past it. rpy confirmed 180 deg
+           rolled from a live captured frame (fingers rendered correctly
+           shaped but upside down); flipping the sign of roll and yaw
+           (pitch stays 0) is an exact 180 deg roll about the optical Z
+           (viewing) axis: verified by matrix multiplication that the
+           combined camera_joint*optical_joint rotation keeps the same +Z
+           forward direction with X/Y both negated, not a re-aim. -->
+      <origin xyz="0.0175 0 0" rpy="${pi/2} 0 ${pi/2}"/>
     </joint>
     <link name="arm_camera_optical_frame"/>
@@ -432,5 +483,14 @@
       <gazebo reference="arm_camera_link">
         <sensor name="arm_camera" type="camera">
-          <pose>0.045 0 0 0 0 0</pose>
+          <!-- This is the pose gz-sim actually renders from, separate
+               from, and NOT driven by, arm_camera_optical_joint's TF chain
+               (that joint only labels frame_id for ROS consumers via
+               optical_frame_id below; editing its rpy alone was verified,
+               via repeated live-captured /camera/image_raw frames, to have
+               zero effect on the rendered image). X was the same stale
+               0.045 (old 60mm box) bug as arm_camera_optical_joint had;
+               fixed to 0.0175 (current box half-extent). Roll=pi added
+               here to fix the confirmed 180 deg upside-down image. -->
+          <pose>0.0175 0 0 3.14159265 0 0</pose>
           <camera>
             <optical_frame_id>arm_camera_optical_frame</optical_frame_id>
