Commit message: fix(arm): correct v3 gripper closed-gap value, exclude finger self-collision

File: src/arm/arm_description/urdf/arm_macro.xacro (robot description, xacro)
@@ -162,20 +162,42 @@
            open/close range in sim.
            finger_x_closed is NOT zero, unlike the rest: mirroring the mesh
-           180 deg about Z at a plain (0,0,0) origin left a real 31.55mm gap
-           between the two finger surfaces at rest (measured as the true
-           nearest-neighbor distance between arm_jaw_gripper_finger_v3.stl's
-           own vertex cloud and its mirrored copy, not just a bbox estimate,
-           which undercounted it); closed did not mean touching. Each side
-           is shifted inward by half that gap (15.775mm). A deliberate
-           overlap (0.016, ~0.45mm interference) was tried first for a
-           solid-looking contact, but under real Gazebo physics (not the
-           fake-hardware mock, which has no collision checking) the
-           interpenetrating collision meshes deadlocked the prismatic
-           joint against its own contact force and the gripper could not
-           open at all — confirmed by commanding gripper_controller with
-           the arm actually spawned in gz-sim and watching /joint_states
-           stay pinned at 0. 0.0155 leaves a ~0.55mm gap instead: visually
-           still reads as closed, but with no interpenetration to jam on. -->
-      <xacro:property name="finger_x_closed" value="0.0155"/>
+           180 deg about Z at a plain (0,0,0) origin leaves the two finger
+           surfaces apart at rest; closed did not mean touching.
+           Correction from review: the first pass here (0.0155) was based
+           on the GLOBAL nearest-neighbor point between the two mirrored
+           meshes, found at Z~82mm — that point is on an unrelated
+           mechanism/recess feature near the finger's base, not the actual
+           grasp surface, and only 0.55mm apart there says nothing about
+           the pads that actually contact an object.
+           Real Gazebo physics (not the fake-hardware mock, which has no
+           collision checking) was found to deadlock the prismatic joint
+           against its own contact force when the collision meshes
+           actually overlap — confirmed by commanding gripper_controller
+           with the arm spawned in gz-sim and watching /joint_states stay
+           pinned once that happened. Since that risk exists anywhere two
+           colliding meshes might touch, not just at the grasp pads, the
+           two finger links' collisions are excluded from each other
+           entirely via SDF collide_bitmask (see the gazebo reference
+           blocks below): they were never meant to bear force against one
+           another, only against a grasped object, so gz-sim simply never
+           runs contact resolution on that pair regardless of how much
+           their meshes overlap.
+           That removes any downside to closing further, which matters
+           because the grasp band (Z in [130,163]mm) is not a flat/parallel
+           pair of surfaces — a per-(Y,Z)-bin gap scan across it found the
+           raw (unshifted) gap ranges from 34.48mm at its tightest ridge up
+           to 76.6mm at its loosest (a curved outer edge). Pushing the
+           offset past the tightest ridge to close more of that spread
+           (tried: half the 90th-percentile raw gap, 20.284mm) was checked
+           visually in Gazebo and rejected — at that offset the fingers
+           visibly overlap/cross each other rather than sit closed, because
+           the mesh's curvature means "more closed" past the ridge stops
+           looking like closing and starts looking like the two fingers
+           passing through one another. 17.24mm (closing only the tightest
+           ridge to ~0 gap) is the actual visual and mechanical maximum:
+           the rest of the nominal "grasp band" keeps a real, larger gap
+           because the mesh itself isn't flat there, not because of a
+           leftover safety margin. -->
+      <xacro:property name="finger_x_closed" value="0.01724"/>
       <xacro:property name="finger_stroke" value="0.012"/>
       <xacro:property name="finger_z" value="0.0"/>
@@ -224,5 +246,12 @@
              the shared assembly frame); same derivation the old v2 value
              used (finger_z + finger local Z max), simplified here since
-             finger_z is now 0. -->
+             finger_z is now 0.
+             Confirmed intentional (review): this places the TCP at the
+             fingertip plane, not the grasp center, ~46mm further out than
+             v2's TCP. That's a real, correct consequence of v3's fingers
+             being physically shorter than v2's, not a calculation error;
+             the formula itself (finger_z + finger local Z max) is
+             unchanged from v2 and matches the SRDF's own tip_link
+             convention for arm_tcp_link (indomitus_arm.srdf). -->
         <origin xyz="0 0 0.1615" rpy="0 0 0"/>
       </xacro:if>
@@ -279,5 +308,16 @@
            (viewing) axis: verified by matrix multiplication that the
            combined camera_joint*optical_joint rotation keeps the same +Z
-           forward direction with X/Y both negated, not a re-aim. -->
+           forward direction with X/Y both negated, not a re-aim.
+           Confirmed intentional (review): this rpy and the Gazebo
+           <sensor><pose> roll fix below are two independently-derived
+           values, but were checked against each other with a ground-truth
+           test, not just re-derived on paper — projected a known mesh
+           vertex (right finger's outer edge) through the live TF chain and
+           the live /camera/camera_info K-matrix to a predicted pixel, then
+           marked that pixel on an actual captured /camera/image_raw frame.
+           The marker landed exactly on the finger's edge in the image, and
+           the rotation here is quaternion-derived so it cannot represent a
+           reflection, ruling out an X-inversion by construction, not just
+           by this one test. -->
       <origin xyz="0.0175 0 0" rpy="${pi/2} 0 ${pi/2}"/>
     </joint>
@@ -469,4 +509,23 @@
             </material>
           </visual>
+          <!-- Excludes right/left finger collision from each other only
+               (bitmasks share no bits: 0x01 & 0x02 = 0), while both keep
+               the default 0xff for every other collision (grasped object,
+               table, itself vs the rest of the arm), since 0x01 & 0xff and
+               0x02 & 0xff are both nonzero. Needed because finger_x_closed
+               below sets the two fingertip pads to physically touch at
+               full close, and letting gz-sim run real contact resolution
+               between two touching/overlapping meshes on this prismatic
+               joint was found to deadlock it (confirmed live: /joint_states
+               stayed pinned once that happened). The fingers were never
+               meant to exert force on each other, only on a grasped object,
+               so excluding just this one pair changes nothing functional. -->
+          <collision>
+            <surface>
+              <contact>
+                <collide_bitmask>0x01</collide_bitmask>
+              </contact>
+            </surface>
+          </collision>
         </gazebo>
         <gazebo reference="arm_jaw_gripper_finger_left_link">
@@ -478,4 +537,13 @@
             </material>
           </visual>
+          <!-- See arm_jaw_gripper_finger_right_link above: excludes this
+               pair from each other (0x01 & 0x02 = 0) only. -->
+          <collision>
+            <surface>
+              <contact>
+                <collide_bitmask>0x02</collide_bitmask>
+              </contact>
+            </surface>
+          </collision>
         </gazebo>
       </xacro:if>

Commit message: fix(arm): give gripper left finger its own ros2_control interface

File: src/arm/arm_description/urdf/arm_macro.xacro (robot description, xacro)
@@ -211,11 +211,21 @@
           <axis xyz="${axis_sign} 0 0"/>
           <limit lower="${limit_lower}" upper="${limit_upper}" effort="20.0" velocity="0.05"/>
-          <xacro:unless value="${side == 'right'}">
-            <!-- Right and left are mirror images (180 deg about Z), so their axes
-                 point opposite ways in the parent frame — multiplier=-1.0 makes
-                 them slide apart symmetrically as the right joint opens, rather
-                 than translating together with a fixed gap. -->
-            <mimic joint="arm_jaw_gripper_finger_right_joint" multiplier="-1.0" offset="0.0"/>
-          </xacro:unless>
+          <!-- Left used to be a <mimic> of right (multiplier=-1.0) instead of
+               having its own ros2_control interface below. Dropped: a <mimic>
+               joint has no state/command interface of its own, so
+               joint_state_broadcaster never publishes it and its real
+               simulated position is invisible to ROS entirely — RViz only
+               ever showed a value *computed* from right's reported position
+               via the mimic formula, never left's actual physics state. Under
+               a fast disturbance elsewhere in the kinematic chain, DART's
+               mimic constraint was found (via direct Gazebo Transport query,
+               bypassing ROS) to drift out of sync and permanently stick,
+               independently of right and with zero ROS-visible symptom —
+               Gazebo's own render showed the gripper open while RViz kept
+               showing it closed, from the exact same live state. Left is now
+               driven by its own explicit position command, kept in lockstep
+               with right by the code that commands both, so its real state
+               is both correctly closed-loop controlled and visible in
+               /joint_states like every other joint. -->
         </joint>
         <link name="arm_jaw_gripper_finger_${side}_link">
@@ -390,8 +400,11 @@
       <xacro:arm_joint_control joint_name="arm_wrist_1_wrist_2_joint"     motor_id="24" direction="-1" offset="0.0"  kp="400.0" kd="5.0"/>
       <xacro:arm_joint_control joint_name="arm_wrist_2_end_effector_joint" motor_id="25" direction="1"  offset="0.0"  kp="350.0" kd="5.0"/>
-      <!-- Only the right finger needs an interface: left is a <mimic> of it.
-           Excluded on real hardware — ArmCanSystem hardcodes NUM_JOINTS=6 and
-           would fail with "Expected 6 joints, got 7"; the JawGripperStub
-           component below covers that case instead. -->
+      <!-- Both fingers get their own interface — left used to be a bare
+           <mimic> of right with no ros2_control entry, which made its real
+           simulated state invisible to ROS (see the joint definition above
+           for the full story of why that was dropped). Excluded on real
+           hardware — ArmCanSystem hardcodes NUM_JOINTS=6 and would fail with
+           "Expected 6 joints, got 7"; the JawGripperStub component below
+           covers that case instead. -->
       <xacro:if value="${('$(arg end_effector)' == 'jaw') and (('$(arg sim)' == 'true') or ('$(arg use_fake_hardware)' == 'true'))}">
         <joint name="arm_jaw_gripper_finger_right_joint">
@@ -399,4 +412,12 @@
             <param name="min">0</param>
             <param name="max">${finger_stroke}</param>
+          </command_interface>
+          <state_interface name="position"/>
+          <state_interface name="velocity"/>
+        </joint>
+        <joint name="arm_jaw_gripper_finger_left_joint">
+          <command_interface name="position">
+            <param name="min">${-finger_stroke}</param>
+            <param name="max">0</param>
           </command_interface>
           <state_interface name="position"/>

Commit message: docs(arm): trim v3 gripper geometry comments to essentials

File: src/arm/arm_description/urdf/arm_macro.xacro (robot description, xacro)
@@ -163,40 +163,14 @@
            finger_x_closed is NOT zero, unlike the rest: mirroring the mesh
            180 deg about Z at a plain (0,0,0) origin leaves the two finger
-           surfaces apart at rest; closed did not mean touching.
-           Correction from review: the first pass here (0.0155) was based
-           on the GLOBAL nearest-neighbor point between the two mirrored
-           meshes, found at Z~82mm — that point is on an unrelated
-           mechanism/recess feature near the finger's base, not the actual
-           grasp surface, and only 0.55mm apart there says nothing about
-           the pads that actually contact an object.
-           Real Gazebo physics (not the fake-hardware mock, which has no
-           collision checking) was found to deadlock the prismatic joint
-           against its own contact force when the collision meshes
-           actually overlap — confirmed by commanding gripper_controller
-           with the arm spawned in gz-sim and watching /joint_states stay
-           pinned once that happened. Since that risk exists anywhere two
-           colliding meshes might touch, not just at the grasp pads, the
-           two finger links' collisions are excluded from each other
-           entirely via SDF collide_bitmask (see the gazebo reference
-           blocks below): they were never meant to bear force against one
-           another, only against a grasped object, so gz-sim simply never
-           runs contact resolution on that pair regardless of how much
-           their meshes overlap.
-           That removes any downside to closing further, which matters
-           because the grasp band (Z in [130,163]mm) is not a flat/parallel
-           pair of surfaces — a per-(Y,Z)-bin gap scan across it found the
-           raw (unshifted) gap ranges from 34.48mm at its tightest ridge up
-           to 76.6mm at its loosest (a curved outer edge). Pushing the
-           offset past the tightest ridge to close more of that spread
-           (tried: half the 90th-percentile raw gap, 20.284mm) was checked
-           visually in Gazebo and rejected — at that offset the fingers
-           visibly overlap/cross each other rather than sit closed, because
-           the mesh's curvature means "more closed" past the ridge stops
-           looking like closing and starts looking like the two fingers
-           passing through one another. 17.24mm (closing only the tightest
-           ridge to ~0 gap) is the actual visual and mechanical maximum:
-           the rest of the nominal "grasp band" keeps a real, larger gap
-           because the mesh itself isn't flat there, not because of a
-           leftover safety margin. -->
+           surfaces apart at rest, so each side is shifted inward. 17.24mm
+           brings the grasp band's tightest ridge (Z~130-163mm) to ~0 gap;
+           the rest of that band stays open because the mesh is curved,
+           not flat, there — pushing the offset further to close more of
+           it makes the fingers visibly cross rather than sit closed.
+           Collisions between the two finger links are excluded from each
+           other via SDF collide_bitmask (gazebo reference blocks below):
+           real Gazebo physics deadlocks the prismatic joint against its
+           own contact force when their meshes overlap, and they only
+           ever need to push against a grasped object, not each other. -->
       <xacro:property name="finger_x_closed" value="0.01724"/>
       <xacro:property name="finger_stroke" value="0.012"/>
@@ -211,21 +185,10 @@
           <axis xyz="${axis_sign} 0 0"/>
           <limit lower="${limit_lower}" upper="${limit_upper}" effort="20.0" velocity="0.05"/>
-          <!-- Left used to be a <mimic> of right (multiplier=-1.0) instead of
-               having its own ros2_control interface below. Dropped: a <mimic>
-               joint has no state/command interface of its own, so
-               joint_state_broadcaster never publishes it and its real
-               simulated position is invisible to ROS entirely — RViz only
-               ever showed a value *computed* from right's reported position
-               via the mimic formula, never left's actual physics state. Under
-               a fast disturbance elsewhere in the kinematic chain, DART's
-               mimic constraint was found (via direct Gazebo Transport query,
-               bypassing ROS) to drift out of sync and permanently stick,
-               independently of right and with zero ROS-visible symptom —
-               Gazebo's own render showed the gripper open while RViz kept
-               showing it closed, from the exact same live state. Left is now
-               driven by its own explicit position command, kept in lockstep
-               with right by the code that commands both, so its real state
-               is both correctly closed-loop controlled and visible in
-               /joint_states like every other joint. -->
+          <!-- Left was a <mimic> of right until a live disturbance test
+               (Gazebo Transport, bypassing ROS) caught DART's mimic
+               constraint drifting out of sync and sticking, invisibly to
+               ROS/RViz since a <mimic> joint has no state interface of
+               its own. Left now has its own ros2_control interface below
+               and is commanded in lockstep with right instead. -->
         </joint>
         <link name="arm_jaw_gripper_finger_${side}_link">
@@ -256,12 +219,10 @@
              the shared assembly frame); same derivation the old v2 value
              used (finger_z + finger local Z max), simplified here since
-             finger_z is now 0.
-             Confirmed intentional (review): this places the TCP at the
-             fingertip plane, not the grasp center, ~46mm further out than
-             v2's TCP. That's a real, correct consequence of v3's fingers
-             being physically shorter than v2's, not a calculation error;
-             the formula itself (finger_z + finger local Z max) is
-             unchanged from v2 and matches the SRDF's own tip_link
-             convention for arm_tcp_link (indomitus_arm.srdf). -->
+             finger_z is now 0. This places the TCP at the fingertip
+             plane, not the grasp center, ~46mm further out than v2's TCP
+             — a correct consequence of v3's fingers being physically
+             shorter than v2's, not a calculation error; the formula
+             itself is unchanged from v2 and matches the SRDF's own
+             tip_link convention for arm_tcp_link (indomitus_arm.srdf). -->
         <origin xyz="0 0 0.1615" rpy="0 0 0"/>
       </xacro:if>
@@ -319,15 +280,9 @@
            combined camera_joint*optical_joint rotation keeps the same +Z
            forward direction with X/Y both negated, not a re-aim.
-           Confirmed intentional (review): this rpy and the Gazebo
-           <sensor><pose> roll fix below are two independently-derived
-           values, but were checked against each other with a ground-truth
-           test, not just re-derived on paper — projected a known mesh
-           vertex (right finger's outer edge) through the live TF chain and
-           the live /camera/camera_info K-matrix to a predicted pixel, then
-           marked that pixel on an actual captured /camera/image_raw frame.
-           The marker landed exactly on the finger's edge in the image, and
-           the rotation here is quaternion-derived so it cannot represent a
-           reflection, ruling out an X-inversion by construction, not just
-           by this one test. -->
+           Verified against the Gazebo <sensor><pose> roll fix below with
+           a live pixel-projection test (TF chain + camera K-matrix
+           predicted a pixel that landed exactly on a known mesh point in
+           a captured frame); the rotation is also quaternion-derived, so
+           it cannot represent a reflection/X-inversion regardless. -->
       <origin xyz="0.0175 0 0" rpy="${pi/2} 0 ${pi/2}"/>
     </joint>
@@ -530,16 +485,7 @@
             </material>
           </visual>
-          <!-- Excludes right/left finger collision from each other only
-               (bitmasks share no bits: 0x01 & 0x02 = 0), while both keep
-               the default 0xff for every other collision (grasped object,
-               table, itself vs the rest of the arm), since 0x01 & 0xff and
-               0x02 & 0xff are both nonzero. Needed because finger_x_closed
-               below sets the two fingertip pads to physically touch at
-               full close, and letting gz-sim run real contact resolution
-               between two touching/overlapping meshes on this prismatic
-               joint was found to deadlock it (confirmed live: /joint_states
-               stayed pinned once that happened). The fingers were never
-               meant to exert force on each other, only on a grasped object,
-               so excluding just this one pair changes nothing functional. -->
+          <!-- Distinct bitmasks (0x01/0x02) exclude only this pair from
+               colliding with each other; both keep the default 0xff
+               against everything else (grasped object, environment). -->
           <collision>
             <surface>
