Commit message: fix(arm): pin gripper limit fix to physical joint stop, gate gripper spawn by hardware mode

File: src/arm/arm_description/urdf/arm_macro.xacro (robot description, xacro)
@@ -175,7 +175,13 @@
       <xacro:property name="finger_x_closed" value="0.01724"/>
       <xacro:property name="finger_stroke" value="0.012"/>
-      <!-- Declared joint/command_interface limit, wider than finger_stroke on
-           purpose — see the finger declarations below for why. -->
-      <xacro:property name="finger_limit_margin" value="${2 * finger_stroke}"/>
+      <!-- Small buffer past the real endpoints (0 and finger_stroke), wider
+           than finger_stroke on purpose — see the finger declarations
+           below for why. A/B/C-tested live (2026-08): padding only the
+           command_interface with the physical <joint><limit> left tight
+           did NOT fix the stuck-finger bug (gz_ros2_control had no effect
+           — DART's own joint stop, from the physical limit, is what the
+           finger was actually resting against); a small epsilon on the
+           physical limit itself did. -->
+      <xacro:property name="finger_limit_epsilon" value="0.002"/>
       <xacro:property name="finger_z" value="0.0"/>
       <xacro:property name="finger_right_y" value="0.0"/>
@@ -208,17 +214,16 @@
       <!-- Same part mounted twice: "left" is the "right" finger rotated 180 deg about Z,
            so both slide outward along their own local +X (axis) to open — no mirrored mesh needed.
-           Both use finger_limit_margin (2x finger_stroke), wider than either one's
-           actually-used range (right only ever commanded in [0, finger_stroke],
-           left in [-finger_stroke, 0] — see keyboard_servo_node.py), because
-           gz_ros2_control 0.7.20 was found (repeated fresh-instance trials) to
-           sometimes silently drop writes to a joint sitting at or very near its own
-           declared command_interface bound — both the 0 rest position and the
-           finger_stroke fully-open position are real endpoints a finger sits at
-           continuously, so neither can be left at the edge of the declared range.
-           Doubling the margin puts both comfortably in the interior; nothing in
-           this repo ever actually commands either finger outside its original,
-           narrower range regardless. -->
-      <xacro:jaw_gripper_finger side="right" x_closed="${finger_x_closed}"  y="${finger_right_y}" yaw="0"      axis_sign="-1" limit_lower="${-finger_limit_margin}" limit_upper="${finger_limit_margin}"/>
-      <xacro:jaw_gripper_finger side="left"  x_closed="${-finger_x_closed}" y="${finger_left_y}"  yaw="${pi}" axis_sign="1"  limit_lower="${-finger_limit_margin}" limit_upper="${finger_limit_margin}"/>
+           Both use finger_limit_epsilon padding past their real travel
+           (right only ever commanded in [0, finger_stroke], left in
+           [-finger_stroke, 0] — see keyboard_servo_node.py), because the
+           0 rest position and the finger_stroke fully-open position are
+           real endpoints a finger sits at continuously, and DART (Gazebo's
+           physics engine) was found to sometimes silently ignore further
+           position commands once a prismatic joint settles exactly on its
+           own <limit> joint stop. See finger_limit_epsilon's declaration
+           above for the A/B/C test that pinned this to the physical
+           <limit>, not the command_interface bound. -->
+      <xacro:jaw_gripper_finger side="right" x_closed="${finger_x_closed}"  y="${finger_right_y}" yaw="0"      axis_sign="-1" limit_lower="${-finger_limit_epsilon}" limit_upper="${finger_stroke + finger_limit_epsilon}"/>
+      <xacro:jaw_gripper_finger side="left"  x_closed="${-finger_x_closed}" y="${finger_left_y}"  yaw="${pi}" axis_sign="1"  limit_lower="${-finger_stroke - finger_limit_epsilon}" limit_upper="${finger_limit_epsilon}"/>
     </xacro:if>
     <joint name="arm_tcp_joint" type="fixed">
@@ -380,6 +385,6 @@
         <joint name="arm_jaw_gripper_finger_right_joint">
           <command_interface name="position">
-            <param name="min">${-finger_limit_margin}</param>
-            <param name="max">${finger_limit_margin}</param>
+            <param name="min">${-finger_limit_epsilon}</param>
+            <param name="max">${finger_stroke + finger_limit_epsilon}</param>
           </command_interface>
           <state_interface name="position"/>
@@ -388,6 +393,6 @@
         <joint name="arm_jaw_gripper_finger_left_joint">
           <command_interface name="position">
-            <param name="min">${-finger_limit_margin}</param>
-            <param name="max">${finger_limit_margin}</param>
+            <param name="min">${-finger_stroke - finger_limit_epsilon}</param>
+            <param name="max">${finger_limit_epsilon}</param>
           </command_interface>
           <state_interface name="position"/>

Commit message: Feature/arm/gripper control (#535)
* feat(arm): swap gripper mesh to v3, fix TCP/camera geometry to match

* fix(arm): correct v3 gripper closed-gap value, exclude finger self-collision

* fix(arm): give gripper left finger its own ros2_control interface

* docs(arm): trim v3 gripper geometry comments to essentials

* feat(arm): add gripper open/close via keyboard, widen finger command_interface bounds

* fix(arm): pin gripper limit fix to physical joint stop, gate gripper spawn by hardware mode

File: src/arm/arm_description/urdf/arm_macro.xacro (robot description, xacro)
@@ -175,4 +175,13 @@
       <xacro:property name="finger_x_closed" value="0.01724"/>
       <xacro:property name="finger_stroke" value="0.012"/>
+      <!-- Small buffer past the real endpoints (0 and finger_stroke), wider
+           than finger_stroke on purpose — see the finger declarations
+           below for why. A/B/C-tested live (2026-08): padding only the
+           command_interface with the physical <joint><limit> left tight
+           did NOT fix the stuck-finger bug (gz_ros2_control had no effect
+           — DART's own joint stop, from the physical limit, is what the
+           finger was actually resting against); a small epsilon on the
+           physical limit itself did. -->
+      <xacro:property name="finger_limit_epsilon" value="0.002"/>
       <xacro:property name="finger_z" value="0.0"/>
       <xacro:property name="finger_right_y" value="0.0"/>
@@ -204,7 +213,17 @@
       </xacro:macro>
       <!-- Same part mounted twice: "left" is the "right" finger rotated 180 deg about Z,
-           so both slide outward along their own local +X (axis) to open — no mirrored mesh needed. -->
-      <xacro:jaw_gripper_finger side="right" x_closed="${finger_x_closed}"  y="${finger_right_y}" yaw="0"      axis_sign="-1" limit_lower="0"                limit_upper="${finger_stroke}"/>
-      <xacro:jaw_gripper_finger side="left"  x_closed="${-finger_x_closed}" y="${finger_left_y}"  yaw="${pi}" axis_sign="1"  limit_lower="${-finger_stroke}" limit_upper="0"/>
+           so both slide outward along their own local +X (axis) to open — no mirrored mesh needed.
+           Both use finger_limit_epsilon padding past their real travel
+           (right only ever commanded in [0, finger_stroke], left in
+           [-finger_stroke, 0] — see keyboard_servo_node.py), because the
+           0 rest position and the finger_stroke fully-open position are
+           real endpoints a finger sits at continuously, and DART (Gazebo's
+           physics engine) was found to sometimes silently ignore further
+           position commands once a prismatic joint settles exactly on its
+           own <limit> joint stop. See finger_limit_epsilon's declaration
+           above for the A/B/C test that pinned this to the physical
+           <limit>, not the command_interface bound. -->
+      <xacro:jaw_gripper_finger side="right" x_closed="${finger_x_closed}"  y="${finger_right_y}" yaw="0"      axis_sign="-1" limit_lower="${-finger_limit_epsilon}" limit_upper="${finger_stroke + finger_limit_epsilon}"/>
+      <xacro:jaw_gripper_finger side="left"  x_closed="${-finger_x_closed}" y="${finger_left_y}"  yaw="${pi}" axis_sign="1"  limit_lower="${-finger_stroke - finger_limit_epsilon}" limit_upper="${finger_limit_epsilon}"/>
     </xacro:if>
     <joint name="arm_tcp_joint" type="fixed">
@@ -220,9 +239,10 @@
              used (finger_z + finger local Z max), simplified here since
              finger_z is now 0. This places the TCP at the fingertip
-             plane, not the grasp center, ~46mm further out than v2's TCP
-             — a correct consequence of v3's fingers being physically
-             shorter than v2's, not a calculation error; the formula
-             itself is unchanged from v2 and matches the SRDF's own
-             tip_link convention for arm_tcp_link (indomitus_arm.srdf). -->
+             plane, not the grasp center, ~46mm closer in (shorter reach)
+             than v2's TCP (0.1615 vs 0.2072) — a correct consequence of
+             v3's fingers being physically shorter than v2's, not a
+             calculation error; the formula itself is unchanged from v2
+             and matches the SRDF's own tip_link convention for
+             arm_tcp_link (indomitus_arm.srdf). -->
         <origin xyz="0 0 0.1615" rpy="0 0 0"/>
       </xacro:if>
@@ -365,6 +385,6 @@
         <joint name="arm_jaw_gripper_finger_right_joint">
           <command_interface name="position">
-            <param name="min">0</param>
-            <param name="max">${finger_stroke}</param>
+            <param name="min">${-finger_limit_epsilon}</param>
+            <param name="max">${finger_stroke + finger_limit_epsilon}</param>
           </command_interface>
           <state_interface name="position"/>
@@ -373,6 +393,6 @@
         <joint name="arm_jaw_gripper_finger_left_joint">
           <command_interface name="position">
-            <param name="min">${-finger_stroke}</param>
-            <param name="max">0</param>
+            <param name="min">${-finger_stroke - finger_limit_epsilon}</param>
+            <param name="max">${finger_limit_epsilon}</param>
           </command_interface>
           <state_interface name="position"/>

Commit message: feat(arm): gripper joint stub fix, torque logging, teleop push boost

File: src/arm/arm_description/urdf/arm_macro.xacro (robot description, xacro)
@@ -132,5 +132,5 @@
       <parent link="arm_wrist_2_link"/>
       <child link="arm_end_effector_link"/>
-      <origin xyz="0.0323 0 -0.035" rpy="${-pi/2} ${pi/2} ${-pi/2}"/>
+      <origin xyz="0.0323 0 -0.035" rpy="${-pi/2} ${pi/3} ${-pi/2}"/>
       <axis xyz="0 0 1"/>
       <limit lower="${-pi}" upper="${pi}" effort="100.0" velocity="1.0"/>
@@ -401,11 +401,11 @@
       </xacro:if>
     </ros2_control>
-    <!-- There is no gripper motor on the real arm yet, but the finger joint must
-         still report state: without it joint_state_broadcaster never publishes
-         the joint, the planning scene monitor sees an incomplete robot state,
-         and move_group/Servo silently refuse to move. GenericSystem echoes
-         commands back as state, so the joint exists for MoveIt while nothing
-         physical moves. Replace with the real gripper hardware plugin once the
-         motor is wired up. -->
+    <!-- There is no gripper motor on the real arm yet, but both finger joints
+         must still report state: without it joint_state_broadcaster never
+         publishes them, the planning scene monitor sees an incomplete robot
+         state, and move_group/Servo silently refuse to move. GenericSystem
+         echoes commands back as state, so both joints exist for MoveIt while
+         nothing physical moves. Replace with the real gripper hardware plugin
+         once the motor is wired up. -->
     <xacro:if value="${('$(arg end_effector)' == 'jaw') and ('$(arg sim)' == 'false') and ('$(arg use_fake_hardware)' == 'false')}">
       <ros2_control name="JawGripperStub" type="system">
@@ -417,4 +417,14 @@
             <param name="min">0</param>
             <param name="max">${finger_stroke}</param>
+          </command_interface>
+          <state_interface name="position">
+            <param name="initial_value">0.0</param>
+          </state_interface>
+          <state_interface name="velocity"/>
+        </joint>
+        <joint name="arm_jaw_gripper_finger_left_joint">
+          <command_interface name="position">
+            <param name="min">${-finger_stroke}</param>
+            <param name="max">0</param>
           </command_interface>
           <state_interface name="position">

Commit message: feat(arm): add drill_sampling tool + dedicated teleop mode

File: src/arm/arm_description/urdf/arm_macro.xacro (robot description, xacro)
@@ -136,4 +136,18 @@
       <limit lower="${-pi}" upper="${pi}" effort="100.0" velocity="1.0"/>
     </joint>
+    <!-- Drill/sample tool masses and volumetric centroids below are computed
+         directly from drill.stl / sampling.stl via the STL divergence-
+         theorem method (signed tetrahedron volumes from the mesh origin) —
+         not vertex-averaging, which is biased by triangulation density
+         (sampling.stl at 77k triangles vs drill.stl at 3.6k would otherwise
+         skew badly). Cross-checked: drill_sampling.stl's own volume
+         (732.47 cm^3) exactly equals drill.stl's (136.67) + sampling.stl's
+         (595.80), confirming both share one assembly frame with
+         arm_end_effector_link (same convention as arm_jaw_gripper_v3.stl) —
+         so both mount here with a plain identity origin, same as jaw.
+         Density is NOT uniform between the two (drill ~14.6 g/cm^3, sample
+         ~1.0 g/cm^3), so drill_sampling's combined COM is the MASS-weighted
+         average of the two tools' own COMs below, not drill_sampling.stl's
+         own (volume-weighted) centroid — those are different points. -->
     <link name="arm_end_effector_link">
       <xacro:if value="${'$(arg end_effector)' == 'jaw'}">
@@ -148,5 +162,35 @@
       <xacro:if value="${'$(arg end_effector)' == 'other_tool'}">
       </xacro:if>
-      <xacro:dummy_inertia mass="0.2"/>
+      <!-- Drill + sample mounted together: one combined mesh (avoids
+           double-rendering drill.stl + sampling.stl on top of each other —
+           drill_sampling.stl already IS their union, see note above).
+           rpy="0 pi pi/2" (unlike jaw's plain identity origin): the raw
+           STL's assembly frame had the tool misoriented relative to
+           arm_end_effector_link's actual orientation — confirmed visually
+           in rviz. ee_tool_com_{x,y,z} below in the <ros2_control> block is
+           rotated the SAME way — URDF rpy convention R = Rz(yaw)*Ry(pitch)*
+           Rx(roll), so here R = Rz(pi/2)*Ry(pi), giving x'=-y, y'=-x, z'=-z
+           — if this origin ever changes again, that COM must be re-rotated
+           to match, or gravity compensation will hold the wrong point. -->
+      <xacro:if value="${'$(arg end_effector)' == 'drill_sampling'}">
+        <visual>
+          <origin xyz="0 0 0" rpy="0 ${pi} ${pi/2}"/>
+          <geometry><mesh filename="${mesh_path}/drill_sampling.stl" scale="${stl_scale}"/></geometry>
+          <material name="light_grey"/>
+        </visual>
+        <collision>
+          <origin xyz="0 0 0" rpy="0 ${pi} ${pi/2}"/>
+          <geometry><mesh filename="${mesh_path}/drill_sampling.stl" scale="${stl_scale}"/></geometry>
+        </collision>
+      </xacro:if>
+      <xacro:if value="${'$(arg end_effector)' == 'jaw'}">
+        <xacro:dummy_inertia mass="0.2"/>
+      </xacro:if>
+      <xacro:if value="${'$(arg end_effector)' == 'drill_sampling'}">
+        <xacro:dummy_inertia mass="2.6"/>
+      </xacro:if>
+      <xacro:if value="${'$(arg end_effector)' == 'other_tool'}">
+        <xacro:dummy_inertia mass="0.2"/>
+      </xacro:if>
     </link>
     <xacro:if value="${'$(arg end_effector)' == 'jaw'}">
@@ -230,5 +274,5 @@
       <parent link="arm_end_effector_link"/>
       <child link="arm_tcp_link"/>
-      <xacro:if value="${'$(arg end_effector)' == 'jaw'}">
+      <xacro:if value="${('$(arg end_effector)' == 'jaw') or ('$(arg end_effector)' == 'drill_sampling')}">
         <!-- v3: X=Y=0 by construction (right/left fingers are the same mesh
              mirrored 180 deg about Z through the shared origin, see the
@@ -244,8 +288,12 @@
              calculation error; the formula itself is unchanged from v2
              and matches the SRDF's own tip_link convention for
-             arm_tcp_link (indomitus_arm.srdf). -->
+             arm_tcp_link (indomitus_arm.srdf).
+             drill_sampling deliberately shares this SAME point (not its
+             own offset) — keyboard_servo_node's drill mode rolls about
+             arm_tcp_link's local Z, and that must be the same physical
+             point/axis jaw already uses, not a second, different pivot. -->
         <origin xyz="0 0 0.1615" rpy="0 0 0"/>
       </xacro:if>
-      <xacro:if value="${'$(arg end_effector)' != 'jaw'}">
+      <xacro:if value="${('$(arg end_effector)' != 'jaw') and ('$(arg end_effector)' != 'drill_sampling')}">
         <origin xyz="0 -0.23 0" rpy="0 0 0"/>
       </xacro:if>
@@ -328,10 +376,38 @@
             <param name="feedback_timeout_secs">2.0</param>
             <param name="gravity_ff_enabled">true</param>
-            <!-- ~3.8 kg hangs below the shoulder with its COM ~0.3 m out, so the
-                 holding torque there reaches ~11 Nm on extended poses. The two
-                 motor families are an order of magnitude apart: Steadywin is
-                 rated 48 Nm, Damiao only 9 Nm continuous. -->
-            <param name="gravity_ff_max_nm_steadywin">20.0</param>
-            <param name="gravity_ff_max_nm_damiao">6.0</param>
+            <!-- Set to each motor family's own real rated capacity, not the
+                 shared MIT-protocol packing scale (48 Nm) — that scale is
+                 NOT a safe ceiling for Damiao on its own: Damiao is only
+                 rated 9 Nm continuous, so clamping it at the protocol's
+                 48 Nm would let sustained gravity-holding torque run at
+                 over 5x its continuous rating. Steadywin's 48 Nm here
+                 already equals its own rated capacity, so this is the most
+                 gravity-ff can use on either family without exceeding what
+                 the motor itself can sustain indefinitely. -->
+            <param name="gravity_ff_max_nm_steadywin">48.0</param>
+            <param name="gravity_ff_max_nm_damiao">9.0</param>
+            <!-- Payload mass + volumetric centroid (assembly frame, meters)
+                 for gravity compensation — see arm_end_effector_link above
+                 for how these were computed and cross-checked. jaw and
+                 other_tool are left unset on purpose: ArmCanSystem's own
+                 defaults (0.4 kg, {0,0,0.06}) are the live-tuned jaw value
+                 from arm_hardware_interface.cpp — do not duplicate it here. -->
+            <xacro:if value="${'$(arg end_effector)' == 'drill_sampling'}">
+              <!-- Mass-weighted average of the drill's own COM (2.0 kg,
+                   (0.45169,-0.00000,-0.02825)) and the sample's own COM
+                   (0.6 kg, (0.00184,0.00317,-0.08465)) in the RAW STL frame
+                   — NOT drill_sampling.stl's own volumetric centroid, which
+                   would be volume-weighted and wrong here since the two
+                   parts have very different density (drill ~14.6 g/cm^3,
+                   sample ~1.0 g/cm^3). Rotated to match the visual/collision
+                   <origin rpy="0 pi pi/2"> above (raw-frame weighted value
+                   was (0.34788, 0.00073, -0.04127); R = Rz(pi/2)*Ry(pi) ->
+                   x'=-y, y'=-x, z'=-z). Keep this in sync if that <origin>
+                   ever changes — see its comment above. -->
+              <param name="ee_tool_mass_kg">2.6</param>
+              <param name="ee_tool_com_x">-0.00073</param>
+              <param name="ee_tool_com_y">-0.34788</param>
+              <param name="ee_tool_com_z">0.04127</param>
+            </xacro:if>
           </xacro:unless>
         </xacro:unless>
