Commit message: feat(arm): decouple viz from core arm_moveit_config for headless Jetson

File: src/arm/arm_description/urdf/arm_macro.xacro (robot description, xacro)
@@ -136,18 +136,8 @@
       <limit lower="${-pi}" upper="${pi}" effort="100.0" velocity="1.0"/>
     </joint>
-    <!-- Drill/sample tool masses and volumetric centroids below are computed
-         directly from drill.stl / sampling.stl via the STL divergence-
-         theorem method (signed tetrahedron volumes from the mesh origin) —
-         not vertex-averaging, which is biased by triangulation density
-         (sampling.stl at 77k triangles vs drill.stl at 3.6k would otherwise
-         skew badly). Cross-checked: drill_sampling.stl's own volume
-         (732.47 cm^3) exactly equals drill.stl's (136.67) + sampling.stl's
-         (595.80), confirming both share one assembly frame with
-         arm_end_effector_link (same convention as arm_jaw_gripper_v3.stl) —
-         so both mount here with a plain identity origin, same as jaw.
-         Density is NOT uniform between the two (drill ~14.6 g/cm^3, sample
-         ~1.0 g/cm^3), so drill_sampling's combined COM is the MASS-weighted
-         average of the two tools' own COMs below, not drill_sampling.stl's
-         own (volume-weighted) centroid — those are different points. -->
+    <!-- Drill/sample masses+centroids: STL divergence-theorem volumes (not
+         vertex-avg, biased by triangle density), mass-weighted COM (density
+         differs: drill ~14.6 g/cm^3, sample ~1.0), not drill_sampling.stl's
+         own volumetric centroid — those are different points. -->
     <link name="arm_end_effector_link">
       <xacro:if value="${'$(arg end_effector)' == 'jaw'}">
@@ -162,15 +152,7 @@
       <xacro:if value="${'$(arg end_effector)' == 'other_tool'}">
       </xacro:if>
-      <!-- Drill + sample mounted together: one combined mesh (avoids
-           double-rendering drill.stl + sampling.stl on top of each other —
-           drill_sampling.stl already IS their union, see note above).
-           rpy="0 pi pi/2" (unlike jaw's plain identity origin): the raw
-           STL's assembly frame had the tool misoriented relative to
-           arm_end_effector_link's actual orientation — confirmed visually
-           in rviz. ee_tool_com_{x,y,z} below in the <ros2_control> block is
-           rotated the SAME way — URDF rpy convention R = Rz(yaw)*Ry(pitch)*
-           Rx(roll), so here R = Rz(pi/2)*Ry(pi), giving x'=-y, y'=-x, z'=-z
-           — if this origin ever changes again, that COM must be re-rotated
-           to match, or gravity compensation will hold the wrong point. -->
+      <!-- rpy="0 pi pi/2" corrects the STL's misoriented assembly frame.
+           ee_tool_com_{x,y,z} in <ros2_control> below is rotated to match
+           (R=Rz(pi/2)*Ry(pi): x'=-y, y'=-x, z'=-z) — re-rotate both together. -->
       <xacro:if value="${'$(arg end_effector)' == 'drill_sampling'}">
         <visual>
@@ -289,8 +271,6 @@
              and matches the SRDF's own tip_link convention for
              arm_tcp_link (indomitus_arm.srdf).
-             drill_sampling deliberately shares this SAME point (not its
-             own offset) — keyboard_servo_node's drill mode rolls about
-             arm_tcp_link's local Z, and that must be the same physical
-             point/axis jaw already uses, not a second, different pivot. -->
+             drill_sampling deliberately shares this same point/axis (drill
+             mode rolls about arm_tcp_link's local Z). -->
         <origin xyz="0 0 0.1615" rpy="0 0 0"/>
       </xacro:if>
@@ -394,15 +374,7 @@
                  from arm_hardware_interface.cpp — do not duplicate it here. -->
             <xacro:if value="${'$(arg end_effector)' == 'drill_sampling'}">
-              <!-- Mass-weighted average of the drill's own COM (2.0 kg,
-                   (0.45169,-0.00000,-0.02825)) and the sample's own COM
-                   (0.6 kg, (0.00184,0.00317,-0.08465)) in the RAW STL frame
-                   — NOT drill_sampling.stl's own volumetric centroid, which
-                   would be volume-weighted and wrong here since the two
-                   parts have very different density (drill ~14.6 g/cm^3,
-                   sample ~1.0 g/cm^3). Rotated to match the visual/collision
-                   <origin rpy="0 pi pi/2"> above (raw-frame weighted value
-                   was (0.34788, 0.00073, -0.04127); R = Rz(pi/2)*Ry(pi) ->
-                   x'=-y, y'=-x, z'=-z). Keep this in sync if that <origin>
-                   ever changes — see its comment above. -->
+              <!-- Mass-weighted COM of drill (2.0kg) + sample (0.6kg), raw-frame
+                   value (0.34788, 0.00073, -0.04127) rotated to match the
+                   <origin rpy="0 pi pi/2"> above — keep in sync if that changes. -->
               <param name="ee_tool_mass_kg">2.6</param>
               <param name="ee_tool_com_x">-0.00073</param>

Commit message: feat(arm): split sampling/drill modes, route home/mode-engage through collision-aware planning

File: src/arm/arm_description/urdf/arm_macro.xacro (robot description, xacro)
@@ -134,5 +134,5 @@
       <origin xyz="0.0323 0 -0.035" rpy="${-pi/2} ${pi/3} ${-pi/2}"/>
       <axis xyz="0 0 1"/>
-      <limit lower="${-pi}" upper="${pi}" effort="100.0" velocity="1.0"/>
+      <limit lower="${-2*pi}" upper="${2*pi}" effort="100.0" velocity="1.0"/>
     </joint>
     <!-- Drill/sample masses+centroids: STL divergence-theorem volumes (not

Commit message: fix(arm): move drill tool COM inward to match real assembly

File: src/arm/arm_description/urdf/arm_macro.xacro (robot description, xacro)
@@ -375,9 +375,15 @@
             <xacro:if value="${'$(arg end_effector)' == 'drill_sampling'}">
               <!-- Mass-weighted COM of drill (2.0kg) + sample (0.6kg), raw-frame
-                   value (0.34788, 0.00073, -0.04127) rotated to match the
-                   <origin rpy="0 pi pi/2"> above — keep in sync if that changes. -->
+                   value (0.15, 0.00073, -0.04127) rotated to match the
+                   <origin rpy="0 pi pi/2"> above — keep in sync if that changes.
+                   Y moved in from 0.34788 to 0.15 on explicit request — the
+                   original STL-derived value put the COM much further out
+                   along the tool than the real assembly's, overstating the
+                   gravity-holding torque ArmCanSystem's feedforward computes
+                   at this joint. X/Z left as originally computed (only the
+                   dominant, along-the-tool axis was flagged as wrong). -->
               <param name="ee_tool_mass_kg">2.6</param>
               <param name="ee_tool_com_x">-0.00073</param>
-              <param name="ee_tool_com_y">-0.34788</param>
+              <param name="ee_tool_com_y">-0.15</param>
               <param name="ee_tool_com_z">0.04127</param>
             </xacro:if>

Commit message: test version

File: src/arm/arm_description/urdf/arm_macro.xacro (robot description, xacro)
@@ -100,5 +100,5 @@
       <origin xyz="-0.0173 0.3 0" rpy="0 ${pi/2} 0"/>
       <axis xyz="0 0 1"/>
-      <limit lower="${-pi/2}" upper="${pi/2}" effort="100.0" velocity="1.0"/>
+      <limit lower="${-pi}" upper="${pi}" effort="100.0" velocity="1.0"/>
     </joint>
     <link name="arm_wrist_1_link">

Commit message: feat(arm): retune joint limits/torque/tool COM, tighten collision margins, route gamepad B/Y home

File: src/arm/arm_description/urdf/arm_macro.xacro (robot description, xacro)
@@ -49,5 +49,5 @@
       <origin xyz="0.06 0 0.021" rpy="0 0 0"/>
       <axis xyz="0 0 1"/>
-      <limit lower="${-pi}" upper="${pi}" effort="100.0" velocity="1.0"/>
+      <limit lower="${-4*pi}" upper="${4*pi}" effort="100.0" velocity="1.0"/>
     </joint>
     <link name="arm_base_link">
@@ -66,5 +66,5 @@
       <origin xyz="-0.040366 -0.000325 0.103" rpy="${pi/3} 0 ${-pi}"/>
       <axis xyz="1 0 0"/>
-      <limit lower="${-pi}" upper="${pi}" effort="100.0" velocity="1.0"/>
+      <limit lower="${-4*pi}" upper="${4*pi}" effort="100.0" velocity="1.0"/>
     </joint>
     <link name="arm_shoulder_link">
@@ -83,5 +83,5 @@
       <origin xyz="0 0.3 0" rpy="${5*pi/12} 0 0"/>
       <axis xyz="1 0 0"/>
-      <limit lower="${-pi/2}" upper="${pi/2}" effort="100.0" velocity="1.0"/>
+      <limit lower="${-4*pi}" upper="${4*pi}" effort="100.0" velocity="1.0"/>
     </joint>
     <link name="arm_forearm_link">
@@ -100,5 +100,5 @@
       <origin xyz="-0.0173 0.3 0" rpy="0 ${pi/2} 0"/>
       <axis xyz="0 0 1"/>
-      <limit lower="${-pi}" upper="${pi}" effort="100.0" velocity="1.0"/>
+      <limit lower="${-4*pi}" upper="${4*pi}" effort="100.0" velocity="1.0"/>
     </joint>
     <link name="arm_wrist_1_link">
@@ -117,5 +117,5 @@
       <origin xyz="0.0323 0 -0.035" rpy="${-pi/2} 0 ${pi/2}"/>
       <axis xyz="0 0 1"/>
-      <limit lower="${-pi}" upper="${pi}" effort="100.0" velocity="1.0"/>
+      <limit lower="${-4*pi}" upper="${4*pi}" effort="100.0" velocity="1.0"/>
     </joint>
     <link name="arm_wrist_2_link">
@@ -134,10 +134,16 @@
       <origin xyz="0.0323 0 -0.035" rpy="${-pi/2} ${pi/3} ${-pi/2}"/>
       <axis xyz="0 0 1"/>
-      <limit lower="${-2*pi}" upper="${2*pi}" effort="100.0" velocity="1.0"/>
+      <limit lower="${-4*pi}" upper="${4*pi}" effort="100.0" velocity="1.0"/>
     </joint>
     <!-- Drill/sample masses+centroids: STL divergence-theorem volumes (not
          vertex-avg, biased by triangle density), mass-weighted COM (density
          differs: drill ~14.6 g/cm^3, sample ~1.0), not drill_sampling.stl's
-         own volumetric centroid — those are different points. -->
+         own volumetric centroid — those are different points. Single source
+         of truth for the drill_sampling tool COM: edit these three, both the
+         gravity-comp <param>s below and the TEMP DEBUG VISUAL marker read
+         from here. -->
+    <xacro:property name="ee_tool_com_x" value="-0.03"/>
+    <xacro:property name="ee_tool_com_y" value="-0.08"/>
+    <xacro:property name="ee_tool_com_z" value="0.05"/>
     <link name="arm_end_effector_link">
       <xacro:if value="${'$(arg end_effector)' == 'jaw'}">
@@ -157,10 +163,10 @@
       <xacro:if value="${'$(arg end_effector)' == 'drill_sampling'}">
         <visual>
-          <origin xyz="0 0 0" rpy="0 ${pi} ${pi/2}"/>
+          <origin xyz="0 0 0.01" rpy="0 ${pi} ${pi/2}"/>
           <geometry><mesh filename="${mesh_path}/drill_sampling.stl" scale="${stl_scale}"/></geometry>
           <material name="light_grey"/>
         </visual>
         <collision>
-          <origin xyz="0 0 0" rpy="0 ${pi} ${pi/2}"/>
+          <origin xyz="0 0 0.01" rpy="0 ${pi} ${pi/2}"/>
           <geometry><mesh filename="${mesh_path}/drill_sampling.stl" scale="${stl_scale}"/></geometry>
         </collision>
@@ -336,4 +342,25 @@
     </joint>
     <link name="arm_camera_optical_frame"/>
+    <!-- TEMP DEBUG VISUAL — sanity-check the assumed tool COM against the
+         real one by eye in RViz. Safe to delete this whole xacro:if block
+         when done; not wired into collision (visual only). Reads
+         ee_tool_com_x/y/z (declared above, also used by the gravity-comp
+         <param>s in <ros2_control> below) — edit the properties, not this
+         origin, and both stay in sync automatically. -->
+    <xacro:if value="${'$(arg end_effector)' == 'drill_sampling'}">
+      <joint name="arm_end_effector_com_debug_joint" type="fixed">
+        <parent link="arm_end_effector_link"/>
+        <child link="arm_end_effector_com_debug_link"/>
+        <origin xyz="${ee_tool_com_x} ${ee_tool_com_y} ${ee_tool_com_z}" rpy="0 0 0"/>
+      </joint>
+      <link name="arm_end_effector_com_debug_link">
+        <visual>
+          <geometry><sphere radius="0.01"/></geometry>
+          <material name="com_debug_red">
+            <color rgba="1.0 0.0 0.0 1.0"/>
+          </material>
+        </visual>
+      </link>
+    </xacro:if>
     <ros2_control name="ArmSystem" type="system">
       <hardware>
@@ -375,16 +402,17 @@
             <xacro:if value="${'$(arg end_effector)' == 'drill_sampling'}">
               <!-- Mass-weighted COM of drill (2.0kg) + sample (0.6kg), raw-frame
-                   value (0.15, 0.00073, -0.04127) rotated to match the
-                   <origin rpy="0 pi pi/2"> above — keep in sync if that changes.
-                   Y moved in from 0.34788 to 0.15 on explicit request — the
-                   original STL-derived value put the COM much further out
-                   along the tool than the real assembly's, overstating the
-                   gravity-holding torque ArmCanSystem's feedforward computes
-                   at this joint. X/Z left as originally computed (only the
-                   dominant, along-the-tool axis was flagged as wrong). -->
-              <param name="ee_tool_mass_kg">2.6</param>
-              <param name="ee_tool_com_x">-0.00073</param>
-              <param name="ee_tool_com_y">-0.15</param>
-              <param name="ee_tool_com_z">0.04127</param>
+                   value rotated to match the <origin rpy="0 pi pi/2"> above —
+                   keep in sync if that changes. Values (ee_tool_com_x/y/z
+                   properties, declared up at arm_end_effector_link) have been
+                   retuned repeatedly on explicit request after live testing
+                   showed too much gravity-holding torque (arm drifting/
+                   pushing up) — the original STL-derived value put the COM
+                   much further out along the tool than the real assembly's.
+                   Edit the xacro:property values, not these <param>s — the
+                   TEMP DEBUG VISUAL marker above reads the same properties. -->
+              <param name="ee_tool_mass_kg">2.8</param>
+              <param name="ee_tool_com_x">${ee_tool_com_x}</param>
+              <param name="ee_tool_com_y">${ee_tool_com_y}</param>
+              <param name="ee_tool_com_z">${ee_tool_com_z}</param>
             </xacro:if>
           </xacro:unless>

Commit message: fix(arm): align joint limits with develop, drop OMPL search-space override

File: src/arm/arm_description/urdf/arm_macro.xacro (robot description, xacro)
@@ -49,5 +49,5 @@
       <origin xyz="0.06 0 0.021" rpy="0 0 0"/>
       <axis xyz="0 0 1"/>
-      <limit lower="${-4*pi}" upper="${4*pi}" effort="100.0" velocity="1.0"/>
+      <limit lower="${-pi}" upper="${pi}" effort="100.0" velocity="1.0"/>
     </joint>
     <link name="arm_base_link">
@@ -66,5 +66,5 @@
       <origin xyz="-0.040366 -0.000325 0.103" rpy="${pi/3} 0 ${-pi}"/>
       <axis xyz="1 0 0"/>
-      <limit lower="${-4*pi}" upper="${4*pi}" effort="100.0" velocity="1.0"/>
+      <limit lower="${-pi}" upper="${pi}" effort="100.0" velocity="1.0"/>
     </joint>
     <link name="arm_shoulder_link">
@@ -83,5 +83,5 @@
       <origin xyz="0 0.3 0" rpy="${5*pi/12} 0 0"/>
       <axis xyz="1 0 0"/>
-      <limit lower="${-4*pi}" upper="${4*pi}" effort="100.0" velocity="1.0"/>
+      <limit lower="${-pi/2}" upper="${pi/2}" effort="100.0" velocity="1.0"/>
     </joint>
     <link name="arm_forearm_link">
@@ -100,5 +100,5 @@
       <origin xyz="-0.0173 0.3 0" rpy="0 ${pi/2} 0"/>
       <axis xyz="0 0 1"/>
-      <limit lower="${-4*pi}" upper="${4*pi}" effort="100.0" velocity="1.0"/>
+      <limit lower="${-pi}" upper="${pi}" effort="100.0" velocity="1.0"/>
     </joint>
     <link name="arm_wrist_1_link">
@@ -117,5 +117,5 @@
       <origin xyz="0.0323 0 -0.035" rpy="${-pi/2} 0 ${pi/2}"/>
       <axis xyz="0 0 1"/>
-      <limit lower="${-4*pi}" upper="${4*pi}" effort="100.0" velocity="1.0"/>
+      <limit lower="${-pi}" upper="${pi}" effort="100.0" velocity="1.0"/>
     </joint>
     <link name="arm_wrist_2_link">
@@ -134,5 +134,5 @@
       <origin xyz="0.0323 0 -0.035" rpy="${-pi/2} ${pi/3} ${-pi/2}"/>
       <axis xyz="0 0 1"/>
-      <limit lower="${-4*pi}" upper="${4*pi}" effort="100.0" velocity="1.0"/>
+      <limit lower="${-pi}" upper="${pi}" effort="100.0" velocity="1.0"/>
     </joint>
     <!-- Drill/sample masses+centroids: STL divergence-theorem volumes (not

Commit message: fix(arm): restore ±2π hardware joint limits on all arm joints

File: src/arm/arm_description/urdf/arm_macro.xacro (robot description, xacro)
@@ -50,5 +50,5 @@
       <origin xyz="0.06 0 0.021" rpy="0 0 0"/>
       <axis xyz="0 0 1"/>
-      <limit lower="${-pi}" upper="${pi}" effort="100.0" velocity="1.0"/>
+      <limit lower="${-2*pi}" upper="${2*pi}" effort="100.0" velocity="1.0"/>
     </joint>
     <link name="arm_base_link">
@@ -67,5 +67,5 @@
       <origin xyz="-0.040366 -0.000325 0.103" rpy="${pi/3} 0 ${-pi}"/>
       <axis xyz="1 0 0"/>
-      <limit lower="${-pi}" upper="${pi}" effort="100.0" velocity="1.0"/>
+      <limit lower="${-2*pi}" upper="${2*pi}" effort="100.0" velocity="1.0"/>
     </joint>
     <link name="arm_shoulder_link">
@@ -84,5 +84,5 @@
       <origin xyz="0 0.3 0" rpy="${5*pi/12} 0 0"/>
       <axis xyz="1 0 0"/>
-      <limit lower="${-pi/2}" upper="${pi/2}" effort="100.0" velocity="1.0"/>
+      <limit lower="${-2*pi}" upper="${2*pi}" effort="100.0" velocity="1.0"/>
     </joint>
     <link name="arm_forearm_link">
@@ -101,5 +101,5 @@
       <origin xyz="-0.0173 0.3 0" rpy="0 ${pi/2} 0"/>
       <axis xyz="0 0 1"/>
-      <limit lower="${-pi}" upper="${pi}" effort="100.0" velocity="1.0"/>
+      <limit lower="${-2*pi}" upper="${2*pi}" effort="100.0" velocity="1.0"/>
     </joint>
     <link name="arm_wrist_1_link">
@@ -118,5 +118,5 @@
       <origin xyz="0.0323 0 -0.035" rpy="${-pi/2} 0 ${pi/2}"/>
       <axis xyz="0 0 1"/>
-      <limit lower="${-pi}" upper="${pi}" effort="100.0" velocity="1.0"/>
+      <limit lower="${-2*pi}" upper="${2*pi}" effort="100.0" velocity="1.0"/>
     </joint>
     <link name="arm_wrist_2_link">
@@ -135,5 +135,5 @@
       <origin xyz="0.0323 0 -0.035" rpy="${-pi/2} ${pi/3} ${-pi/2}"/>
       <axis xyz="0 0 1"/>
-      <limit lower="${-pi}" upper="${pi}" effort="100.0" velocity="1.0"/>
+      <limit lower="${-2*pi}" upper="${2*pi}" effort="100.0" velocity="1.0"/>
     </joint>
     <!-- Drill/sample masses+centroids: STL divergence-theorem volumes (not
