Commit message: Feature/arm/teleop push boost (#560)
* feat(arm): gripper joint stub fix, torque logging, teleop push boost

* feat(arm): add drill_sampling tool + dedicated teleop mode

* feat(arm): decouple viz from core arm_moveit_config for headless Jetson

* feat(arm): split sampling/drill modes, route home/mode-engage through collision-aware planning

* fix(arm): move drill tool COM inward to match real assembly

* fix(arm): propagate end_effector arg to every robot_description build in sim launch

* feat(arm): add collision-checked tool-leveling command with pitch/yaw lock

* test version

* feat(arm): retune joint limits/torque/tool COM, tighten collision margins, route gamepad B/Y home

* chore(arm): change jaw gripper address

* fix(arm): align joint limits with develop, drop OMPL search-space override

* fix(arm): restore develop collision-check settings, retune self-collision threshold for jaw

* feat(arm_sim): propagate end_effector through Gazebo move_group/servo

* fix(arm_tasks): correct moveit_servo StatusCode table, distinguish decelerate from halt

* feat(arm_tasks): panel_align/orient_gripper service, TF timeout, panel-pose staleness margin

* feat(arm_tasks): ERC activity-indicator delay for r/p/f + gripper-only reorient on 'm'

* fix(arm): level camera roll to world-up instead of panel tilt

* feat(arm): auto-restart camera on crash, re-apply focus/brightness on respawn

* feat(arm): add drill_sampling claw/drill/lock gamepad control, invert drill-mode axes

ClawDrillCanBus mirrors GripperCanBus for the drill_sampling tool's
ESP32 firmware (CAN 0x1E): buttons 11/13 now route to claw open/close
or drill up/down depending on sampling/drill sub-mode, buttons 12/14
drive the tool's electric lock. Also inverts the three drill-mode stick
axes per operator feedback, and documents the full mapping for ground
station in docs/arm/arm_gamepad_mapping.md.

* chore(arm): change collision limits

* feat(arm): move end-effector CAN control into arm_peripherals bridge node

* fix(arm_tasks): tighter orientation tolerance for 'm' gripper reorient

* chore(arm): shorten comments in keyboard_servo_node.py

* feat(arm_task): launch files for the gamepad control splitted to two with nodes need to be run on the rover and on the laptop/gs

* feat(arm): namespace the whole arm stack under /arm

* feat(arm): fix(arm): un-namespace-double RViz/servo/controller_manager params

* refactor(arm): change packages structure and isolate vizualization

* fix(arm): restore ±2π hardware joint limits on all arm joints

* fix(arm_moveit_config): raise KDL IK timeout for the tighter panel joint limits

* fix(arm_tasks): bound OMPL to panel joint limits, protect orient_gripper with panel collision

* feat(arm): replace /tmp flock with a networked cross-host arm-motion lock

* test(arm_teleop): fix tests for the new arm_motion_lock signature

* fix(arm_teleop): defer sampling/drill mode commit until home move succeeds

* chore(arm): isolate using panel only for jaw gripper

---------

Co-authored-by: Martik-k <kosiv.marta@gmail.com>
Co-authored-by: BohdanZasymovych <bohdan.zasymovych@gmail.com>

File: src/arm/arm_description/urdf/arm_macro.xacro (robot description, xacro)
@@ -4,4 +4,5 @@
   <xacro:arg name="end_effector" default="jaw"/>
   <xacro:arg name="sim" default="false"/>
+  <xacro:arg name="can_interface" default="can0"/>
   <!-- When the arm is mounted into another robot's URDF (e.g. the rover, see
        rover_description's mount_arm arg) that outer URDF already adds its
@@ -49,5 +50,5 @@
       <origin xyz="0.06 0 0.021" rpy="0 0 0"/>
       <axis xyz="0 0 1"/>
-      <limit lower="${-pi}" upper="${pi}" effort="100.0" velocity="1.0"/>
+      <limit lower="${-2*pi}" upper="${2*pi}" effort="100.0" velocity="1.0"/>
     </joint>
     <link name="arm_base_link">
@@ -66,5 +67,5 @@
       <origin xyz="-0.040366 -0.000325 0.103" rpy="${pi/3} 0 ${-pi}"/>
       <axis xyz="1 0 0"/>
-      <limit lower="${-pi}" upper="${pi}" effort="100.0" velocity="1.0"/>
+      <limit lower="${-2*pi}" upper="${2*pi}" effort="100.0" velocity="1.0"/>
     </joint>
     <link name="arm_shoulder_link">
@@ -83,5 +84,5 @@
       <origin xyz="0 0.3 0" rpy="${5*pi/12} 0 0"/>
       <axis xyz="1 0 0"/>
-      <limit lower="${-pi/2}" upper="${pi/2}" effort="100.0" velocity="1.0"/>
+      <limit lower="${-2*pi}" upper="${2*pi}" effort="100.0" velocity="1.0"/>
     </joint>
     <link name="arm_forearm_link">
@@ -100,5 +101,5 @@
       <origin xyz="-0.0173 0.3 0" rpy="0 ${pi/2} 0"/>
       <axis xyz="0 0 1"/>
-      <limit lower="${-pi/2}" upper="${pi/2}" effort="100.0" velocity="1.0"/>
+      <limit lower="${-2*pi}" upper="${2*pi}" effort="100.0" velocity="1.0"/>
     </joint>
     <link name="arm_wrist_1_link">
@@ -117,5 +118,5 @@
       <origin xyz="0.0323 0 -0.035" rpy="${-pi/2} 0 ${pi/2}"/>
       <axis xyz="0 0 1"/>
-      <limit lower="${-pi}" upper="${pi}" effort="100.0" velocity="1.0"/>
+      <limit lower="${-2*pi}" upper="${2*pi}" effort="100.0" velocity="1.0"/>
     </joint>
     <link name="arm_wrist_2_link">
@@ -132,8 +133,18 @@
       <parent link="arm_wrist_2_link"/>
       <child link="arm_end_effector_link"/>
-      <origin xyz="0.0323 0 -0.035" rpy="${-pi/2} ${pi/2} ${-pi/2}"/>
+      <origin xyz="0.0323 0 -0.035" rpy="${-pi/2} ${pi/3} ${-pi/2}"/>
       <axis xyz="0 0 1"/>
-      <limit lower="${-pi}" upper="${pi}" effort="100.0" velocity="1.0"/>
-    </joint>
+      <limit lower="${-2*pi}" upper="${2*pi}" effort="100.0" velocity="1.0"/>
+    </joint>
+    <!-- Drill/sample masses+centroids: STL divergence-theorem volumes (not
+         vertex-avg, biased by triangle density), mass-weighted COM (density
+         differs: drill ~14.6 g/cm^3, sample ~1.0), not drill_sampling.stl's
+         own volumetric centroid — those are different points. Single source
+         of truth for the drill_sampling tool COM: edit these three, both the
+         gravity-comp <param>s below and the TEMP DEBUG VISUAL marker read
+         from here. -->
+    <xacro:property name="ee_tool_com_x" value="-0.03"/>
+    <xacro:property name="ee_tool_com_y" value="-0.08"/>
+    <xacro:property name="ee_tool_com_z" value="0.05"/>
     <link name="arm_end_effector_link">
       <xacro:if value="${'$(arg end_effector)' == 'jaw'}">
@@ -148,5 +159,27 @@
       <xacro:if value="${'$(arg end_effector)' == 'other_tool'}">
       </xacro:if>
-      <xacro:dummy_inertia mass="0.2"/>
+      <!-- rpy="0 pi pi/2" corrects the STL's misoriented assembly frame.
+           ee_tool_com_{x,y,z} in <ros2_control> below is rotated to match
+           (R=Rz(pi/2)*Ry(pi): x'=-y, y'=-x, z'=-z) — re-rotate both together. -->
+      <xacro:if value="${'$(arg end_effector)' == 'drill_sampling'}">
+        <visual>
+          <origin xyz="0 0 0.01" rpy="0 ${pi} ${pi/2}"/>
+          <geometry><mesh filename="${mesh_path}/drill_sampling.stl" scale="${stl_scale}"/></geometry>
+          <material name="light_grey"/>
+        </visual>
+        <collision>
+          <origin xyz="0 0 0.01" rpy="0 ${pi} ${pi/2}"/>
+          <geometry><mesh filename="${mesh_path}/drill_sampling.stl" scale="${stl_scale}"/></geometry>
+        </collision>
+      </xacro:if>
+      <xacro:if value="${'$(arg end_effector)' == 'jaw'}">
+        <xacro:dummy_inertia mass="0.2"/>
+      </xacro:if>
+      <xacro:if value="${'$(arg end_effector)' == 'drill_sampling'}">
+        <xacro:dummy_inertia mass="2.6"/>
+      </xacro:if>
+      <xacro:if value="${'$(arg end_effector)' == 'other_tool'}">
+        <xacro:dummy_inertia mass="0.2"/>
+      </xacro:if>
     </link>
     <xacro:if value="${'$(arg end_effector)' == 'jaw'}">
@@ -230,5 +263,5 @@
       <parent link="arm_end_effector_link"/>
       <child link="arm_tcp_link"/>
-      <xacro:if value="${'$(arg end_effector)' == 'jaw'}">
+      <xacro:if value="${('$(arg end_effector)' == 'jaw') or ('$(arg end_effector)' == 'drill_sampling')}">
         <!-- v3: X=Y=0 by construction (right/left fingers are the same mesh
              mirrored 180 deg about Z through the shared origin, see the
@@ -244,8 +277,10 @@
              calculation error; the formula itself is unchanged from v2
              and matches the SRDF's own tip_link convention for
-             arm_tcp_link (indomitus_arm.srdf). -->
+             arm_tcp_link (indomitus_arm.srdf).
+             drill_sampling deliberately shares this same point/axis (drill
+             mode rolls about arm_tcp_link's local Z). -->
         <origin xyz="0 0 0.1615" rpy="0 0 0"/>
       </xacro:if>
-      <xacro:if value="${'$(arg end_effector)' != 'jaw'}">
+      <xacro:if value="${('$(arg end_effector)' != 'jaw') and ('$(arg end_effector)' != 'drill_sampling')}">
         <origin xyz="0 -0.23 0" rpy="0 0 0"/>
       </xacro:if>
@@ -308,4 +343,25 @@
     </joint>
     <link name="arm_camera_optical_frame"/>
+    <!-- TEMP DEBUG VISUAL — sanity-check the assumed tool COM against the
+         real one by eye in RViz. Safe to delete this whole xacro:if block
+         when done; not wired into collision (visual only). Reads
+         ee_tool_com_x/y/z (declared above, also used by the gravity-comp
+         <param>s in <ros2_control> below) — edit the properties, not this
+         origin, and both stay in sync automatically. -->
+    <xacro:if value="${'$(arg end_effector)' == 'drill_sampling'}">
+      <joint name="arm_end_effector_com_debug_joint" type="fixed">
+        <parent link="arm_end_effector_link"/>
+        <child link="arm_end_effector_com_debug_link"/>
+        <origin xyz="${ee_tool_com_x} ${ee_tool_com_y} ${ee_tool_com_z}" rpy="0 0 0"/>
+      </joint>
+      <link name="arm_end_effector_com_debug_link">
+        <visual>
+          <geometry><sphere radius="0.01"/></geometry>
+          <material name="com_debug_red">
+            <color rgba="1.0 0.0 0.0 1.0"/>
+          </material>
+        </visual>
+      </link>
+    </xacro:if>
     <ros2_control name="ArmSystem" type="system">
       <hardware>
@@ -319,5 +375,5 @@
           <xacro:unless value="$(arg use_fake_hardware)">
             <plugin>arm_hardware_interface/ArmCanSystem</plugin>
-            <param name="can_interface">can0</param>
+            <param name="can_interface">$(arg can_interface)</param>
             <!-- Stiffness ramps 0 -> 100% over this many seconds after activation -->
             <param name="gain_ramp_secs">15.0</param>
@@ -328,10 +384,37 @@
             <param name="feedback_timeout_secs">2.0</param>
             <param name="gravity_ff_enabled">true</param>
-            <!-- ~3.8 kg hangs below the shoulder with its COM ~0.3 m out, so the
-                 holding torque there reaches ~11 Nm on extended poses. The two
-                 motor families are an order of magnitude apart: Steadywin is
-                 rated 48 Nm, Damiao only 9 Nm continuous. -->
-            <param name="gravity_ff_max_nm_steadywin">20.0</param>
-            <param name="gravity_ff_max_nm_damiao">6.0</param>
+            <!-- Set to each motor family's own real rated capacity, not the
+                 shared MIT-protocol packing scale (48 Nm) — that scale is
+                 NOT a safe ceiling for Damiao on its own: Damiao is only
+                 rated 9 Nm continuous, so clamping it at the protocol's
+                 48 Nm would let sustained gravity-holding torque run at
+                 over 5x its continuous rating. Steadywin's 48 Nm here
+                 already equals its own rated capacity, so this is the most
+                 gravity-ff can use on either family without exceeding what
+                 the motor itself can sustain indefinitely. -->
+            <param name="gravity_ff_max_nm_steadywin">48.0</param>
+            <param name="gravity_ff_max_nm_damiao">9.0</param>
+            <!-- Payload mass + volumetric centroid (assembly frame, meters)
+                 for gravity compensation — see arm_end_effector_link above
+                 for how these were computed and cross-checked. jaw and
+                 other_tool are left unset on purpose: ArmCanSystem's own
+                 defaults (0.4 kg, {0,0,0.06}) are the live-tuned jaw value
+                 from arm_hardware_interface.cpp — do not duplicate it here. -->
+            <xacro:if value="${'$(arg end_effector)' == 'drill_sampling'}">
+              <!-- Mass-weighted COM of drill (2.0kg) + sample (0.6kg), raw-frame
+                   value rotated to match the <origin rpy="0 pi pi/2"> above —
+                   keep in sync if that changes. Values (ee_tool_com_x/y/z
+                   properties, declared up at arm_end_effector_link) have been
+                   retuned repeatedly on explicit request after live testing
+                   showed too much gravity-holding torque (arm drifting/
+                   pushing up) — the original STL-derived value put the COM
+                   much further out along the tool than the real assembly's.
+                   Edit the xacro:property values, not these <param>s — the
+                   TEMP DEBUG VISUAL marker above reads the same properties. -->
+              <param name="ee_tool_mass_kg">2.8</param>
+              <param name="ee_tool_com_x">${ee_tool_com_x}</param>
+              <param name="ee_tool_com_y">${ee_tool_com_y}</param>
+              <param name="ee_tool_com_z">${ee_tool_com_z}</param>
+            </xacro:if>
           </xacro:unless>
         </xacro:unless>
@@ -401,11 +484,11 @@
       </xacro:if>
     </ros2_control>
-    <!-- There is no gripper motor on the real arm yet, but the finger joint must
-         still report state: without it joint_state_broadcaster never publishes
-         the joint, the planning scene monitor sees an incomplete robot state,
-         and move_group/Servo silently refuse to move. GenericSystem echoes
-         commands back as state, so the joint exists for MoveIt while nothing
-         physical moves. Replace with the real gripper hardware plugin once the
-         motor is wired up. -->
+    <!-- There is no gripper motor on the real arm yet, but both finger joints
+         must still report state: without it joint_state_broadcaster never
+         publishes them, the planning scene monitor sees an incomplete robot
+         state, and move_group/Servo silently refuse to move. GenericSystem
+         echoes commands back as state, so both joints exist for MoveIt while
+         nothing physical moves. Replace with the real gripper hardware plugin
+         once the motor is wired up. -->
     <xacro:if value="${('$(arg end_effector)' == 'jaw') and ('$(arg sim)' == 'false') and ('$(arg use_fake_hardware)' == 'false')}">
       <ros2_control name="JawGripperStub" type="system">
@@ -417,4 +500,14 @@
             <param name="min">0</param>
             <param name="max">${finger_stroke}</param>
+          </command_interface>
+          <state_interface name="position">
+            <param name="initial_value">0.0</param>
+          </state_interface>
+          <state_interface name="velocity"/>
+        </joint>
+        <joint name="arm_jaw_gripper_finger_left_joint">
+          <command_interface name="position">
+            <param name="min">${-finger_stroke}</param>
+            <param name="max">0</param>
           </command_interface>
           <state_interface name="position">

Commit message: fix(arm): restore historical ±90°/±200° hardware joint limits

File: src/arm/arm_description/urdf/arm_macro.xacro (robot description, xacro)
@@ -50,5 +50,5 @@
       <origin xyz="0.06 0 0.021" rpy="0 0 0"/>
       <axis xyz="0 0 1"/>
-      <limit lower="${-2*pi}" upper="${2*pi}" effort="100.0" velocity="1.0"/>
+      <limit lower="${-20*pi/18}" upper="${20*pi/18}" effort="100.0" velocity="1.0"/>
     </joint>
     <link name="arm_base_link">
@@ -67,5 +67,5 @@
       <origin xyz="-0.040366 -0.000325 0.103" rpy="${pi/3} 0 ${-pi}"/>
       <axis xyz="1 0 0"/>
-      <limit lower="${-2*pi}" upper="${2*pi}" effort="100.0" velocity="1.0"/>
+      <limit lower="${-20*pi/18}" upper="${20*pi/18}" effort="100.0" velocity="1.0"/>
     </joint>
     <link name="arm_shoulder_link">
@@ -84,5 +84,5 @@
       <origin xyz="0 0.3 0" rpy="${5*pi/12} 0 0"/>
       <axis xyz="1 0 0"/>
-      <limit lower="${-2*pi}" upper="${2*pi}" effort="100.0" velocity="1.0"/>
+      <limit lower="${-pi/2}" upper="${pi/2}" effort="100.0" velocity="1.0"/>
     </joint>
     <link name="arm_forearm_link">
@@ -101,5 +101,5 @@
       <origin xyz="-0.0173 0.3 0" rpy="0 ${pi/2} 0"/>
       <axis xyz="0 0 1"/>
-      <limit lower="${-2*pi}" upper="${2*pi}" effort="100.0" velocity="1.0"/>
+      <limit lower="${-20*pi/18}" upper="${20*pi/18}" effort="100.0" velocity="1.0"/>
     </joint>
     <link name="arm_wrist_1_link">
@@ -118,5 +118,5 @@
       <origin xyz="0.0323 0 -0.035" rpy="${-pi/2} 0 ${pi/2}"/>
       <axis xyz="0 0 1"/>
-      <limit lower="${-2*pi}" upper="${2*pi}" effort="100.0" velocity="1.0"/>
+      <limit lower="${-20*pi/18}" upper="${20*pi/18}" effort="100.0" velocity="1.0"/>
     </joint>
     <link name="arm_wrist_2_link">
@@ -135,5 +135,5 @@
       <origin xyz="0.0323 0 -0.035" rpy="${-pi/2} ${pi/3} ${-pi/2}"/>
       <axis xyz="0 0 1"/>
-      <limit lower="${-2*pi}" upper="${2*pi}" effort="100.0" velocity="1.0"/>
+      <limit lower="${-20*pi/18}" upper="${20*pi/18}" effort="100.0" velocity="1.0"/>
     </joint>
     <!-- Drill/sample masses+centroids: STL divergence-theorem volumes (not
