Commit message: feat: add astrobio as a real end_effector

File: src/arm/arm_description/urdf/arm_macro.xacro (robot description, xacro)
@@ -144,9 +144,28 @@
          gravity-comp <param>s below and the TEMP DEBUG VISUAL marker read
          from here. -->
-    <xacro:property name="ee_tool_com_x" value="-0.03"/>
-    <xacro:property name="ee_tool_com_y" value="-0.08"/>
-    <xacro:property name="ee_tool_com_z" value="0.05"/>
+    <xacro:property name="drill_ee_tool_com_x" value="-0.03"/>
+    <xacro:property name="drill_ee_tool_com_y" value="-0.08"/>
+    <xacro:property name="drill_ee_tool_com_z" value="0.05"/>
+    <!-- astrobio, physically mounted, has no mesh/finger geometry of its
+         own yet — reuses the jaw STL purely as a visual/collision stand-in
+         (see the xacro:if just below) and the jaw gravity-comp defaults as
+         a starting payload point, both by explicit request. CAN routing
+         (end_effector_can_node.py) and this payload are otherwise fully
+         separate from real jaw: 'astrobio' is its own end_effector value
+         everywhere (safe CAN no-op — no firmware yet — see can_bus.md;
+         its own poses.json "astrobio_home"; its own gravity-comp <param>
+         override below in <ros2_control>, gated on 'astrobio' specifically
+         so real jaw keeps using arm_hardware_interface.hpp's own tuned
+         default, 0.4kg/{0,0,0.06}, untouched). COM not yet measured —
+         starts at jaw's old default, tune against the TEMP DEBUG VISUAL
+         marker below. astrobio has NO finger joints modeled (see the
+         jaw-only xacro:if further below) — it shows as one rigid body,
+         matching that there is nothing to open/close on the CAN side either. -->
+    <xacro:property name="astrobio_ee_tool_mass_kg" value="0.4"/>
+    <xacro:property name="astrobio_ee_tool_com_x" value="0.0"/>
+    <xacro:property name="astrobio_ee_tool_com_y" value="0.0"/>
+    <xacro:property name="astrobio_ee_tool_com_z" value="0.08"/>
     <link name="arm_end_effector_link">
-      <xacro:if value="${'$(arg end_effector)' == 'jaw'}">
+      <xacro:if value="${('$(arg end_effector)' == 'jaw') or ('$(arg end_effector)' == 'astrobio')}">
         <visual>
           <geometry><mesh filename="${mesh_path}/arm_jaw_gripper_v3.stl" scale="${stl_scale}"/></geometry>
@@ -182,5 +201,18 @@
         <xacro:dummy_inertia mass="0.2"/>
       </xacro:if>
+      <!-- Matches astrobio_ee_tool_mass_kg above — keep in sync (this is
+           the sim/RViz-facing inertial mass, that one the real gravity-comp
+           payload; same number, two separate places by URDF/ros2_control's
+           own design, not a bug). -->
+      <xacro:if value="${'$(arg end_effector)' == 'astrobio'}">
+        <xacro:dummy_inertia mass="${astrobio_ee_tool_mass_kg}"/>
+      </xacro:if>
     </link>
+    <!-- Deliberately gated on 'jaw' ONLY, not astrobio too: astrobio has no
+         known finger/gripper mechanism (real hardware has no firmware for
+         it yet — see can_bus.md), so it gets no prismatic finger joints and
+         no gripper_right/left_controller (arm_bringup/arm.launch.py's own
+         gripper spawner condition is 'jaw' only already). It shows as one
+         rigid body reusing the jaw mesh above, nothing to open/close. -->
     <xacro:if value="${'$(arg end_effector)' == 'jaw'}">
       <!-- v3: no CAD dimension doc available (unlike v2 above). Derived from
@@ -263,5 +295,5 @@
       <parent link="arm_end_effector_link"/>
       <child link="arm_tcp_link"/>
-      <xacro:if value="${('$(arg end_effector)' == 'jaw') or ('$(arg end_effector)' == 'drill_sampling')}">
+      <xacro:if value="${('$(arg end_effector)' == 'jaw') or ('$(arg end_effector)' == 'drill_sampling') or ('$(arg end_effector)' == 'astrobio')}">
         <!-- v3: X=Y=0 by construction (right/left fingers are the same mesh
              mirrored 180 deg about Z through the shared origin, see the
@@ -279,8 +311,12 @@
              arm_tcp_link (indomitus_arm.srdf).
              drill_sampling deliberately shares this same point/axis (drill
-             mode rolls about arm_tcp_link's local Z). -->
+             mode rolls about arm_tcp_link's local Z). astrobio shares it
+             too: it reuses the jaw mesh (no fingers of its own — see the
+             xacro:if gating those, jaw-only), so its TCP is placed at the
+             same fingertip point that mesh actually renders at. Revisit
+             once astrobio has real geometry/reach of its own. -->
         <origin xyz="0 0 0.1615" rpy="0 0 0"/>
       </xacro:if>
-      <xacro:if value="${('$(arg end_effector)' != 'jaw') and ('$(arg end_effector)' != 'drill_sampling')}">
+      <xacro:if value="${('$(arg end_effector)' != 'jaw') and ('$(arg end_effector)' != 'drill_sampling') and ('$(arg end_effector)' != 'astrobio')}">
         <origin xyz="0 -0.23 0" rpy="0 0 0"/>
       </xacro:if>
@@ -344,14 +380,17 @@
     <link name="arm_camera_optical_frame"/>
     <!-- TEMP DEBUG VISUAL — sanity-check the assumed tool COM against the
-         real one by eye in RViz. Safe to delete this whole xacro:if block
-         when done; not wired into collision (visual only). Reads
-         ee_tool_com_x/y/z (declared above, also used by the gravity-comp
+         real one by eye in RViz, one red ball per end_effector. Safe to
+         delete this whole macro + xacro:if pair when done; not wired into
+         collision (visual only). Each branch reads that tool's own
+         *_ee_tool_com_x/y/z (declared above, also used by the gravity-comp
          <param>s in <ros2_control> below) — edit the properties, not this
-         origin, and both stay in sync automatically. -->
-    <xacro:if value="${'$(arg end_effector)' == 'drill_sampling'}">
+         origin, and both stay in sync automatically. Only one xacro:if
+         below is ever true for a given end_effector, so both are safe to
+         emit the same joint/link name. -->
+    <xacro:macro name="ee_tool_com_debug_marker" params="com_x com_y com_z">
       <joint name="arm_end_effector_com_debug_joint" type="fixed">
         <parent link="arm_end_effector_link"/>
         <child link="arm_end_effector_com_debug_link"/>
-        <origin xyz="${ee_tool_com_x} ${ee_tool_com_y} ${ee_tool_com_z}" rpy="0 0 0"/>
+        <origin xyz="${com_x} ${com_y} ${com_z}" rpy="0 0 0"/>
       </joint>
       <link name="arm_end_effector_com_debug_link">
@@ -363,4 +402,16 @@
         </visual>
       </link>
+    </xacro:macro>
+    <!-- No jaw branch here on purpose: real jaw's COM lives only in
+         arm_hardware_interface.hpp's own C++ default (0.4kg/{0,0,0.06}),
+         not exposed as an xacro property, so there is nothing for this
+         marker to read for end_effector:=jaw. -->
+    <xacro:if value="${'$(arg end_effector)' == 'astrobio'}">
+      <xacro:ee_tool_com_debug_marker
+        com_x="${astrobio_ee_tool_com_x}" com_y="${astrobio_ee_tool_com_y}" com_z="${astrobio_ee_tool_com_z}"/>
+    </xacro:if>
+    <xacro:if value="${'$(arg end_effector)' == 'drill_sampling'}">
+      <xacro:ee_tool_com_debug_marker
+        com_x="${drill_ee_tool_com_x}" com_y="${drill_ee_tool_com_y}" com_z="${drill_ee_tool_com_z}"/>
     </xacro:if>
     <ros2_control name="ArmSystem" type="system">
@@ -399,10 +450,19 @@
                  for how these were computed and cross-checked. jaw and
                  other_tool are left unset on purpose: ArmCanSystem's own
-                 defaults (0.4 kg, {0,0,0.06}) are the live-tuned jaw value
-                 from arm_hardware_interface.cpp — do not duplicate it here. -->
+                 defaults (0.4 kg, {0,0,0.06}) are the real jaw tool's tuned
+                 value from arm_hardware_interface.cpp — do not duplicate it
+                 here. astrobio DOES get an explicit override below — see
+                 astrobio_ee_tool_mass_kg/com_{x,y,z}'s own comment up at
+                 arm_end_effector_link. -->
+            <xacro:if value="${'$(arg end_effector)' == 'astrobio'}">
+              <param name="ee_tool_mass_kg">${astrobio_ee_tool_mass_kg}</param>
+              <param name="ee_tool_com_x">${astrobio_ee_tool_com_x}</param>
+              <param name="ee_tool_com_y">${astrobio_ee_tool_com_y}</param>
+              <param name="ee_tool_com_z">${astrobio_ee_tool_com_z}</param>
+            </xacro:if>
             <xacro:if value="${'$(arg end_effector)' == 'drill_sampling'}">
               <!-- Mass-weighted COM of drill (2.0kg) + sample (0.6kg), raw-frame
                    value rotated to match the <origin rpy="0 pi pi/2"> above —
-                   keep in sync if that changes. Values (ee_tool_com_x/y/z
+                   keep in sync if that changes. Values (drill_ee_tool_com_x/y/z
                    properties, declared up at arm_end_effector_link) have been
                    retuned repeatedly on explicit request after live testing
@@ -413,7 +473,7 @@
                    TEMP DEBUG VISUAL marker above reads the same properties. -->
               <param name="ee_tool_mass_kg">2.8</param>
-              <param name="ee_tool_com_x">${ee_tool_com_x}</param>
-              <param name="ee_tool_com_y">${ee_tool_com_y}</param>
-              <param name="ee_tool_com_z">${ee_tool_com_z}</param>
+              <param name="ee_tool_com_x">${drill_ee_tool_com_x}</param>
+              <param name="ee_tool_com_y">${drill_ee_tool_com_y}</param>
+              <param name="ee_tool_com_z">${drill_ee_tool_com_z}</param>
             </xacro:if>
           </xacro:unless>

Commit message: feat(arm): add probing container position

File: src/arm/arm_description/urdf/arm_macro.xacro (robot description, xacro)
@@ -48,7 +48,7 @@
       <parent link="arm_mount_link"/>
       <child link="arm_base_link"/>
-      <origin xyz="0.06 0 0.021" rpy="0 0 0"/>
+      <origin xyz="0.06 0 0.021" rpy="0 0 ${-pi/2}"/>
       <axis xyz="0 0 1"/>
-      <limit lower="${-20*pi/18}" upper="${20*pi/18}" effort="100.0" velocity="1.0"/>
+      <limit lower="${-pi/2}" upper="${pi/2}" effort="100.0" velocity="1.0"/>
     </joint>
     <link name="arm_base_link">

Commit message: chore(arm_description): limits for arm_mount_base_joint updated

File: src/arm/arm_description/urdf/arm_macro.xacro (robot description, xacro)
@@ -50,5 +50,5 @@
       <origin xyz="0.06 0 0.021" rpy="0 0 ${-pi/2}"/>
       <axis xyz="0 0 1"/>
-      <limit lower="${-pi/2}" upper="${pi/2}" effort="100.0" velocity="1.0"/>
+      <limit lower="${-pi}" upper="${0}" effort="100.0" velocity="1.0"/>
     </joint>
     <link name="arm_base_link">

Commit message: fixes to make simulation with rover and arm possible

File: src/arm/arm_description/urdf/arm_macro.xacro (robot description, xacro)
@@ -5,12 +5,4 @@
   <xacro:arg name="sim" default="false"/>
   <xacro:arg name="can_interface" default="can0"/>
-  <!-- When the arm is mounted into another robot's URDF (e.g. the rover, see
-       rover_description's mount_arm arg) that outer URDF already adds its
-       own single gz_ros2_control-system plugin covering every <ros2_control>
-       block in the combined model. Set this to false in that case so the
-       arm doesn't register a second, redundant controller_manager plugin
-       for the same Gazebo model. Standalone arm sim (arm_sim) leaves this
-       at the default so it keeps adding its own plugin as before. -->
-  <xacro:arg name="standalone_gz_plugin" default="true"/>
   <!-- camera:=false drops the simulated camera sensor (the URDF link and
        frames stay). Camera rendering is the main real-time-factor cost
@@ -578,12 +570,8 @@
       </ros2_control>
     </xacro:if>
+    <!-- No gz_ros2_control plugin here: the assembly that gets spawned into
+         Gazebo adds it (arm_standalone.urdf.xacro for arm-only sim,
+         indomitus_description's indomitus_gz.urdf.xacro when mounted). -->
     <xacro:if value="$(arg sim)">
-      <xacro:if value="$(arg standalone_gz_plugin)">
-        <gazebo>
-          <plugin filename="gz_ros2_control-system" name="gz_ros2_control::GazeboSimROS2ControlPlugin">
-            <parameters>$(find arm_sim)/config/ros2_controllers.yaml</parameters>
-          </plugin>
-        </gazebo>
-      </xacro:if>
       <gazebo reference="arm_mount_link">
         <visual>

File: src/arm/arm_description/urdf/arm_standalone.urdf.xacro (robot description, xacro)
@@ -1,4 +1,5 @@
 <?xml version="1.0"?>
 <robot name="indomitus_arm" xmlns:xacro="http://www.ros.org/wiki/xacro">
+  <!-- Arm-only assembly. The world root fixes the model in Gazebo. -->
   <xacro:arg name="end_effector" default="jaw"/>
   <xacro:include filename="$(find arm_description)/urdf/arm_macro.xacro"/>
@@ -7,3 +8,15 @@
     <origin xyz="0 0 0" rpy="0 0 0"/>
   </xacro:indomitus_arm>
+  <!-- Its controller_manager lives under /arm, same as on hardware, and
+       reads robot_description from /arm/robot_state_publisher. -->
+  <xacro:if value="$(arg sim)">
+    <gazebo>
+      <plugin filename="gz_ros2_control-system" name="gz_ros2_control::GazeboSimROS2ControlPlugin">
+        <ros>
+          <namespace>/arm</namespace>
+        </ros>
+        <parameters>$(find arm_sim)/config/ros2_controllers.yaml</parameters>
+      </plugin>
+    </gazebo>
+  </xacro:if>
 </robot>

File: src/panel/panel_description/urdf/panel_macro.xacro (robot description, xacro)
@@ -660,5 +660,5 @@
       <!-- panel_base_link only: no gravity, so the board itself neither
            falls nor tips over on sloped terrain and just sits exactly at
-           its spawn pose (see panel_x/y/z/yaw in sim_gz_full.launch.py).
+           its spawn pose (see panel_x/y/z/yaw in indomitus_bringup/sim_rover_arm.launch.py).
            This means that pose must now match the real terrain height by
            hand: there is no physics settling to correct a wrong z.

File: src/rover_description/urdf/rover.urdf.xacro (robot description, xacro)
@@ -7,7 +7,4 @@
   <xacro:include filename="$(find rover_description)/urdf/macros/stereo_camera.xacro"/>
   <xacro:include filename="$(find rover_description)/urdf/macros/lidar.xacro"/>
-  <xacro:if value="$(arg mount_arm)">
-    <xacro:include filename="$(find arm_description)/urdf/arm_macro.xacro"/>
-  </xacro:if>
   <!-- ===================== MATERIALS ===================== -->
   <material name="blue_body">
@@ -128,11 +125,3 @@
   <xacro:stop_button_accessory suffix="l" y_sign="1"/>
   <xacro:stop_button_accessory suffix="r" y_sign="-1"/>
-  <!-- ===================== ARM (OPTIONAL) ===================== -->
-  <!-- Placeholder mount pose; update once the real MR_ARM_ATT attachment
-       point from CAD is known. -->
-  <xacro:if value="$(arg mount_arm)">
-    <xacro:indomitus_arm parent_link="main_body_link">
-      <origin xyz="0.2 0 0.1" rpy="0 0 0"/>
-    </xacro:indomitus_arm>
-  </xacro:if>
 </robot>

File: src/rover_description/urdf/rover.xacro (robot description, xacro)
@@ -17,6 +17,4 @@
   <xacro:arg name="stereo_camera_simulate_depth" default="false"/>
   <xacro:arg name="stereo_camera_simulate_imu" default="true"/>
-  <!-- mount_arm:=true bolts the indomitus_arm onto main_body_link.-->
-  <xacro:arg name="mount_arm" default="false"/>
   <!-- Main robot description -->
   <xacro:include filename="$(find rover_description)/urdf/rover.urdf.xacro"/>

Commit message: fix incorrect offset, poses. fix closure of keyboard_servo_node

File: src/arm/arm_description/urdf/arm_macro.xacro (robot description, xacro)
@@ -42,5 +42,7 @@
       <origin xyz="0.06 0 0.021" rpy="0 0 ${-pi/2}"/>
       <axis xyz="0 0 1"/>
-      <limit lower="${-pi}" upper="${0}" effort="100.0" velocity="1.0"/>
+      <!-- 0 = facing straight ahead along arm_mount_link (with the -pi/2
+           origin yaw above), +-90 deg either side. -->
+      <limit lower="${-pi/2}" upper="${pi/2}" effort="100.0" velocity="1.0"/>
     </joint>
     <link name="arm_base_link">

File: src/indomitus_description/urdf/mount.xacro (robot description, xacro)
@@ -5,8 +5,7 @@
        indomitus_gz.urdf.xacro (Gazebo model) mount the arm through this
        macro, so TF and physics always agree. -->
-  <!-- TODO: placeholder carried over from the old mount_arm block. The real
-       pose must come from CAD (MR_ARM_ATT); this one sits inside the
-       main body box. -->
-  <xacro:property name="arm_mount_xyz" value="0.2 0 0.1"/>
+  <!-- Checked by eye against the real rover; the base sitting inside the
+       main body box is expected. -->
+  <xacro:property name="arm_mount_xyz" value="0.17 0 0.12"/>
   <xacro:property name="arm_mount_rpy" value="0 0 0"/>
   <xacro:include filename="$(find arm_description)/urdf/arm_macro.xacro"/>

Commit message: add package for cameras

File: src/arm/arm_description/urdf/arm_macro.xacro (robot description, xacro)
@@ -337,6 +337,6 @@
           <box size="0.035 0.035 0.05"/>
         </geometry>
-        <material name="camera_blue">
-          <color rgba="0.0 0.0 1.0 1.0"/>
+        <material name="camera_black">
+          <color rgba="0.05 0.05 0.05 1.0"/>
         </material>
       </visual>

File: src/rover/rover_description/urdf/properties.xacro (robot description, xacro)
@@ -82,4 +82,30 @@
   <xacro:property name="zed2i_ry" value="${pi/12}"/>
   <xacro:property name="zed2i_rz" value="0.0"/>
+  <!-- ===================== CAMERA MAST ===================== -->
+  <!-- Vertical 2x2 cm pole on the rear face of the main body, 1 m tall, its bottom
+       level with the body's bottom. Centred left-right: CALIBRATE (measure). -->
+  <xacro:property name="mast_size" value="0.02"/>
+  <xacro:property name="mast_height" value="1.0"/>
+  <xacro:property name="mast_mass" value="0.3"/>
+  <xacro:property name="mast_x" value="${-body_length / 2.0 - mast_size / 2.0}"/>
+  <xacro:property name="mast_y" value="0.0"/>
+  <xacro:property name="mast_z" value="${-body_height / 2.0 + mast_height / 2.0}"/>
+  <!-- ===================== USB CAMERAS (rover_cameras) ===================== -->
+  <!-- Hand-measured mounting poses, relative to the parent link's origin; pitch > 0
+       looks down. Every value marked CALIBRATE is a tape-measure estimate to replace
+       with an extrinsic calibration (grep CALIBRATE). -->
+  <!-- arducam-fr-bottom: under the main body, 15 cm forward of its centre, 3 cm below
+       its bottom, looking forward 15 deg down. CALIBRATE: y (assumed centred), z, pitch. -->
+  <xacro:property name="arducam_fr_bottom_x" value="0.15"/>
+  <xacro:property name="arducam_fr_bottom_y" value="0.0"/>
+  <xacro:property name="arducam_fr_bottom_z" value="${-body_height / 2.0 - 0.03}"/>
+  <xacro:property name="arducam_fr_bottom_pitch" value="${15.0 * pi / 180.0}"/>
+  <!-- arducam-mast: on the mast (relative to mast_link, the pole's centre), 5 cm
+       below its top, 2 cm to the left of the pole, looking forward 25 deg down.
+       CALIBRATE: y (2 cm from the pole's axis assumed), x, pitch. -->
+  <xacro:property name="arducam_mast_x" value="0.0"/>
+  <xacro:property name="arducam_mast_y" value="0.02"/>
+  <xacro:property name="arducam_mast_z" value="${mast_height / 2.0 - 0.05}"/>
+  <xacro:property name="arducam_mast_pitch" value="${25.0 * pi / 180.0}"/>
   <!-- ===================== LIDAR POSSITION ===================== -->
   <xacro:property name="lidar_x" value="0.0"/>

File: src/rover/rover_description/urdf/rover.urdf.xacro (robot description, xacro)
@@ -7,4 +7,5 @@
   <xacro:include filename="$(find rover_description)/urdf/macros/stereo_camera.xacro"/>
   <xacro:include filename="$(find rover_description)/urdf/macros/lidar.xacro"/>
+  <xacro:include filename="$(find rover_description)/urdf/macros/usb_camera.xacro"/>
   <!-- ===================== MATERIALS ===================== -->
   <material name="blue_body">
@@ -121,4 +122,39 @@
     <origin xyz="${lidar_x} ${lidar_y} ${lidar_z}" rpy="0 0 0"/>
   </joint>
+  <!-- ===================== CAMERA MAST ===================== -->
+  <link name="mast_link">
+    <inertial>
+      <origin xyz="0 0 0" rpy="0 0 0"/>
+      <mass value="${mast_mass}"/>
+      <xacro:box_inertia m="${mast_mass}" x="${mast_size}" y="${mast_size}" z="${mast_height}"/>
+    </inertial>
+    <visual>
+      <geometry>
+        <box size="${mast_size} ${mast_size} ${mast_height}"/>
+      </geometry>
+      <material name="grey_structure"/>
+    </visual>
+    <collision>
+      <geometry>
+        <box size="${mast_size} ${mast_size} ${mast_height}"/>
+      </geometry>
+    </collision>
+  </link>
+  <joint name="mast_joint" type="fixed">
+    <parent link="main_body_link"/>
+    <child link="mast_link"/>
+    <origin xyz="${mast_x} ${mast_y} ${mast_z}" rpy="0 0 0"/>
+  </joint>
+  <!-- ===================== USB CAMERAS (rover_cameras) ===================== -->
+  <!-- Poses in properties.xacro (CALIBRATE markers). Not yet modelled:
+       arducam-front, thermal-camera-front (positions unknown). -->
+  <xacro:usb_camera name="arducam_fr_bottom" parent="main_body_link">
+    <origin xyz="${arducam_fr_bottom_x} ${arducam_fr_bottom_y} ${arducam_fr_bottom_z}"
+            rpy="0 ${arducam_fr_bottom_pitch} 0"/>
+  </xacro:usb_camera>
+  <xacro:usb_camera name="arducam_mast" parent="mast_link">
+    <origin xyz="${arducam_mast_x} ${arducam_mast_y} ${arducam_mast_z}"
+            rpy="0 ${arducam_mast_pitch} 0"/>
+  </xacro:usb_camera>
   <!-- ===================== ROCKERS + WHEELS ===================== -->
   <xacro:rocker_assembly side="l" y_sign="1"/>
