Commit message: chore: location of the lidar xacro cahnged, stl for the zed2i removed

File: src/rover_description/urdf/macros/lidar.xacro (robot description, xacro)
@@ -20,5 +20,5 @@
         <origin xyz="0 0 -0.057" rpy="-1.5708 0 3.1416"/>
         <geometry>
-          <mesh filename="package://rover_description/meshes/navigation/lidar/rplidar_s2.stl" scale="0.001 0.001 0.001"/>
+          <mesh filename="package://rover_description/meshes/navigation/rplidar_s2.stl" scale="0.001 0.001 0.001"/>
         </geometry>
         <material name="lidar_black"/>
