Commit message: fix(panel): resolve panel placement, ArUco orientation, and MoveIt frame bugs blocking align

File: src/panel/panel_description/urdf/panel_standalone.urdf.xacro (robot description, xacro)
@@ -2,10 +2,15 @@
 <robot name="indomitus_panel" xmlns:xacro="http://www.ros.org/wiki/xacro">
   <xacro:include filename="$(find panel_description)/urdf/panel_macro.xacro"/>
-  <!-- Must match whatever pose the panel is actually spawned at in Gazebo
-       (e.g. sim_gz_full.launch.py's panel_x/panel_y/panel_z/panel_yaw
-       launch args), or the published world -> panel_base_link TF will
-       disagree with where the model physically is. Defaults to identity
-       for standalone visualization (panel_standalone.launch.py), where
-       there is no separate spawn pose to match. -->
+  <!-- panel_x/y/z/yaw are declared for callers that pass them (e.g.
+       arm_gazebo.launch.py's Command(...) invocation), but must NOT also
+       be applied here: arm_gazebo.launch.py's ros_gz_sim spawn already
+       places this model's root ("world" link) at that exact pose in
+       Gazebo. Reapplying the same offset to panel_mount_joint here would
+       place panel_base_link there A SECOND TIME, relative to the
+       already-offset "world" link. Confirmed live via TF as an actual
+       bug (panel_base_link ended up at a doubled offset/rotation from
+       the intended spawn pose, ~1m and ~30 deg off). This joint's origin
+       must stay identity; the physical/TF placement is the spawn
+       command's job alone. -->
   <xacro:arg name="panel_x" default="0"/>
   <xacro:arg name="panel_y" default="0"/>
@@ -14,5 +19,5 @@
   <link name="world"/>
   <xacro:indomitus_panel parent_link="world">
-    <origin xyz="$(arg panel_x) $(arg panel_y) $(arg panel_z)" rpy="0 0 $(arg panel_yaw)"/>
+    <origin xyz="0 0 0" rpy="0 0 0"/>
   </xacro:indomitus_panel>
 </robot>
