Commit message: feat(panel): color-code panel elements and add indicators/sockets/markers

File: src/panel/panel_description/urdf/panel_macro.xacro (robot description, xacro)
@@ -20,4 +20,19 @@
       <color rgba="0.5 0.5 0.55 1.0"/>
     </material>
+    <material name="power_switch_pink">
+      <color rgba="0.83 0.42 0.5 1.0"/>
+    </material>
+    <material name="breaker_white">
+      <color rgba="0.92 0.92 0.92 1.0"/>
+    </material>
+    <material name="indicator_green">
+      <color rgba="0.25 0.85 0.3 1.0"/>
+    </material>
+    <material name="socket_grey">
+      <color rgba="0.65 0.65 0.68 1.0"/>
+    </material>
+    <material name="marker_black">
+      <color rgba="0.03 0.03 0.03 1.0"/>
+    </material>
     <xacro:macro name="dummy_inertia" params="mass">
       <inertial>
@@ -61,5 +76,5 @@
       <visual>
         <geometry><mesh filename="${mesh_path}/main_switch.stl" scale="${stl_scale}"/></geometry>
-        <material name="panel_grey"/>
+        <material name="power_switch_pink"/>
       </visual>
       <collision>
@@ -81,5 +96,5 @@
       <visual>
         <geometry><mesh filename="${mesh_path}/main_switch.stl" scale="${stl_scale}"/></geometry>
-        <material name="panel_grey"/>
+        <material name="power_switch_pink"/>
       </visual>
       <collision>
@@ -201,5 +216,5 @@
       <visual>
         <geometry><mesh filename="${mesh_path}/MCB_1P.stl" scale="${stl_scale}"/></geometry>
-        <material name="panel_grey"/>
+        <material name="breaker_white"/>
       </visual>
       <collision>
@@ -221,5 +236,5 @@
       <visual>
         <geometry><mesh filename="${mesh_path}/MCB_1P.stl" scale="${stl_scale}"/></geometry>
-        <material name="panel_grey"/>
+        <material name="breaker_white"/>
       </visual>
       <collision>
@@ -241,5 +256,5 @@
       <visual>
         <geometry><mesh filename="${mesh_path}/MCB_1P.stl" scale="${stl_scale}"/></geometry>
-        <material name="panel_grey"/>
+        <material name="breaker_white"/>
       </visual>
       <collision>
@@ -261,5 +276,5 @@
       <visual>
         <geometry><mesh filename="${mesh_path}/MCB_1P.stl" scale="${stl_scale}"/></geometry>
-        <material name="panel_grey"/>
+        <material name="breaker_white"/>
       </visual>
       <collision>
@@ -281,5 +296,5 @@
       <visual>
         <geometry><mesh filename="${mesh_path}/MCB_1P.stl" scale="${stl_scale}"/></geometry>
-        <material name="panel_grey"/>
+        <material name="breaker_white"/>
       </visual>
       <collision>
@@ -301,5 +316,5 @@
       <visual>
         <geometry><mesh filename="${mesh_path}/MCB_1P.stl" scale="${stl_scale}"/></geometry>
-        <material name="panel_grey"/>
+        <material name="breaker_white"/>
       </visual>
       <collision>
@@ -321,5 +336,5 @@
       <visual>
         <geometry><mesh filename="${mesh_path}/MCB_1P.stl" scale="${stl_scale}"/></geometry>
-        <material name="panel_grey"/>
+        <material name="breaker_white"/>
       </visual>
       <collision>
@@ -341,5 +356,5 @@
       <visual>
         <geometry><mesh filename="${mesh_path}/MCB_1P.stl" scale="${stl_scale}"/></geometry>
-        <material name="panel_grey"/>
+        <material name="breaker_white"/>
       </visual>
       <collision>
@@ -361,5 +376,5 @@
       <visual>
         <geometry><mesh filename="${mesh_path}/MCB_1P.stl" scale="${stl_scale}"/></geometry>
-        <material name="panel_grey"/>
+        <material name="breaker_white"/>
       </visual>
       <collision>
@@ -381,5 +396,5 @@
       <visual>
         <geometry><mesh filename="${mesh_path}/MCB_1P.stl" scale="${stl_scale}"/></geometry>
-        <material name="panel_grey"/>
+        <material name="breaker_white"/>
       </visual>
       <collision>
@@ -401,5 +416,5 @@
       <visual>
         <geometry><mesh filename="${mesh_path}/MCB_1P.stl" scale="${stl_scale}"/></geometry>
-        <material name="panel_grey"/>
+        <material name="breaker_white"/>
       </visual>
       <collision>
@@ -421,5 +436,5 @@
       <visual>
         <geometry><mesh filename="${mesh_path}/MCB_1P.stl" scale="${stl_scale}"/></geometry>
-        <material name="panel_grey"/>
+        <material name="breaker_white"/>
       </visual>
       <collision>
@@ -441,5 +456,5 @@
       <visual>
         <geometry><mesh filename="${mesh_path}/MCB_1P.stl" scale="${stl_scale}"/></geometry>
-        <material name="panel_grey"/>
+        <material name="breaker_white"/>
       </visual>
       <collision>
@@ -461,5 +476,5 @@
       <visual>
         <geometry><mesh filename="${mesh_path}/MCB_1P.stl" scale="${stl_scale}"/></geometry>
-        <material name="panel_grey"/>
+        <material name="breaker_white"/>
       </visual>
       <collision>
@@ -481,5 +496,5 @@
       <visual>
         <geometry><mesh filename="${mesh_path}/MCB_1P.stl" scale="${stl_scale}"/></geometry>
-        <material name="panel_grey"/>
+        <material name="breaker_white"/>
       </visual>
       <collision>
@@ -501,5 +516,5 @@
       <visual>
         <geometry><mesh filename="${mesh_path}/MCB_1P.stl" scale="${stl_scale}"/></geometry>
-        <material name="panel_grey"/>
+        <material name="breaker_white"/>
       </visual>
       <collision>
@@ -521,11 +536,90 @@
       <visual>
         <geometry><mesh filename="${mesh_path}/MCB_1P.stl" scale="${stl_scale}"/></geometry>
-        <material name="panel_grey"/>
-      </visual>
-      <collision>
-        <geometry><mesh filename="${mesh_path}/MCB_1P.stl" scale="${stl_scale}"/></geometry>
-      </collision>
-      <xacro:dummy_inertia mass="0.01"/>
-    </link>
+        <material name="breaker_white"/>
+      </visual>
+      <collision>
+        <geometry><mesh filename="${mesh_path}/MCB_1P.stl" scale="${stl_scale}"/></geometry>
+      </collision>
+      <xacro:dummy_inertia mass="0.01"/>
+    </link>
+    <!-- ===================== INDICATOR LIGHTS (primitive, no STL) =====================
+         Row of 5 status LEDs above the breaker row, per "All of the five
+         indicators are lit up" in the Expected Results. No source mesh for
+         these exists, so they're flat green boxes flush with the panel
+         face — positioned/sized by eye against the reference render, same
+         placeholder-until-verified caveat as everything else in this file. -->
+    <xacro:macro name="panel_indicator" params="suffix x z">
+      <joint name="panel_indicator_${suffix}_joint" type="fixed">
+        <parent link="panel_base_link"/>
+        <child link="panel_indicator_${suffix}_link"/>
+        <origin xyz="${x} -0.003 ${z}" rpy="0 0 0"/>
+      </joint>
+      <link name="panel_indicator_${suffix}_link">
+        <visual>
+          <geometry><box size="0.022 0.004 0.014"/></geometry>
+          <material name="indicator_green"/>
+        </visual>
+        <collision>
+          <geometry><box size="0.022 0.004 0.014"/></geometry>
+        </collision>
+        <xacro:dummy_inertia mass="0.001"/>
+      </link>
+    </xacro:macro>
+    <xacro:panel_indicator suffix="1" x="-0.119578" z="0.365"/>
+    <xacro:panel_indicator suffix="2" x="-0.059789" z="0.365"/>
+    <xacro:panel_indicator suffix="3" x="0"         z="0.365"/>
+    <xacro:panel_indicator suffix="4" x="0.059789"  z="0.365"/>
+    <xacro:panel_indicator suffix="5" x="0.119578"  z="0.365"/>
+    <!-- ===================== SOCKETS (primitive, no STL) =====================
+         The two IEC320 C14 plug sockets ("insert the plug into one of the
+         two sockets"), placed left of the pink rotary power switches at the
+         same row height (panel_main_switch_1/2 are at z=0.109905). Small
+         grey cylinders standing proud of the panel face. -->
+    <xacro:macro name="panel_socket" params="suffix x z">
+      <joint name="panel_socket_${suffix}_joint" type="fixed">
+        <parent link="panel_base_link"/>
+        <child link="panel_socket_${suffix}_link"/>
+        <origin xyz="${x} -0.006 ${z}" rpy="${pi/2} 0 0"/>
+      </joint>
+      <link name="panel_socket_${suffix}_link">
+        <visual>
+          <geometry><cylinder radius="0.012" length="0.012"/></geometry>
+          <material name="socket_grey"/>
+        </visual>
+        <collision>
+          <geometry><cylinder radius="0.012" length="0.012"/></geometry>
+        </collision>
+        <xacro:dummy_inertia mass="0.005"/>
+      </link>
+    </xacro:macro>
+    <xacro:panel_socket suffix="1" x="-0.10" z="0.109905"/>
+    <xacro:panel_socket suffix="2" x="-0.06" z="0.109905"/>
+    <!-- ===================== ArUco MARKER MOUNTS (primitive, no STL) =====================
+         Flat black squares for pose-detection markers ("AruCo detection"
+         in the scoring sheet). Three of the four corners are marked in the
+         reference render (top-left, top-right, bottom-left) — the actual
+         ArUco pattern (numbered tag) is applied as a texture/decal on top
+         of this base square by whichever code renders/prints the markers;
+         this link is just the physical black mount square. -->
+    <xacro:macro name="panel_marker" params="suffix x z">
+      <joint name="panel_marker_${suffix}_joint" type="fixed">
+        <parent link="panel_base_link"/>
+        <child link="panel_marker_${suffix}_link"/>
+        <origin xyz="${x} -0.003 ${z}" rpy="0 0 0"/>
+      </joint>
+      <link name="panel_marker_${suffix}_link">
+        <visual>
+          <geometry><box size="0.04 0.002 0.04"/></geometry>
+          <material name="marker_black"/>
+        </visual>
+        <collision>
+          <geometry><box size="0.04 0.002 0.04"/></geometry>
+        </collision>
+        <xacro:dummy_inertia mass="0.001"/>
+      </link>
+    </xacro:macro>
+    <xacro:panel_marker suffix="top_left"    x="-0.135" z="0.415"/>
+    <xacro:panel_marker suffix="top_right"   x="0.135"  z="0.415"/>
+    <xacro:panel_marker suffix="bottom_left" x="-0.135" z="0.035"/>
     <xacro:if value="$(arg sim)">
       <!-- panel_base_link only: no gravity, so the board itself neither

Commit message: fix(panel): sync Gazebo spawn pose with TF, add frame_prefix, fix breaker limits

File: src/panel/panel_description/urdf/panel_macro.xacro (robot description, xacro)
@@ -210,5 +210,5 @@
       <origin xyz="-0.150607 0.000926 0.305081" rpy="0 0 0"/>
       <axis xyz="1 0 0"/>
-      <limit lower="${pi/6}" upper="${pi/2}" effort="5.0" velocity="2.0"/>
+      <limit lower="0" upper="${pi/3}" effort="5.0" velocity="2.0"/>
       <dynamics damping="0.02" friction="0.02"/>
     </joint>
@@ -230,5 +230,5 @@
       <origin xyz="-0.132607 0.000926 0.305081" rpy="0 0 0"/>
       <axis xyz="1 0 0"/>
-      <limit lower="${pi/6}" upper="${pi/2}" effort="5.0" velocity="2.0"/>
+      <limit lower="0" upper="${pi/3}" effort="5.0" velocity="2.0"/>
       <dynamics damping="0.02" friction="0.02"/>
     </joint>
@@ -250,5 +250,5 @@
       <origin xyz="-0.114607 0.000926 0.305081" rpy="0 0 0"/>
       <axis xyz="1 0 0"/>
-      <limit lower="${pi/6}" upper="${pi/2}" effort="5.0" velocity="2.0"/>
+      <limit lower="0" upper="${pi/3}" effort="5.0" velocity="2.0"/>
       <dynamics damping="0.02" friction="0.02"/>
     </joint>
@@ -270,5 +270,5 @@
       <origin xyz="-0.096607 0.000926 0.305081" rpy="0 0 0"/>
       <axis xyz="1 0 0"/>
-      <limit lower="${pi/6}" upper="${pi/2}" effort="5.0" velocity="2.0"/>
+      <limit lower="0" upper="${pi/3}" effort="5.0" velocity="2.0"/>
       <dynamics damping="0.02" friction="0.02"/>
     </joint>
@@ -290,5 +290,5 @@
       <origin xyz="-0.078607 0.000926 0.305081" rpy="0 0 0"/>
       <axis xyz="1 0 0"/>
-      <limit lower="${pi/6}" upper="${pi/2}" effort="5.0" velocity="2.0"/>
+      <limit lower="0" upper="${pi/3}" effort="5.0" velocity="2.0"/>
       <dynamics damping="0.02" friction="0.02"/>
     </joint>
@@ -310,5 +310,5 @@
       <origin xyz="-0.060607 0.000926 0.305081" rpy="0 0 0"/>
       <axis xyz="1 0 0"/>
-      <limit lower="${pi/6}" upper="${pi/2}" effort="5.0" velocity="2.0"/>
+      <limit lower="0" upper="${pi/3}" effort="5.0" velocity="2.0"/>
       <dynamics damping="0.02" friction="0.02"/>
     </joint>
@@ -330,5 +330,5 @@
       <origin xyz="-0.042607 0.000926 0.305081" rpy="0 0 0"/>
       <axis xyz="1 0 0"/>
-      <limit lower="${pi/6}" upper="${pi/2}" effort="5.0" velocity="2.0"/>
+      <limit lower="0" upper="${pi/3}" effort="5.0" velocity="2.0"/>
       <dynamics damping="0.02" friction="0.02"/>
     </joint>
@@ -350,5 +350,5 @@
       <origin xyz="-0.024607 0.000926 0.305081" rpy="0 0 0"/>
       <axis xyz="1 0 0"/>
-      <limit lower="${pi/6}" upper="${pi/2}" effort="5.0" velocity="2.0"/>
+      <limit lower="0" upper="${pi/3}" effort="5.0" velocity="2.0"/>
       <dynamics damping="0.02" friction="0.02"/>
     </joint>
@@ -370,5 +370,5 @@
       <origin xyz="-0.006607 0.000926 0.305081" rpy="0 0 0"/>
       <axis xyz="1 0 0"/>
-      <limit lower="${pi/6}" upper="${pi/2}" effort="5.0" velocity="2.0"/>
+      <limit lower="0" upper="${pi/3}" effort="5.0" velocity="2.0"/>
       <dynamics damping="0.02" friction="0.02"/>
     </joint>
@@ -390,5 +390,5 @@
       <origin xyz="0.011393 0.000926 0.305081" rpy="0 0 0"/>
       <axis xyz="1 0 0"/>
-      <limit lower="${pi/6}" upper="${pi/2}" effort="5.0" velocity="2.0"/>
+      <limit lower="0" upper="${pi/3}" effort="5.0" velocity="2.0"/>
       <dynamics damping="0.02" friction="0.02"/>
     </joint>
@@ -410,5 +410,5 @@
       <origin xyz="0.029393 0.000926 0.305081" rpy="0 0 0"/>
       <axis xyz="1 0 0"/>
-      <limit lower="${pi/6}" upper="${pi/2}" effort="5.0" velocity="2.0"/>
+      <limit lower="0" upper="${pi/3}" effort="5.0" velocity="2.0"/>
       <dynamics damping="0.02" friction="0.02"/>
     </joint>
@@ -430,5 +430,5 @@
       <origin xyz="0.047393 0.000926 0.305081" rpy="0 0 0"/>
       <axis xyz="1 0 0"/>
-      <limit lower="${pi/6}" upper="${pi/2}" effort="5.0" velocity="2.0"/>
+      <limit lower="0" upper="${pi/3}" effort="5.0" velocity="2.0"/>
       <dynamics damping="0.02" friction="0.02"/>
     </joint>
@@ -450,5 +450,5 @@
       <origin xyz="0.065393 0.000926 0.305081" rpy="0 0 0"/>
       <axis xyz="1 0 0"/>
-      <limit lower="${pi/6}" upper="${pi/2}" effort="5.0" velocity="2.0"/>
+      <limit lower="0" upper="${pi/3}" effort="5.0" velocity="2.0"/>
       <dynamics damping="0.02" friction="0.02"/>
     </joint>
@@ -470,5 +470,5 @@
       <origin xyz="0.083393 0.000926 0.305081" rpy="0 0 0"/>
       <axis xyz="1 0 0"/>
-      <limit lower="${pi/6}" upper="${pi/2}" effort="5.0" velocity="2.0"/>
+      <limit lower="0" upper="${pi/3}" effort="5.0" velocity="2.0"/>
       <dynamics damping="0.02" friction="0.02"/>
     </joint>
@@ -490,5 +490,5 @@
       <origin xyz="0.101393 0.000926 0.305081" rpy="0 0 0"/>
       <axis xyz="1 0 0"/>
-      <limit lower="${pi/6}" upper="${pi/2}" effort="5.0" velocity="2.0"/>
+      <limit lower="0" upper="${pi/3}" effort="5.0" velocity="2.0"/>
       <dynamics damping="0.02" friction="0.02"/>
     </joint>
@@ -510,5 +510,5 @@
       <origin xyz="0.119393 0.000926 0.305081" rpy="0 0 0"/>
       <axis xyz="1 0 0"/>
-      <limit lower="${pi/6}" upper="${pi/2}" effort="5.0" velocity="2.0"/>
+      <limit lower="0" upper="${pi/3}" effort="5.0" velocity="2.0"/>
       <dynamics damping="0.02" friction="0.02"/>
     </joint>
@@ -530,5 +530,5 @@
       <origin xyz="0.137393 0.000926 0.305081" rpy="0 0 0"/>
       <axis xyz="1 0 0"/>
-      <limit lower="${pi/6}" upper="${pi/2}" effort="5.0" velocity="2.0"/>
+      <limit lower="0" upper="${pi/3}" effort="5.0" velocity="2.0"/>
       <dynamics damping="0.02" friction="0.02"/>
     </joint>

File: src/panel/panel_description/urdf/panel_standalone.urdf.xacro (robot description, xacro)
@@ -2,7 +2,17 @@
 <robot name="indomitus_panel" xmlns:xacro="http://www.ros.org/wiki/xacro">
   <xacro:include filename="$(find panel_description)/urdf/panel_macro.xacro"/>
+  <!-- Must match whatever pose the panel is actually spawned at in Gazebo
+       (e.g. sim_gz_full.launch.py's panel_x/panel_y/panel_z/panel_yaw
+       launch args), or the published world -> panel_base_link TF will
+       disagree with where the model physically is. Defaults to identity
+       for standalone visualization (panel_standalone.launch.py), where
+       there is no separate spawn pose to match. -->
+  <xacro:arg name="panel_x" default="0"/>
+  <xacro:arg name="panel_y" default="0"/>
+  <xacro:arg name="panel_z" default="0"/>
+  <xacro:arg name="panel_yaw" default="0"/>
   <link name="world"/>
   <xacro:indomitus_panel parent_link="world">
-    <origin xyz="0 0 0" rpy="0 0 0"/>
+    <origin xyz="$(arg panel_x) $(arg panel_y) $(arg panel_z)" rpy="0 0 $(arg panel_yaw)"/>
   </xacro:indomitus_panel>
 </robot>

Commit message: feat(arm): add ArUco panel detection and MoveIt-based alignment (WIP)

File: src/panel/panel_description/urdf/panel_macro.xacro (robot description, xacro)
@@ -598,8 +598,23 @@
          Flat black squares for pose-detection markers ("AruCo detection"
          in the scoring sheet). Three of the four corners are marked in the
-         reference render (top-left, top-right, bottom-left) — the actual
-         ArUco pattern (numbered tag) is applied as a texture/decal on top
-         of this base square by whichever code renders/prints the markers;
-         this link is just the physical black mount square. -->
+         reference render (top-left, top-right, bottom-left).
+         Tag IDs (4X4_50 dictionary, matching rover_aruco/config/aruco_params.yaml's
+         marker_dict): top_left=20, top_right=21, bottom_left=22. Chosen
+         arbitrarily — nothing was previously assigned anywhere in this repo
+         or on real hardware (see git history). Reassign freely here (and
+         regenerate textures/aruco_tags/*.png + panel_perception's marker-ID
+         params) if the real/competition panel ends up using different
+         numbers. Generated via:
+           cv2.aruco.drawMarker(cv2.aruco.Dictionary_get(cv2.aruco.DICT_4X4_50), <id>, 400)
+         (OpenCV 4.5's legacy API — this workspace's opencv is 4.5.4, which
+         predates the newer generateImageMarker() name.)
+         In sim, the numbered pattern is a separate textured quad mesh
+         (meshes/aruco_tags/panel_marker_<suffix>.obj+.mtl+.png) laid
+         directly on top of the black mount box below — a first attempt
+         using a PBR albedo-map <gazebo><material> override directly on
+         the box primitive silently rendered as flat black (gz-sim's
+         URDF-import path doesn't appear to carry that through), so this
+         uses the same textured-mesh mechanism as any other visual mesh
+         in this file instead, which is the well-supported path. -->
     <xacro:macro name="panel_marker" params="suffix x z">
       <joint name="panel_marker_${suffix}_joint" type="fixed">
@@ -613,4 +628,7 @@
           <material name="marker_black"/>
         </visual>
+        <visual>
+          <geometry><mesh filename="${mesh_path}/aruco_tags/panel_marker_${suffix}.obj"/></geometry>
+        </visual>
         <collision>
           <geometry><box size="0.04 0.002 0.04"/></geometry>
@@ -619,7 +637,7 @@
       </link>
     </xacro:macro>
-    <xacro:panel_marker suffix="top_left"    x="-0.135" z="0.415"/>
-    <xacro:panel_marker suffix="top_right"   x="0.135"  z="0.415"/>
-    <xacro:panel_marker suffix="bottom_left" x="-0.135" z="0.035"/>
+    <xacro:panel_marker suffix="top_left"    x="-0.135" z="0.415"/>  <!-- ArUco id 20 -->
+    <xacro:panel_marker suffix="top_right"   x="0.135"  z="0.415"/>  <!-- ArUco id 21 -->
+    <xacro:panel_marker suffix="bottom_left" x="-0.135" z="0.035"/>  <!-- ArUco id 22 -->
     <xacro:if value="$(arg sim)">
       <!-- panel_base_link only: no gravity, so the board itself neither
