Commit message: feat(panel): support any competition ArUco ID per mount, switch to ARUCO_ORIGINAL dictionary

File: src/panel/panel_description/urdf/panel_macro.xacro (robot description, xacro)
@@ -6,4 +6,18 @@
        with via contact physics, not actuated joints. -->
   <xacro:arg name="sim" default="false"/>
+  <!-- Which ArUco ID sits at which of the panel's 3 fixed physical mounts
+       (top_left/top_right/bottom_left) — per competition rules the panel
+       may use any 3 of IDs {11,13,14,15} in any of these 3 positions, so
+       this is a launch-time choice, not a fixed constant. Defaults below
+       are just one valid arrangement (15 unused) — override via
+       `marker_id_top_left:=13` etc. when building for a real/competition
+       panel layout, or see arm_gazebo.launch.py for randomizing this
+       choice on every sim launch. Must stay in sync with
+       panel_perception's matching `marker_id_top_left`/
+       `marker_id_top_right`/`marker_id_bottom_left` ROS parameters on
+       panel_pose_fuser_node — see that package for the other half. -->
+  <xacro:arg name="marker_id_top_left" default="11"/>
+  <xacro:arg name="marker_id_top_right" default="13"/>
+  <xacro:arg name="marker_id_bottom_left" default="14"/>
   <xacro:macro name="indomitus_panel" params="parent_link *origin">
     <xacro:property name="mesh_path" value="package://panel_description/meshes"/>
@@ -599,23 +613,26 @@
          in the scoring sheet). Three of the four corners are marked in the
          reference render (top-left, top-right, bottom-left).
-         Tag IDs (4X4_50 dictionary, matching rover_aruco/config/aruco_params.yaml's
-         marker_dict): top_left=20, top_right=21, bottom_left=22. Chosen
-         arbitrarily — nothing was previously assigned anywhere in this repo
-         or on real hardware (see git history). Reassign freely here (and
-         regenerate textures/aruco_tags/*.png + panel_perception's marker-ID
-         params) if the real/competition panel ends up using different
-         numbers. Generated via:
-           cv2.aruco.drawMarker(cv2.aruco.Dictionary_get(cv2.aruco.DICT_4X4_50), <id>, 400)
-         (OpenCV 4.5's legacy API — this workspace's opencv is 4.5.4, which
-         predates the newer generateImageMarker() name.)
+         Tag IDs (ARUCO_ORIGINAL dictionary — the original ArUco set, per
+         competition rules, NOT 4X4_50 — matching
+         rover_aruco/config/aruco_params.yaml's marker_dict) are a
+         launch-time choice now, not fixed per mount —
+         see the marker_id_top_left/top_right/bottom_left xacro:args above.
+         The textured quad mesh referenced below is picked BY ID
+         (meshes/aruco_tags/marker_<id>.obj+.mtl+.png), decoupled from
+         which physical corner (suffix) it's mounted at, so any of the 4
+         competition IDs {11,13,14,15} can go on any of the 3 mounts.
+         Pre-generated for IDs {11,13,14,15} plus this repo's own dev/sim
+         defaults {20,21,22} — regenerate via
+         generate_marker_meshes.py + the PNG recipe in this directory's
+         README.md if a different ID is ever needed.
          In sim, the numbered pattern is a separate textured quad mesh
-         (meshes/aruco_tags/panel_marker_<suffix>.obj+.mtl+.png) laid
-         directly on top of the black mount box below — a first attempt
-         using a PBR albedo-map <gazebo><material> override directly on
-         the box primitive silently rendered as flat black (gz-sim's
-         URDF-import path doesn't appear to carry that through), so this
-         uses the same textured-mesh mechanism as any other visual mesh
-         in this file instead, which is the well-supported path. -->
-    <xacro:macro name="panel_marker" params="suffix x z">
+         laid directly on top of the black mount box below — a first
+         attempt using a PBR albedo-map <gazebo><material> override
+         directly on the box primitive silently rendered as flat black
+         (gz-sim's URDF-import path doesn't appear to carry that through),
+         so this uses the same textured-mesh mechanism as any other
+         visual mesh in this file instead, which is the well-supported
+         path. -->
+    <xacro:macro name="panel_marker" params="suffix marker_id x z">
       <joint name="panel_marker_${suffix}_joint" type="fixed">
         <parent link="panel_base_link"/>
@@ -629,5 +646,5 @@
         </visual>
         <visual>
-          <geometry><mesh filename="${mesh_path}/aruco_tags/panel_marker_${suffix}.obj"/></geometry>
+          <geometry><mesh filename="${mesh_path}/aruco_tags/marker_${marker_id}.obj"/></geometry>
         </visual>
         <collision>
@@ -637,7 +654,7 @@
       </link>
     </xacro:macro>
-    <xacro:panel_marker suffix="top_left"    x="-0.135" z="0.415"/>  <!-- ArUco id 20 -->
-    <xacro:panel_marker suffix="top_right"   x="0.135"  z="0.415"/>  <!-- ArUco id 21 -->
-    <xacro:panel_marker suffix="bottom_left" x="-0.135" z="0.035"/>  <!-- ArUco id 22 -->
+    <xacro:panel_marker suffix="top_left"    marker_id="$(arg marker_id_top_left)"    x="-0.135" z="0.415"/>
+    <xacro:panel_marker suffix="top_right"   marker_id="$(arg marker_id_top_right)"   x="0.135"  z="0.415"/>
+    <xacro:panel_marker suffix="bottom_left" marker_id="$(arg marker_id_bottom_left)" x="-0.135" z="0.035"/>
     <xacro:if value="$(arg sim)">
       <!-- panel_base_link only: no gravity, so the board itself neither

Commit message: Feature/arm/panel detection align (#540)
* feat(arm): add ArUco panel detection and MoveIt-based alignment (WIP)

* fix(panel): resolve panel placement, ArUco orientation, and MoveIt frame bugs blocking align

* fix(arm): fix stale key state on panel prompt, stale docstring, and scipy/numpy ABI conflict

* fix(rover_aruco): install config/launch as subdirectories, not flattened into share root

* feat(arm): replay first successful panel-align position instead of re-planning every 'p'

* fix(arm): pin panel align to OMPL pipeline (was silently falling back to CHOMP), drop Ruckig from adapter chain

* chore(panel): make panel_pose_fuser_node's topic defaults absolute, matching consumers

* fix(arm): pin move_group to OMPL pipeline and complete arm_standalone's real-hardware bringup

* fix(arm): raise Servo start/stop timeouts to match real hardware's slower response

* feat(arm): make panel align standoff and aim height configurable, tuned for the real panel

* feat(panel): fuse panel orientation from marker edge geometry instead of per-marker averaging

* feat(panel): make marker ID to mount assignment configurable, require all 3 markers to publish

* feat(panel): support any competition ArUco ID per mount, switch to ARUCO_ORIGINAL dictionary

* feat(sim): randomize panel marker ID layout on every launch

* chore(arm): add wrist camera calibration data for the real arm

* chore(arm): drop redundant raw calibration artifacts, default camera_info_url to the checked-in calibration

* feat(arm): add cross-process arm-motion lock (flock-based, not just per-process threading.Lock)

* fix(arm): cancel hung execution goals, block home/align races, replay via collision-checked MoveIt plan

* fix(panel): scope sim marker layout file by ROS_DOMAIN_ID, ignore stale leftovers

* fix(sim): scope marker layout file by domain, support reproducible seed, clean up on shutdown

* fix(arm): move camera calibration into arm_sensors package, resolve path via FindPackageShare

* chore(arm): pin scipy to an exact version instead of an open-ended floor

File: src/panel/panel_description/urdf/panel_macro.xacro (robot description, xacro)
@@ -6,4 +6,18 @@
        with via contact physics, not actuated joints. -->
   <xacro:arg name="sim" default="false"/>
+  <!-- Which ArUco ID sits at which of the panel's 3 fixed physical mounts
+       (top_left/top_right/bottom_left) — per competition rules the panel
+       may use any 3 of IDs {11,13,14,15} in any of these 3 positions, so
+       this is a launch-time choice, not a fixed constant. Defaults below
+       are just one valid arrangement (15 unused) — override via
+       `marker_id_top_left:=13` etc. when building for a real/competition
+       panel layout, or see arm_gazebo.launch.py for randomizing this
+       choice on every sim launch. Must stay in sync with
+       panel_perception's matching `marker_id_top_left`/
+       `marker_id_top_right`/`marker_id_bottom_left` ROS parameters on
+       panel_pose_fuser_node — see that package for the other half. -->
+  <xacro:arg name="marker_id_top_left" default="11"/>
+  <xacro:arg name="marker_id_top_right" default="13"/>
+  <xacro:arg name="marker_id_bottom_left" default="14"/>
   <xacro:macro name="indomitus_panel" params="parent_link *origin">
     <xacro:property name="mesh_path" value="package://panel_description/meshes"/>
@@ -598,9 +612,27 @@
          Flat black squares for pose-detection markers ("AruCo detection"
          in the scoring sheet). Three of the four corners are marked in the
-         reference render (top-left, top-right, bottom-left) — the actual
-         ArUco pattern (numbered tag) is applied as a texture/decal on top
-         of this base square by whichever code renders/prints the markers;
-         this link is just the physical black mount square. -->
-    <xacro:macro name="panel_marker" params="suffix x z">
+         reference render (top-left, top-right, bottom-left).
+         Tag IDs (ARUCO_ORIGINAL dictionary — the original ArUco set, per
+         competition rules, NOT 4X4_50 — matching
+         rover_aruco/config/aruco_params.yaml's marker_dict) are a
+         launch-time choice now, not fixed per mount —
+         see the marker_id_top_left/top_right/bottom_left xacro:args above.
+         The textured quad mesh referenced below is picked BY ID
+         (meshes/aruco_tags/marker_<id>.obj+.mtl+.png), decoupled from
+         which physical corner (suffix) it's mounted at, so any of the 4
+         competition IDs {11,13,14,15} can go on any of the 3 mounts.
+         Pre-generated for IDs {11,13,14,15} plus this repo's own dev/sim
+         defaults {20,21,22} — regenerate via
+         generate_marker_meshes.py + the PNG recipe in this directory's
+         README.md if a different ID is ever needed.
+         In sim, the numbered pattern is a separate textured quad mesh
+         laid directly on top of the black mount box below — a first
+         attempt using a PBR albedo-map <gazebo><material> override
+         directly on the box primitive silently rendered as flat black
+         (gz-sim's URDF-import path doesn't appear to carry that through),
+         so this uses the same textured-mesh mechanism as any other
+         visual mesh in this file instead, which is the well-supported
+         path. -->
+    <xacro:macro name="panel_marker" params="suffix marker_id x z">
       <joint name="panel_marker_${suffix}_joint" type="fixed">
         <parent link="panel_base_link"/>
@@ -613,4 +645,7 @@
           <material name="marker_black"/>
         </visual>
+        <visual>
+          <geometry><mesh filename="${mesh_path}/aruco_tags/marker_${marker_id}.obj"/></geometry>
+        </visual>
         <collision>
           <geometry><box size="0.04 0.002 0.04"/></geometry>
@@ -619,7 +654,7 @@
       </link>
     </xacro:macro>
-    <xacro:panel_marker suffix="top_left"    x="-0.135" z="0.415"/>
-    <xacro:panel_marker suffix="top_right"   x="0.135"  z="0.415"/>
-    <xacro:panel_marker suffix="bottom_left" x="-0.135" z="0.035"/>
+    <xacro:panel_marker suffix="top_left"    marker_id="$(arg marker_id_top_left)"    x="-0.135" z="0.415"/>
+    <xacro:panel_marker suffix="top_right"   marker_id="$(arg marker_id_top_right)"   x="0.135"  z="0.415"/>
+    <xacro:panel_marker suffix="bottom_left" marker_id="$(arg marker_id_bottom_left)" x="-0.135" z="0.035"/>
     <xacro:if value="$(arg sim)">
       <!-- panel_base_link only: no gravity, so the board itself neither
